File: iceberg20.sch (EAGLE design)
At the start: 0 parts

Commit message: und nochmal etwas merge
Other:
- note added: "IR-Empfänger"
- note added: "IR-Sender"

Commit message: ultimate merge yeah!
Changed lines of the file:
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@@
 <setting verticaltext="up"/>
 </settings>
-<grid distance="0.1" unitdist="inch" unit="inch" style="lines" multiple="1" display="no" altdistance="0.01" altunitdist="inch" altunit="inch"/>
+<grid distance="0.1" unitdist="inch" unit="inch" style="lines" multiple="2" display="yes" altdistance="0.01" altunitdist="inch" altunit="inch"/>
 <layers>
 <layer number="1" name="Top" color="4" fill="1" visible="no" active="no"/>
@@
 <part name="GND6" library="supply1" library_urn="urn:adsk.eagle:library:371" deviceset="GND" device=""/>
 <part name="FRAME1" library="frames" library_urn="urn:adsk.eagle:library:229" deviceset="A4L-LOC" device=""/>
-<part name="+" library="testpad" library_urn="urn:adsk.eagle:library:385" deviceset="TP" device="B1,27" package3d_urn="urn:adsk.eagle:package:27944/1" value="TPB1,27"/>
-<part name="-" library="testpad" library_urn="urn:adsk.eagle:library:385" deviceset="TP" device="B1,27" package3d_urn="urn:adsk.eagle:package:27944/1" value="TPB1,27"/>
-<part name="I" library="testpad" library_urn="urn:adsk.eagle:library:385" deviceset="TP" device="B1,27" package3d_urn="urn:adsk.eagle:package:27944/1" value="TPB1,27"/>
-<part name="EN" library="testpad" library_urn="urn:adsk.eagle:library:385" deviceset="TP" device="B1,27" package3d_urn="urn:adsk.eagle:package:27944/1" value="TPB1,27"/>
-<part name="IN2" library="testpad" library_urn="urn:adsk.eagle:library:385" deviceset="TP" device="B1,27" package3d_urn="urn:adsk.eagle:package:27944/1" value="TPB1,27"/>
-<part name="IN1" library="testpad" library_urn="urn:adsk.eagle:library:385" deviceset="TP" device="B1,27" package3d_urn="urn:adsk.eagle:package:27944/1" value="TPB1,27"/>
-<part name="VS" library="testpad" library_urn="urn:adsk.eagle:library:385" deviceset="TP" device="B1,27" package3d_urn="urn:adsk.eagle:package:27944/1" value="TPB1,27"/>
+<part name="+" library="testpad" library_urn="urn:adsk.eagle:library:385" deviceset="TP" device="B1,27" package3d_urn="urn:adsk.eagle:package:27944/2" value="TPB1,27"/>
+<part name="-" library="testpad" library_urn="urn:adsk.eagle:library:385" deviceset="TP" device="B1,27" package3d_urn="urn:adsk.eagle:package:27944/2" value="TPB1,27"/>
+<part name="I" library="testpad" library_urn="urn:adsk.eagle:library:385" deviceset="TP" device="B1,27" package3d_urn="urn:adsk.eagle:package:27944/2" value="TPB1,27"/>
+<part name="EN" library="testpad" library_urn="urn:adsk.eagle:library:385" deviceset="TP" device="B1,27" package3d_urn="urn:adsk.eagle:package:27944/2" value="TPB1,27"/>
+<part name="IN2" library="testpad" library_urn="urn:adsk.eagle:library:385" deviceset="TP" device="B1,27" package3d_urn="urn:adsk.eagle:package:27944/2" value="TPB1,27"/>
+<part name="IN1" library="testpad" library_urn="urn:adsk.eagle:library:385" deviceset="TP" device="B1,27" package3d_urn="urn:adsk.eagle:package:27944/2" value="TPB1,27"/>
+<part name="VS" library="testpad" library_urn="urn:adsk.eagle:library:385" deviceset="TP" device="B1,27" package3d_urn="urn:adsk.eagle:package:27944/2" value="TPB1,27"/>
 </parts>
 <sheets>
@@
 <part name="P+3" library="supply1" library_urn="urn:adsk.eagle:library:371" deviceset="+5V" device=""/>
 <part name="GND3" library="supply1" library_urn="urn:adsk.eagle:library:371" deviceset="GND" device=""/>
-<part name="C1" library="iceberg20" deviceset="ELKO" device="-THT-1UF" package3d_urn="urn:adsk.eagle:package:12868066/1" value="1 uF"/>
+<part name="C1" library="iceberg20" deviceset="ELKO" device="-THT-1UF" package3d_urn="urn:adsk.eagle:package:12868066/1" value="1 uF, 50 V, ±20 %"/>
 <part name="GND4" library="supply1" library_urn="urn:adsk.eagle:library:371" deviceset="GND" device=""/>
 <part name="P+4" library="supply1" library_urn="urn:adsk.eagle:library:371" deviceset="+5V" device=""/>
@@
 </modules>
 <parts>
-<part name="GND1" library="iceberg20" deviceset="GND" device=""/>
-<part name="GND2" library="iceberg20" deviceset="GND" device=""/>
-<part name="GND3" library="iceberg20" deviceset="GND" device=""/>
-<part name="GND4" library="iceberg20" deviceset="GND" device=""/>
-<part name="GND5" library="iceberg20" deviceset="GND" device=""/>
-<part name="P+1" library="iceberg20" deviceset="+12V" device=""/>
-<part name="GND6" library="iceberg20" deviceset="GND" device=""/>
-<part name="P+2" library="iceberg20" deviceset="+12V" device=""/>
 </parts>
 <sheets>
@@
 </moduleinsts>
 <instances>
-<instance part="GND1" gate="1" x="146.05" y="128.27" smashed="yes">
-<attribute name="VALUE" x="143.51" y="125.73" size="1.778" layer="96"/>
-</instance>
-<instance part="GND2" gate="1" x="148.59" y="82.55" smashed="yes">
-<attribute name="VALUE" x="146.05" y="80.01" size="1.778" layer="96"/>
-</instance>
-<instance part="GND3" gate="1" x="148.59" y="44.45" smashed="yes">
-<attribute name="VALUE" x="146.05" y="41.91" size="1.778" layer="96"/>
-</instance>
-<instance part="GND4" gate="1" x="148.59" y="6.35" smashed="yes">
-<attribute name="VALUE" x="146.05" y="3.81" size="1.778" layer="96"/>
-</instance>
-<instance part="GND5" gate="1" x="148.59" y="-31.75" smashed="yes">
-<attribute name="VALUE" x="146.05" y="-34.29" size="1.778" layer="96"/>
-</instance>
-<instance part="P+1" gate="1" x="158.75" y="158.75" smashed="yes">
-<attribute name="VALUE" x="156.21" y="161.29" size="1.778" layer="96"/>
-</instance>
-<instance part="GND6" gate="1" x="110.49" y="148.59" smashed="yes">
-<attribute name="VALUE" x="107.95" y="146.05" size="1.778" layer="96"/>
-</instance>
-<instance part="P+2" gate="1" x="110.49" y="168.91" smashed="yes">
-<attribute name="VALUE" x="107.95" y="171.45" size="1.778" layer="96"/>
-</instance>
 </instances>
 <busses>
@@
 </busses>
 <nets>
-<net name="GND" class="0">
-<segment>
-<portref moduleinst="F1" port="GND"/>
-<pinref part="GND1" gate="1" pin="GND"/>
-<wire x1="148.59" y1="130.81" x2="146.05" y2="130.81" width="0.1524" layer="91"/>
-</segment>
-<segment>
-<portref moduleinst="M0" port="GND"/>
-<pinref part="GND2" gate="1" pin="GND"/>
-</segment>
-<segment>
-<portref moduleinst="M1" port="GND"/>
-<pinref part="GND3" gate="1" pin="GND"/>
-</segment>
-<segment>
-<portref moduleinst="M2" port="GND"/>
-<pinref part="GND4" gate="1" pin="GND"/>
-</segment>
-<segment>
-<portref moduleinst="M3" port="GND"/>
-<pinref part="GND5" gate="1" pin="GND"/>
-</segment>
-<segment>
-<pinref part="GND6" gate="1" pin="GND"/>
-<portref moduleinst="P1" port="GND"/>
-<wire x1="109.22" y1="152.4" x2="110.49" y2="152.4" width="0.1524" layer="91"/>
-<wire x1="110.49" y1="152.4" x2="110.49" y2="151.13" width="0.1524" layer="91"/>
-</segment>
-</net>
 <net name="MOTOR-SUPPLY" class="0">
 <segment>
@@
 <wire x1="115.57" y1="19.05" x2="97.79" y2="19.05" width="0.1524" layer="91"/>
 <label x="104.14" y="16.51" size="1.778" layer="95"/>
-</segment>
-</net>
-<net name="+12V" class="0">
-<segment>
-<pinref part="P+1" gate="1" pin="+12V"/>
-<portref moduleinst="F1" port="IN"/>
-<wire x1="158.75" y1="156.21" x2="158.75" y2="153.67" width="0.1524" layer="91"/>
-</segment>
-<segment>
-<pinref part="P+2" gate="1" pin="+12V"/>
-<portref moduleinst="P1" port="PWR+"/>
-<wire x1="110.49" y1="166.37" x2="110.49" y2="162.56" width="0.1524" layer="91"/>
-<wire x1="110.49" y1="162.56" x2="109.22" y2="162.56" width="0.1524" layer="91"/>
 </segment>
 </net>
@@
 packages will not be understood (or retained) with this version.
 </note>
+<note version="8.4" severity="warning">
+Since Version 8.4, EAGLE supports properties for SPICE simulation.
+Probes in schematics and SPICE mapping objects found in parts and library devices
+will not be understood with this version. Update EAGLE to the latest version
+for full support of SPICE simulation.
+</note>
 </compatibility>

Commit message: + sch (Bluetooth)
Other:
- note added: "Bluetooth HC-05"

Commit message: + sch(Sensoren)
Other:
- note added: "Sensoren"

Commit message: + sch(Anschlüsse NOT FINISHED)
Other:
- note added: "Anschlüsse"
Changed lines of the file:
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@@
+</sheets>
+</module>
+<module name="ANSCHLUESSE" prefix="" dx="30.48" dy="20.32">
+<ports>
+</ports>
+<variantdefs>
+</variantdefs>
+<parts>
+<part name="FRAME1" library="iceberg20" deviceset="FRAME" device=""/>
+</parts>
+<sheets>
+<sheet>
+<plain>
+<text x="217.258928125" y="20.404425" size="2.54" layer="94">Anschlüsse</text>
+</plain>
+<instances>
+<instance part="FRAME1" gate="G$1" x="0" y="0" smashed="yes">
+<attribute name="DRAWING_NAME" x="217.17" y="15.24" size="2.54" layer="94"/>
+<attribute name="LAST_DATE_TIME" x="217.17" y="10.16" size="2.286" layer="94"/>
+<attribute name="SHEET" x="230.505" y="5.08" size="2.54" layer="94"/>
+</instance>
+</instances>
+<busses>
+</busses>
+<nets>
+</nets>
+</sheet>
 </sheets>
 </module>

Commit message: + lbr sch (Encoder, Jumper)
Other:
- note added: "Encoder"
Changed lines of the file:
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@@
 <setting verticaltext="up"/>
 </settings>
-<grid distance="0.1" unitdist="inch" unit="inch" style="lines" multiple="1" display="yes" altdistance="0.01" altunitdist="inch" altunit="inch"/>
+<grid distance="0.1" unitdist="inch" unit="inch" style="lines" multiple="1" display="no" altdistance="0.01" altunitdist="inch" altunit="inch"/>
 <layers>
 <layer number="1" name="Top" color="4" fill="1" visible="no" active="no"/>
@@
 </sheets>
 </module>
-<module name="SENSOREN" prefix="" dx="30.48" dy="20.32">
+<module name="ANSCHLUESSE" prefix="" dx="30.48" dy="20.32">
 <ports>
 </ports>
@@
 <parts>
 <part name="FRAME1" library="iceberg20" deviceset="FRAME" device=""/>
+<part name="FRAME2" library="iceberg20" deviceset="FRAME" device=""/>
 <part name="IC1" library="iceberg20" deviceset="LM-35" device=""/>
 <part name="IC4" library="iceberg20" deviceset="SRF-08" device=""/>
@@
 </plain>
 <instances>
-<instance part="FRAME1" gate="G$1" x="0" y="0" smashed="yes">
+<instance part="FRAME2" gate="G$1" x="0" y="0" smashed="yes">
 <attribute name="DRAWING_NAME" x="217.17" y="15.24" size="2.54" layer="94"/>
 <attribute name="LAST_DATE_TIME" x="217.17" y="10.16" size="2.286" layer="94"/>
@@
 </nets>
 </sheet>
-</sheets>
-</module>
-<module name="ANSCHLUESSE" prefix="" dx="30.48" dy="20.32">
-<ports>
-</ports>
-<variantdefs>
-</variantdefs>
-<parts>
-<part name="FRAME1" library="iceberg20" deviceset="FRAME" device=""/>
-</parts>
-<sheets>
 <sheet>
 <plain>
@@
 </nets>
 </sheet>
+</sheets>
+</module>
+<module name="ENCODER" prefix="ENC" dx="30.48" dy="20.32">
+<ports>
+</ports>
+<variantdefs>
+</variantdefs>
+<parts>
+<part name="FRAME1" library="iceberg20" deviceset="FRAME" device=""/>
+<part name="IC1" library="iceberg20" deviceset="TEENSY-3.2" device=""/>
+<part name="GND1" library="supply1" library_urn="urn:adsk.eagle:library:371" deviceset="GND" device=""/>
+<part name="P+1" library="supply1" library_urn="urn:adsk.eagle:library:371" deviceset="+5V" device=""/>
+</parts>
+<sheets>
+<sheet>
+<plain>
+<text x="217.17" y="20.32" size="2.54" layer="94">Encoder</text>
+</plain>
+<instances>
+<instance part="FRAME1" gate="G$1" x="0" y="0" smashed="yes">
+<attribute name="DRAWING_NAME" x="217.17" y="15.24" size="2.54" layer="94"/>
+<attribute name="LAST_DATE_TIME" x="217.17" y="10.16" size="2.286" layer="94"/>
+<attribute name="SHEET" x="230.505" y="5.08" size="2.54" layer="94"/>
+</instance>
+<instance part="IC1" gate="G$1" x="129.54" y="93.98" smashed="yes">
+<attribute name="NAME" x="124.46" y="124.714" size="1.778" layer="95" font="vector"/>
+<attribute name="VALUE" x="124.46" y="60.706" size="1.778" layer="96" font="vector" align="top-left"/>
+</instance>
+<instance part="GND1" gate="1" x="111.76" y="55.88" smashed="yes">
+<attribute name="VALUE" x="111.76" y="53.34" size="1.778" layer="96"/>
+</instance>
+<instance part="P+1" gate="1" x="104.14" y="91.44" smashed="yes">
+<attribute name="VALUE" x="101.6" y="86.36" size="1.778" layer="96" rot="R90"/>
+</instance>
+</instances>
+<busses>
+<bus name="ENCODER-SIGNALS:ENA[0..3],ENB[0..3]">
+<segment>
+<wire x1="99.06" y1="114.3" x2="99.06" y2="129.54" width="0.762" layer="92"/>
+<wire x1="99.06" y1="129.54" x2="165.1" y2="129.54" width="0.762" layer="92"/>
+<wire x1="165.1" y1="129.54" x2="165.1" y2="93.98" width="0.762" layer="92"/>
+</segment>
+</bus>
+</busses>
+<nets>
+<net name="N$11" class="0">
+<segment>
+<wire x1="104.14" y1="86.36" x2="104.14" y2="88.9" width="0.1524" layer="91"/>
+<pinref part="P+1" gate="1" pin="+5V"/>
+<pinref part="IC1" gate="G$1" pin="VIN"/>
+<wire x1="104.14" y1="86.36" x2="111.76" y2="86.36" width="0.1524" layer="91"/>
+</segment>
+</net>
+<net name="GND" class="0">
+<segment>
+<pinref part="IC1" gate="G$1" pin="AGND"/>
+<pinref part="IC1" gate="G$1" pin="GND"/>
+<wire x1="111.76" y1="68.58" x2="111.76" y2="66.04" width="0.1524" layer="91"/>
+<pinref part="IC1" gate="G$1" pin="GND1"/>
+<wire x1="111.76" y1="66.04" x2="111.76" y2="63.5" width="0.1524" layer="91"/>
+<junction x="111.76" y="66.04"/>
+<pinref part="GND1" gate="1" pin="GND"/>
+<wire x1="111.76" y1="63.5" x2="111.76" y2="58.42" width="0.1524" layer="91"/>
+<junction x="111.76" y="63.5"/>
+</segment>
+</net>
+<net name="SCL" class="0">
+<segment>
+<pinref part="IC1" gate="G$1" pin="A5/19/SCL0"/>
+<label x="154.94" y="114.3" size="1.778" layer="95" xref="yes"/>
+<wire x1="144.78" y1="114.3" x2="154.94" y2="114.3" width="0.1524" layer="91"/>
+</segment>
+</net>
+<net name="SDA" class="0">
+<segment>
+<pinref part="IC1" gate="G$1" pin="A4/18/SDA0"/>
+<wire x1="144.78" y1="116.84" x2="147.32" y2="116.84" width="0.1524" layer="91"/>
+<label x="147.32" y="116.84" size="1.778" layer="95" xref="yes"/>
+</segment>
+</net>
+<net name="ENA0" class="0">
+<segment>
+<pinref part="IC1" gate="G$1" pin="2"/>
+<wire x1="144.78" y1="101.6" x2="165.1" y2="101.6" width="0.1524" layer="91"/>
+<label x="154.94" y="101.6" size="1.778" layer="95"/>
+</segment>
+</net>
+<net name="ENB0" class="0">
+<segment>
+<pinref part="IC1" gate="G$1" pin="3*"/>
+<wire x1="144.78" y1="99.06" x2="165.1" y2="99.06" width="0.1524" layer="91"/>
+<label x="154.94" y="99.06" size="1.778" layer="95"/>
+</segment>
+</net>
+<net name="ENA1" class="0">
+<segment>
+<pinref part="IC1" gate="G$1" pin="4*"/>
+<wire x1="144.78" y1="96.52" x2="165.1" y2="96.52" width="0.1524" layer="91"/>
+<label x="154.94" y="96.52" size="1.778" layer="95"/>
+</segment>
+</net>
+<net name="ENB1" class="0">
+<segment>
+<pinref part="IC1" gate="G$1" pin="5*"/>
+<wire x1="144.78" y1="93.98" x2="165.1" y2="93.98" width="0.1524" layer="91"/>
+<label x="154.94" y="93.98" size="1.778" layer="95"/>
+</segment>
+</net>
+<net name="ENA3" class="0">
+<segment>
+<pinref part="IC1" gate="G$1" pin="A2/16"/>
+<wire x1="111.76" y1="116.84" x2="99.06" y2="116.84" width="0.1524" layer="91"/>
+<label x="101.6" y="116.84" size="1.778" layer="95"/>
+</segment>
+</net>
+<net name="ENB3" class="0">
+<segment>
+<pinref part="IC1" gate="G$1" pin="A3/17"/>
+<wire x1="111.76" y1="114.3" x2="99.06" y2="114.3" width="0.1524" layer="91"/>
+<label x="101.6" y="114.3" size="1.778" layer="95"/>
+</segment>
+</net>
+<net name="ENB2" class="0">
+<segment>
+<pinref part="IC1" gate="G$1" pin="A1/15"/>
+<wire x1="111.76" y1="119.38" x2="99.06" y2="119.38" width="0.1524" layer="91"/>
+<label x="101.6" y="119.38" size="1.778" layer="95"/>
+</segment>
+</net>
+<net name="ENA2" class="0">
+<segment>
+<pinref part="IC1" gate="G$1" pin="A0/14"/>
+<wire x1="111.76" y1="121.92" x2="99.06" y2="121.92" width="0.1524" layer="91"/>
+<label x="101.6" y="121.92" size="1.778" layer="95"/>
+</segment>
+</net>
+</nets>
+</sheet>
