File: iceberg20.sch (EAGLE design)
At the start: 0 parts

Commit message: + sch(Sensoren, Ein/Ausgabe)
Other:
- note removed: "Anschlüsse"

Commit message: + sch (Ein/Ausgabe)
Other:
- note added: "Ein/Ausgabe"

Commit message: + sch (Anschlüsse)
Other:
- note added: "Anschlüsse"

Commit message: + sch (5V-Linearwandler)
Other:
- note added: "5V-Wandler"
Changed lines of the file:
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@@
 <?xml version="1.0" encoding="utf-8"?>
 <!DOCTYPE eagle SYSTEM "eagle.dtd">
-<eagle version="9.5.0">
+<eagle version="9.4.2">
 <drawing>
 <settings>
@@
 </segment>
 </net>
+</nets>
+</sheet>
+</sheets>
+</module>
+<module name="5V-WANDLER" prefix="" dx="30.48" dy="20.32">
+<ports>
+</ports>
+<variantdefs>
+</variantdefs>
+<parts>
+<part name="FRAME1" library="iceberg20" deviceset="FRAME" device=""/>
+<part name="IC1" library="iceberg20" deviceset="L7805CV" device="" package3d_urn="urn:adsk.eagle:package:13445399/1"/>
+<part name="C1" library="iceberg20" deviceset="C" device="0805" package3d_urn="urn:adsk.eagle:package:12867820/1" value="0.1uF"/>
+<part name="C2" library="iceberg20" deviceset="C" device="0805" package3d_urn="urn:adsk.eagle:package:12867820/1" value="0.33uF"/>
+<part name="GND4" library="supply1" library_urn="urn:adsk.eagle:library:371" deviceset="GND" device=""/>
+<part name="P+2" library="supply1" library_urn="urn:adsk.eagle:library:371" deviceset="+12V" device=""/>
+<part name="P+3" library="supply1" library_urn="urn:adsk.eagle:library:371" deviceset="+5V" device=""/>
+</parts>
+<sheets>
+<sheet>
+<plain>
+<text x="217.17" y="20.32" size="2.54" layer="94">5V-Wandler</text>
+</plain>
+<instances>
+<instance part="FRAME1" gate="G$1" x="0" y="0" smashed="yes">
+<attribute name="DRAWING_NAME" x="217.17" y="15.24" size="2.54" layer="94"/>
+<attribute name="LAST_DATE_TIME" x="217.17" y="10.16" size="2.286" layer="94"/>
+<attribute name="SHEET" x="230.505" y="5.08" size="2.54" layer="94"/>
+</instance>
+<instance part="IC1" gate="G$1" x="124.46" y="93.98" smashed="yes">
+<attribute name="NAME" x="116.84" y="104.14" size="1.27" layer="95" align="top-left"/>
+<attribute name="VALUE" x="116.84" y="88.9" size="1.27" layer="96"/>
+</instance>
+<instance part="C1" gate="G$1" x="139.7" y="93.98" smashed="yes">
+<attribute name="NAME" x="141.224" y="94.361" size="1.778" layer="95"/>
+<attribute name="VALUE" x="141.224" y="89.281" size="1.778" layer="96"/>
+</instance>
+<instance part="C2" gate="G$1" x="109.22" y="93.98" smashed="yes">
+<attribute name="NAME" x="110.744" y="94.361" size="1.778" layer="95"/>
+<attribute name="VALUE" x="110.744" y="89.281" size="1.778" layer="96"/>
+</instance>
+<instance part="GND4" gate="1" x="124.46" y="78.74" smashed="yes">
+<attribute name="VALUE" x="121.92" y="76.2" size="1.778" layer="96"/>
+</instance>
+<instance part="P+2" gate="1" x="104.14" y="106.68" smashed="yes">
+<attribute name="VALUE" x="101.6" y="101.6" size="1.778" layer="96" rot="R90"/>
+</instance>
+<instance part="P+3" gate="1" x="144.78" y="106.68" smashed="yes">
+<attribute name="VALUE" x="147.32" y="109.22" size="1.778" layer="96" rot="R180"/>
+</instance>
+</instances>
+<busses>
+</busses>
+<nets>
+<net name="GND" class="0">
+<segment>
+<pinref part="C2" gate="G$1" pin="2"/>
+<wire x1="109.22" y1="88.9" x2="109.22" y2="86.36" width="0.1524" layer="91"/>
+<wire x1="109.22" y1="86.36" x2="124.46" y2="86.36" width="0.1524" layer="91"/>
+<pinref part="IC1" gate="G$1" pin="GND"/>
+<wire x1="124.46" y1="86.36" x2="124.46" y2="88.9" width="0.1524" layer="91"/>
+<pinref part="C1" gate="G$1" pin="2"/>
+<wire x1="139.7" y1="88.9" x2="139.7" y2="86.36" width="0.1524" layer="91"/>
+<wire x1="139.7" y1="86.36" x2="124.46" y2="86.36" width="0.1524" layer="91"/>
+<wire x1="124.46" y1="86.36" x2="124.46" y2="81.28" width="0.1524" layer="91"/>
+<junction x="124.46" y="86.36"/>
+<pinref part="GND4" gate="1" pin="GND"/>
+</segment>
+</net>
+<net name="+12V" class="0">
+<segment>
+<pinref part="IC1" gate="G$1" pin="V-I"/>
+<wire x1="114.3" y1="99.06" x2="109.22" y2="99.06" width="0.1524" layer="91"/>
+<pinref part="C2" gate="G$1" pin="1"/>
+<wire x1="109.22" y1="99.06" x2="109.22" y2="96.52" width="0.1524" layer="91"/>
+<wire x1="109.22" y1="99.06" x2="104.14" y2="99.06" width="0.1524" layer="91"/>
+<junction x="109.22" y="99.06"/>
+<pinref part="P+2" gate="1" pin="+12V"/>
+<wire x1="104.14" y1="104.14" x2="104.14" y2="99.06" width="0.1524" layer="91"/>
+</segment>
+</net>
+<net name="+5V" class="0">
+<segment>
+<pinref part="C1" gate="G$1" pin="1"/>
+<wire x1="139.7" y1="96.52" x2="139.7" y2="99.06" width="0.1524" layer="91"/>
+<pinref part="IC1" gate="G$1" pin="V-O"/>
+<wire x1="139.7" y1="99.06" x2="134.62" y2="99.06" width="0.1524" layer="91"/>
+<wire x1="139.7" y1="99.06" x2="144.78" y2="99.06" width="0.1524" layer="91"/>
+<junction x="139.7" y="99.06"/>
+<pinref part="P+3" gate="1" pin="+5V"/>
+<wire x1="144.78" y1="104.14" x2="144.78" y2="99.06" width="0.1524" layer="91"/>
+</segment>
+</net>

Commit message: + sch (5V-Linearwandler, Schaltregler Module)
Other:
- note added: "5V-Schaltregler"
- note added: "Linearwandler"
- note removed: "5V-Wandler"
