File: iceberg20.sch (EAGLE design)
At the start: 0 parts

Commit message: ~ sch (Motor: alte Bauteile mit neuen ausgetauscht)
Other:
- note added: "Motor"

Commit message: + sch (Beschriftung)
Other:
- note added: "12V"
- note added: "5V"
- note added: "Analog"
- note added: "Digital"
- note added: "Display"
- note added: "Heartbeat"
- note added: "I2C"
- note added: "Knöpfe..."
- note added: "Kompass"
- note added: "LEDs"
- note added: "Oscillator"
- note added: "Phototransistor"
- note added: "Real Time Clock"
- note added: "Reflektion"
- note added: "Speaker"
- note added: "Switch"
- note added: "Temperatur"
- note added: "Ultraschall"
Changed lines of the file:
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@@
 <sheet>
 <plain>
-<text x="181.61" y="41.91" size="2.54" layer="97" rot="R90">Stromsensor</text>
-<text x="107.95" y="74.93" size="2.54" layer="97" rot="R180">Motortreiber</text>
+<text x="176.53" y="38.1" size="3.81" layer="97" rot="R90">Stromsensor</text>
+<text x="111.76" y="76.2" size="3.81" layer="97" rot="R180">Motortreiber</text>
 <text x="74.93" y="36.83" size="2.54" layer="97">EN-Pin</text>
 <text x="29.21" y="67.31" size="1.27" layer="97">DIR-Pins</text>
-<text x="171.45" y="85.09" size="2.54" layer="97">Motor-Anschluss</text>
+<text x="177.8" y="81.28" size="3.81" layer="97">Motor-Anschluss</text>
 <text x="217.17" y="-7.62" size="2.54" layer="94">Motor</text>
 </plain>
@@
 <plain>
 <text x="217.17" y="20.32" size="2.54" layer="94">PUI</text>
+<text x="119.38" y="111.76" size="3.81" layer="97">Display</text>
+<text x="157.48" y="111.76" size="3.81" layer="97">Knöpfe...</text>
 </plain>
 <instances>
@@
 <plain>
 <text x="216.9851625" y="20.32" size="2.54" layer="94">IR-Sender</text>
+<text x="68.58" y="58.42" size="3.81" layer="97">Oscillator</text>
 </plain>
 <instances>
@@
 <plain>
 <text x="217.12224375" y="20.515271875" size="2.54" layer="94">Sensoren</text>
+<text x="127" y="152.4" size="3.81" layer="97">Real Time Clock</text>
+<text x="69.85" y="152.4" size="3.81" layer="97">Temperatur</text>
+<text x="139.7" y="101.6" size="3.81" layer="97">Ultraschall</text>
+<text x="218.44" y="81.28" size="3.81" layer="97">Phototransistor</text>
+<text x="199.39" y="118.11" size="3.81" layer="97">Kompass</text>
+<text x="203.2" y="165.1" size="3.81" layer="97">Reflektion</text>
 </plain>
 <instances>
@@
 <attribute name="VALUE" x="185.42" y="88.9" size="1.778" layer="96"/>
 </instance>
-<instance part="X1" gate="G$1" x="193.04" y="149.86" smashed="yes" rot="R270">
-<attribute name="NAME" x="190.5" y="152.908" size="1.778" layer="95" font="vector"/>
-</instance>
-<instance part="X2" gate="G$1" x="208.28" y="149.86" smashed="yes" rot="R270">
-<attribute name="NAME" x="205.74" y="152.908" size="1.778" layer="95" font="vector"/>
-</instance>
-<instance part="GND12" gate="1" x="195.58" y="124.46" smashed="yes">
-<attribute name="VALUE" x="193.04" y="121.92" size="1.778" layer="96"/>
-</instance>
-<instance part="R2" gate="G$1" x="208.28" y="137.16" smashed="yes" rot="R270">
-<attribute name="NAME" x="207.01" y="135.6614" size="1.778" layer="95" rot="R180"/>
-<attribute name="VALUE" x="207.01" y="137.922" size="1.778" layer="96" rot="R180"/>
-</instance>
-<instance part="GND13" gate="1" x="210.82" y="124.46" smashed="yes">
-<attribute name="VALUE" x="208.28" y="121.92" size="1.778" layer="96"/>
+<instance part="X1" gate="G$1" x="200.66" y="156.21" smashed="yes" rot="R270">
+<attribute name="NAME" x="198.12" y="159.258" size="1.778" layer="95" font="vector"/>
+</instance>
+<instance part="X2" gate="G$1" x="215.9" y="156.21" smashed="yes" rot="R270">
+<attribute name="NAME" x="213.36" y="159.258" size="1.778" layer="95" font="vector"/>
+</instance>
+<instance part="GND12" gate="1" x="203.2" y="130.81" smashed="yes">
+<attribute name="VALUE" x="200.66" y="128.27" size="1.778" layer="96"/>
+</instance>
+<instance part="R2" gate="G$1" x="215.9" y="143.51" smashed="yes" rot="R270">
+<attribute name="NAME" x="214.63" y="142.0114" size="1.778" layer="95" rot="R180"/>
+<attribute name="VALUE" x="214.63" y="144.272" size="1.778" layer="96" rot="R180"/>
+</instance>
+<instance part="GND13" gate="1" x="218.44" y="130.81" smashed="yes">
+<attribute name="VALUE" x="215.9" y="128.27" size="1.778" layer="96"/>
 </instance>
 </instances>
@@
 <segment>
 <pinref part="X2" gate="G$1" pin="2"/>
-<wire x1="210.82" y1="142.24" x2="210.82" y2="127" width="0.1524" layer="91"/>
+<wire x1="218.44" y1="148.59" x2="218.44" y2="133.35" width="0.1524" layer="91"/>
 <pinref part="GND13" gate="1" pin="GND"/>
 </segment>
@@
 <segment>
 <pinref part="X1" gate="G$1" pin="1"/>
-<wire x1="193.04" y1="142.24" x2="193.04" y2="127" width="0.1524" layer="91"/>
-<label x="190.5" y="127" size="1.778" layer="95" rot="R90" align="top-left"/>
+<wire x1="200.66" y1="148.59" x2="200.66" y2="133.35" width="0.1524" layer="91"/>
+<label x="198.12" y="133.35" size="1.778" layer="95" rot="R90" align="top-left"/>
 </segment>
 <segment>
@@
 <segment>
 <pinref part="R2" gate="G$1" pin="2"/>
-<wire x1="208.28" y1="132.08" x2="208.28" y2="127" width="0.1524" layer="91"/>
-<label x="205.74" y="127" size="1.778" layer="95" rot="R90" align="top-left"/>
+<wire x1="215.9" y1="138.43" x2="215.9" y2="133.35" width="0.1524" layer="91"/>
+<label x="213.36" y="133.35" size="1.778" layer="95" rot="R90" align="top-left"/>
 </segment>
 <segment>
@@
 <segment>
 <pinref part="X1" gate="G$1" pin="2"/>
-<wire x1="195.58" y1="142.24" x2="195.58" y2="127" width="0.1524" layer="91"/>
+<wire x1="203.2" y1="148.59" x2="203.2" y2="133.35" width="0.1524" layer="91"/>
 <pinref part="GND12" gate="1" pin="GND"/>
 </segment>
@@
 <plain>
 <text x="217.17" y="20.32" size="2.54" layer="94">Ein/Ausgabe</text>
+<text x="109.22" y="156.21" size="3.81" layer="97">Heartbeat</text>
+<text x="165.1" y="134.62" size="3.81" layer="97">Speaker</text>
+<text x="208.28" y="135.89" size="3.81" layer="97">Switch</text>
+<text x="161.29" y="85.09" size="3.81" layer="97">LEDs</text>
 </plain>
 <instances>
@@
 <plain>
 <text x="217.17" y="20.32" size="2.54" layer="94">Anschlüsse</text>
+<text x="115.57" y="137.16" size="3.81" layer="97">I2C</text>
+<text x="66.04" y="115.57" size="3.81" layer="97">Analog</text>
+<text x="66.04" y="85.09" size="3.81" layer="97">Digital</text>
+<text x="123.19" y="88.9" size="3.81" layer="97">5V</text>
+<text x="121.92" y="58.42" size="3.81" layer="97">12V</text>
 </plain>
 <instances>

Commit message: ~ sch (mehr alte Teile ausgetauscht)
Other:
- note added: "Arduino"
- note added: "Sicherung"
Changed lines of the file:
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@@
 <parts>
 <part name="FRAME1" library="frames" library_urn="urn:adsk.eagle:library:229" deviceset="A4L-LOC" device=""/>
-<part name="F1" library="fuse" library_urn="urn:adsk.eagle:library:233" deviceset="FUSE" device="SH22,5" package3d_urn="urn:adsk.eagle:package:14059/1"/>
-<part name="LED2" library="led" library_urn="urn:adsk.eagle:library:259" deviceset="LED" device="CHIPLED_1206" package3d_urn="urn:adsk.eagle:package:15823/2"/>
-<part name="LED1" library="led" library_urn="urn:adsk.eagle:library:259" deviceset="LED" device="CHIPLED_1206" package3d_urn="urn:adsk.eagle:package:15823/2"/>
 <part name="GND89" library="supply1" library_urn="urn:adsk.eagle:library:371" deviceset="GND" device=""/>
-<part name="R1" library="iceberg20" deviceset="R" device="" package3d_urn="urn:adsk.eagle:package:23553/2" value="330R"/>
+<part name="LED1" library="iceberg20" deviceset="LED-GREEN1" device="" package3d_urn="urn:adsk.eagle:package:12172548/5"/>
+<part name="LED2" library="iceberg20" deviceset="LED-GREEN1" device="" package3d_urn="urn:adsk.eagle:package:12172548/5"/>
+<part name="R1" library="iceberg20" deviceset="R" device="" package3d_urn="urn:adsk.eagle:package:23553/2" value="270"/>
+<part name="F1" library="iceberg20" deviceset="SICHERUNGSHALTER" device="" package3d_urn="urn:adsk.eagle:package:14059/1"/>
 </parts>
 <sheets>
 <sheet>
 <plain>
+<text x="217.17" y="20.32" size="2.54" layer="94">Sicherung</text>
 </plain>
 <instances>
@@
 <attribute name="SHEET" x="230.505" y="5.08" size="2.54" layer="94"/>
 </instance>
-<instance part="F1" gate="G$1" x="119.38" y="88.9" smashed="yes" rot="MR0">
-<attribute name="NAME" x="123.19" y="90.297" size="1.016" layer="95" rot="MR0"/>
-</instance>
-<instance part="LED2" gate="G$1" x="129.54" y="60.96" smashed="yes">
-<attribute name="NAME" x="132.588" y="59.944" size="1.778" layer="95"/>
-<attribute name="VALUE" x="135.255" y="56.388" size="1.778" layer="96" rot="R90"/>
-</instance>
-<instance part="LED1" gate="G$1" x="129.54" y="71.12" smashed="yes">
-<attribute name="NAME" x="132.588" y="70.104" size="1.778" layer="95"/>
-<attribute name="VALUE" x="135.255" y="66.548" size="1.778" layer="96" rot="R90"/>
-</instance>
 <instance part="GND89" gate="1" x="129.54" y="50.8" smashed="yes">
 <attribute name="VALUE" x="127" y="48.26" size="1.778" layer="96"/>
 </instance>
-<instance part="R1" gate="G$1" x="129.54" y="81.28" smashed="yes" rot="MR90">
-<attribute name="NAME" x="132.08" y="82.3214" size="1.778" layer="95" rot="MR180"/>
-<attribute name="VALUE" x="132.08" y="79.502" size="1.778" layer="96" rot="MR180"/>
+<instance part="LED1" gate="G$1" x="129.54" y="71.12" smashed="yes">
+<attribute name="NAME" x="131.318" y="68.834" size="1.778" layer="95"/>
+</instance>
+<instance part="LED2" gate="G$1" x="129.54" y="60.96" smashed="yes">
+<attribute name="NAME" x="131.318" y="58.674" size="1.778" layer="95"/>
+</instance>
+<instance part="R1" gate="G$1" x="129.54" y="81.28" smashed="yes" rot="R90">
+<attribute name="NAME" x="130.81" y="81.5086" size="1.778" layer="95"/>
+<attribute name="VALUE" x="130.81" y="79.248" size="1.778" layer="96"/>
+</instance>
+<instance part="F1" gate="1" x="119.38" y="88.9" smashed="yes">
+<attribute name="NAME" x="115.57" y="90.297" size="1.778" layer="95"/>
+<attribute name="VALUE" x="115.57" y="85.979" size="1.778" layer="96"/>
 </instance>
 </instances>
@@
 <segment>
 <pinref part="GND89" gate="1" pin="GND"/>
+<wire x1="129.54" y1="53.34" x2="129.54" y2="55.88" width="0.1524" layer="91"/>
 <pinref part="LED2" gate="G$1" pin="C"/>
-<wire x1="129.54" y1="53.34" x2="129.54" y2="55.88" width="0.1524" layer="91"/>
 </segment>
 </net>
 <net name="OUT" class="0">
 <segment>
-<pinref part="F1" gate="G$1" pin="1"/>
-<pinref part="R1" gate="G$1" pin="2"/>
-<wire x1="129.54" y1="86.36" x2="129.54" y2="88.9" width="0.1524" layer="91"/>
 <wire x1="129.54" y1="88.9" x2="124.46" y2="88.9" width="0.1524" layer="91"/>
 <junction x="129.54" y="88.9"/>
 <wire x1="129.54" y1="88.9" x2="134.62" y2="88.9" width="0.1524" layer="91"/>
 <label x="134.62" y="88.9" size="1.778" layer="95" xref="yes"/>
+<pinref part="R1" gate="G$1" pin="2"/>
+<wire x1="129.54" y1="88.9" x2="129.54" y2="86.36" width="0.1524" layer="91"/>
+<pinref part="F1" gate="1" pin="2"/>
 </segment>
 </net>
 <net name="N$165" class="0">
 <segment>
+<wire x1="129.54" y1="63.5" x2="129.54" y2="66.04" width="0.1524" layer="91"/>
+<pinref part="LED1" gate="G$1" pin="C"/>
 <pinref part="LED2" gate="G$1" pin="A"/>
-<pinref part="LED1" gate="G$1" pin="C"/>
-<wire x1="129.54" y1="63.5" x2="129.54" y2="66.04" width="0.1524" layer="91"/>
-</segment>
-</net>
-<net name="N$166" class="0">
-<segment>
-<pinref part="LED1" gate="G$1" pin="A"/>
-<wire x1="129.54" y1="73.66" x2="129.54" y2="76.2" width="0.1524" layer="91"/>
-<pinref part="R1" gate="G$1" pin="1"/>
 </segment>
 </net>
 <net name="IN" class="0">
 <segment>
-<pinref part="F1" gate="G$1" pin="2"/>
 <wire x1="114.3" y1="88.9" x2="109.22" y2="88.9" width="0.1524" layer="91"/>
 <label x="109.22" y="88.9" size="1.778" layer="95" rot="R180" xref="yes"/>
+<pinref part="F1" gate="1" pin="1"/>
+</segment>
+</net>
+<net name="N$1" class="0">
+<segment>
+<pinref part="R1" gate="G$1" pin="1"/>
+<pinref part="LED1" gate="G$1" pin="A"/>
+<wire x1="129.54" y1="76.2" x2="129.54" y2="73.66" width="0.1524" layer="91"/>
 </segment>
 </net>
@@
 <sheet>
 <plain>
+<text x="344.17" y="20.32" size="2.54" layer="94">Arduino</text>
 </plain>
 <instances>

Commit message: + sch (Anschlüsse nach unten, NOT FINISHED)
Other:
- note added: "Anschlüsse nach unten"
