File: bottom20.sch (EAGLE design)
At the start: 0 parts

Commit message: + bot.sch (LED, Transistor)
Other:
- note added: "Led"
- note added: "Phototransistor"

Commit message: - bot.sch (LED, Transistor, Arduino, Anschluss)
Other:
- note added: "Anschluss"
- note added: "Arduino"

Commit message: + bot.sch (5V-Schaltregler)
Other:
- note added: "5V-Schaltregler"
