File: bottom20.sch (EAGLE design)
At the start: 0 parts

Commit message: - bot.sch (Übersicht)
Changed lines of the file:
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@@
 </sheets>
 </module>
-<module name="5V-SCHALTREGLER" prefix="" dx="35.56" dy="17.78">
+<module name="5V-SCHALTREGLER" prefix="" dx="38.1" dy="25.4">
 <ports>
 <port name="+12V" side="top" coord="2.54" direction="pwr"/>
@@
 <part name="P+3" library="supply1" library_urn="urn:adsk.eagle:library:371" deviceset="+5V" device=""/>
 <part name="GND3" library="supply1" library_urn="urn:adsk.eagle:library:371" deviceset="GND" device=""/>
+<part name="GND4" library="supply1" library_urn="urn:adsk.eagle:library:371" deviceset="GND" device=""/>
+<part name="P+8" library="supply1" library_urn="urn:adsk.eagle:library:371" deviceset="+5V" device=""/>
 </parts>
 <sheets>
@@
 </plain>
 <moduleinsts>
-<moduleinst name="5V-SCHALTREGLER1" module="5V-SCHALTREGLER" x="33.02" y="142.24">
-<attribute name="NAME" x="33.02" y="142.24" size="2.032" layer="95" align="bottom-center"/>
+<moduleinst name="5V-SCHALTREGLER1" module="5V-SCHALTREGLER" x="35.56" y="142.24">
+<attribute name="NAME" x="35.56" y="142.24" size="2.032" layer="95" align="bottom-center"/>
 </moduleinst>
 <moduleinst name="PHOTOTRANSISTOR1" module="PHOTOTRANSISTOR" x="223.52" y="101.6" rot="R180">
@@
 <attribute name="NAME" x="35.56" y="91.44" size="2.032" layer="95" align="bottom-center"/>
 </moduleinst>
-<moduleinst name="ANSCHLUSS1" module="ANSCHLUSS" x="50.8" y="38.1">
-<attribute name="NAME" x="50.8" y="38.1" size="2.032" layer="95" align="bottom-center"/>
+<moduleinst name="ANSCHLUSS1" module="ANSCHLUSS" x="40.64" y="40.64">
+<attribute name="NAME" x="40.64" y="40.64" size="2.032" layer="95" align="bottom-center"/>
 </moduleinst>
 <moduleinst name="PHOTOTRANSISTOR2" module="PHOTOTRANSISTOR" x="101.6" y="119.38">
@@
 <attribute name="SHEET" x="230.505" y="5.08" size="2.54" layer="94"/>
 </instance>
-<instance part="P+1" gate="1" x="35.56" y="162.56" smashed="yes">
-<attribute name="VALUE" x="33.02" y="157.48" size="1.778" layer="96" rot="R90"/>
-</instance>
-<instance part="P+2" gate="1" x="43.18" y="162.56" smashed="yes">
-<attribute name="VALUE" x="40.64" y="157.48" size="1.778" layer="96" rot="R90"/>
+<instance part="P+1" gate="1" x="38.1" y="165.1" smashed="yes">
+<attribute name="VALUE" x="35.56" y="160.02" size="1.778" layer="96" rot="R90"/>
+</instance>
+<instance part="P+2" gate="1" x="45.72" y="165.1" smashed="yes">
+<attribute name="VALUE" x="43.18" y="160.02" size="1.778" layer="96" rot="R90"/>
 </instance>
 <instance part="P+4" gate="1" x="210.82" y="86.36" smashed="yes">
@@
 <attribute name="VALUE" x="236.22" y="116.84" size="1.778" layer="96"/>
 </instance>
-<instance part="P+6" gate="1" x="50.8" y="63.5" smashed="yes">
-<attribute name="VALUE" x="48.26" y="58.42" size="1.778" layer="96" rot="R90"/>
-</instance>
-<instance part="GND6" gate="1" x="66.04" y="15.24" smashed="yes">
-<attribute name="VALUE" x="63.5" y="12.7" size="1.778" layer="96"/>
+<instance part="P+6" gate="1" x="40.64" y="66.04" smashed="yes">
+<attribute name="VALUE" x="38.1" y="60.96" size="1.778" layer="96" rot="R90"/>
+</instance>
+<instance part="GND6" gate="1" x="55.88" y="17.78" smashed="yes">
+<attribute name="VALUE" x="53.34" y="15.24" size="1.778" layer="96"/>
 </instance>
 <instance part="P+5" gate="1" x="109.22" y="142.24" smashed="yes">
@@
 <instance part="GND3" gate="1" x="165.1" y="76.2" smashed="yes">
 <attribute name="VALUE" x="162.56" y="73.66" size="1.778" layer="96"/>
+</instance>
+<instance part="GND4" gate="1" x="45.72" y="119.38" smashed="yes">
+<attribute name="VALUE" x="43.18" y="116.84" size="1.778" layer="96"/>
+</instance>
+<instance part="P+8" gate="1" x="73.66" y="40.64" smashed="yes">
+<attribute name="VALUE" x="71.12" y="35.56" size="1.778" layer="96" rot="R90"/>
 </instance>
 </instances>
@@
 <segment>
 <portref moduleinst="5V-SCHALTREGLER1" port="+12V"/>
-<wire x1="35.56" y1="156.21" x2="35.56" y2="160.02" width="0.1524" layer="91"/>
 <pinref part="P+1" gate="1" pin="+12V"/>
+<wire x1="38.1" y1="162.56" x2="38.1" y2="160.02" width="0.1524" layer="91"/>
 </segment>
 </net>
@@
 <segment>
 <portref moduleinst="5V-SCHALTREGLER1" port="+5V"/>
-<wire x1="43.18" y1="156.21" x2="43.18" y2="160.02" width="0.1524" layer="91"/>
 <pinref part="P+2" gate="1" pin="+5V"/>
+<wire x1="45.72" y1="162.56" x2="45.72" y2="160.02" width="0.1524" layer="91"/>
 </segment>
 <segment>
@@
 <pinref part="P+5" gate="1" pin="+5V"/>
 </segment>
+<segment>
+<portref moduleinst="ANSCHLUSS1" port="VID"/>
+<wire x1="66.04" y1="35.56" x2="73.66" y2="35.56" width="0.1524" layer="91"/>
+<wire x1="73.66" y1="35.56" x2="73.66" y2="38.1" width="0.1524" layer="91"/>
+<pinref part="P+8" gate="1" pin="+5V"/>
+</segment>
 </net>
 <net name="GND" class="0">
@@
 <segment>
 <portref moduleinst="ANSCHLUSS1" port="GND"/>
-<wire x1="66.04" y1="20.32" x2="66.04" y2="17.78" width="0.1524" layer="91"/>
+<wire x1="55.88" y1="22.86" x2="55.88" y2="20.32" width="0.1524" layer="91"/>
 <pinref part="GND6" gate="1" pin="GND"/>
 </segment>
@@
 <pinref part="GND3" gate="1" pin="GND"/>
 </segment>
+<segment>
+<portref moduleinst="5V-SCHALTREGLER1" port="GND"/>
+<wire x1="45.72" y1="124.46" x2="45.72" y2="121.92" width="0.1524" layer="91"/>
+<pinref part="GND4" gate="1" pin="GND"/>
+</segment>
 </net>
 <net name="LED-IN" class="0">
@@
 <segment>
 <portref moduleinst="ANSCHLUSS1" port="LED-IN"/>
-<wire x1="25.4" y1="45.72" x2="22.86" y2="45.72" width="0.1524" layer="91"/>
-<label x="22.86" y="45.72" size="1.778" layer="95" align="center-right"/>
+<wire x1="15.24" y1="48.26" x2="12.7" y2="48.26" width="0.1524" layer="91"/>
+<label x="12.7" y="48.26" size="1.778" layer="95" align="center-right"/>
 </segment>
 </net>
@@
 <segment>
 <portref moduleinst="ANSCHLUSS1" port="DTR"/>
-<wire x1="76.2" y1="45.72" x2="78.74" y2="45.72" width="0.1524" layer="91"/>
-<label x="78.74" y="45.72" size="1.778" layer="95"/>
+<wire x1="66.04" y1="48.26" x2="68.58" y2="48.26" width="0.1524" layer="91"/>
+<label x="68.58" y="48.26" size="1.778" layer="95"/>
 </segment>
 </net>
@@
 <segment>
 <portref moduleinst="ANSCHLUSS1" port="TX"/>
-<wire x1="76.2" y1="40.64" x2="78.74" y2="40.64" width="0.1524" layer="91"/>
-<label x="78.74" y="40.64" size="1.778" layer="95"/>
+<wire x1="66.04" y1="43.18" x2="68.58" y2="43.18" width="0.1524" layer="91"/>
+<label x="68.58" y="43.18" size="1.778" layer="95"/>
 </segment>
 </net>
@@
 <segment>
 <portref moduleinst="ANSCHLUSS1" port="RX"/>
-<wire x1="76.2" y1="43.18" x2="78.74" y2="43.18" width="0.1524" layer="91"/>
-<label x="78.74" y="43.18" size="1.778" layer="95"/>
+<wire x1="66.04" y1="45.72" x2="68.58" y2="45.72" width="0.1524" layer="91"/>
+<label x="68.58" y="45.72" size="1.778" layer="95"/>
 </segment>
 </net>
@@
 <segment>
 <portref moduleinst="ANSCHLUSS1" port="SCL"/>
-<wire x1="25.4" y1="43.18" x2="22.86" y2="43.18" width="0.1524" layer="91"/>
-<label x="22.86" y="43.18" size="1.778" layer="95" align="center-right"/>
+<wire x1="15.24" y1="45.72" x2="12.7" y2="45.72" width="0.1524" layer="91"/>
+<label x="12.7" y="45.72" size="1.778" layer="95" align="center-right"/>
 </segment>
 <segment>
@@
 <segment>
 <portref moduleinst="ANSCHLUSS1" port="SDA"/>
-<wire x1="25.4" y1="40.64" x2="22.86" y2="40.64" width="0.1524" layer="91"/>
-<label x="22.86" y="40.64" size="1.778" layer="95" align="center-right"/>
+<wire x1="15.24" y1="43.18" x2="12.7" y2="43.18" width="0.1524" layer="91"/>
+<label x="12.7" y="43.18" size="1.778" layer="95" align="center-right"/>
 </segment>
 <segment>
@@
 <segment>
 <portref moduleinst="ANSCHLUSS1" port="ARD-IN"/>
-<wire x1="25.4" y1="48.26" x2="22.86" y2="48.26" width="0.1524" layer="91"/>
-<label x="22.86" y="48.26" size="1.778" layer="95" align="center-right"/>
+<wire x1="15.24" y1="50.8" x2="12.7" y2="50.8" width="0.1524" layer="91"/>
+<label x="12.7" y="50.8" size="1.778" layer="95" align="center-right"/>
 </segment>
 <segment>
@@
 <segment>
 <portref moduleinst="ANSCHLUSS1" port="+12V"/>
-<wire x1="50.8" y1="55.88" x2="50.8" y2="60.96" width="0.1524" layer="91"/>
+<wire x1="40.64" y1="58.42" x2="40.64" y2="63.5" width="0.1524" layer="91"/>
 <pinref part="P+6" gate="1" pin="+12V"/>
 </segment>
@@
 <segment>
 <portref moduleinst="ANSCHLUSS1" port="CTS"/>
-<wire x1="76.2" y1="48.26" x2="78.74" y2="48.26" width="0.1524" layer="91"/>
-<label x="78.74" y="48.26" size="1.778" layer="95"/>
-</segment>
-</net>
+<wire x1="66.04" y1="50.8" x2="68.58" y2="50.8" width="0.1524" layer="91"/>
+<label x="68.58" y="50.8" size="1.778" layer="95"/>
+</segment>
+</net>

Commit message: + brd (layout)
Changed lines of the file:
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@@
 <port name="D5" side="top" coord="-2.54" direction="io"/>
 <port name="GND" side="left" coord="-7.62" direction="pwr"/>
-<port name="RX" side="bottom" coord="-17.78" direction="out"/>
+<port name="RX" side="bottom" coord="-17.78" direction="in"/>
 <port name="TX" side="bottom" coord="-15.24" direction="out"/>
 <port name="SCL" side="top" coord="-15.24" direction="io"/>
@@
 <port name="CTS" side="right" coord="10.16" direction="in"/>
 <port name="DTR" side="right" coord="7.62" direction="in"/>
-<port name="RX" side="right" coord="5.08" direction="in"/>
+<port name="RX" side="right" coord="5.08" direction="out"/>
 <port name="TX" side="right" coord="2.54" direction="in"/>
 <port name="VID" side="right" coord="-5.08" direction="pwr"/>
@@
 </segment>
 </net>
-<net name="TX" class="0">
+<net name="RX" class="0">
 <segment>
 <pinref part="X1" gate="G$1" pin="4"/>
 <wire x1="99.06" y1="104.14" x2="101.6" y2="104.14" width="0.1524" layer="91"/>
 <label x="101.6" y="104.14" size="1.778" layer="95" xref="yes"/>
-</segment>
-</net>
-<net name="RX" class="0">
-<segment>
-<pinref part="X1" gate="G$1" pin="5"/>
-<wire x1="99.06" y1="106.68" x2="109.22" y2="106.68" width="0.1524" layer="91"/>
-<label x="109.22" y="106.68" size="1.778" layer="95" xref="yes"/>
 </segment>
 </net>
@@
 <wire x1="99.06" y1="71.12" x2="101.6" y2="71.12" width="0.1524" layer="91"/>
 <label x="101.6" y="71.12" size="1.778" layer="95" xref="yes"/>
+</segment>
+</net>
+<net name="TX" class="0">
+<segment>
+<pinref part="X1" gate="G$1" pin="5"/>
+<wire x1="99.06" y1="106.68" x2="109.22" y2="106.68" width="0.1524" layer="91"/>
+<label x="109.22" y="106.68" size="1.778" layer="95" xref="yes"/>
 </segment>
 </net>
@@
 <net name="TX" class="0">
 <segment>
+<portref moduleinst="ANSCHLUSS1" port="TX"/>
+<wire x1="66.04" y1="43.18" x2="68.58" y2="43.18" width="0.1524" layer="91"/>
+<label x="68.58" y="43.18" size="1.778" layer="95"/>
+</segment>
+<segment>
+<portref moduleinst="ARDUINO1" port="TX"/>
+<wire x1="175.26" y1="96.52" x2="177.8" y2="96.52" width="0.1524" layer="91"/>
+<label x="177.8" y="96.52" size="1.778" layer="95" align="center-left"/>
+</segment>
+</net>
+<net name="RX" class="0">
+<segment>
+<portref moduleinst="ANSCHLUSS1" port="RX"/>
+<wire x1="66.04" y1="45.72" x2="68.58" y2="45.72" width="0.1524" layer="91"/>
+<label x="68.58" y="45.72" size="1.778" layer="95"/>
+</segment>
+<segment>
 <portref moduleinst="ARDUINO1" port="RX"/>
 <wire x1="175.26" y1="93.98" x2="177.8" y2="93.98" width="0.1524" layer="91"/>
 <label x="177.8" y="93.98" size="1.778" layer="95" align="center-left"/>
 </segment>
-<segment>
-<portref moduleinst="ANSCHLUSS1" port="TX"/>
-<wire x1="66.04" y1="43.18" x2="68.58" y2="43.18" width="0.1524" layer="91"/>
-<label x="68.58" y="43.18" size="1.778" layer="95"/>
-</segment>
-</net>
-<net name="RX" class="0">
-<segment>
-<portref moduleinst="ARDUINO1" port="TX"/>
-<wire x1="175.26" y1="96.52" x2="177.8" y2="96.52" width="0.1524" layer="91"/>
-<label x="177.8" y="96.52" size="1.778" layer="95" align="center-left"/>
-</segment>
-<segment>
-<portref moduleinst="ANSCHLUSS1" port="RX"/>
-<wire x1="66.04" y1="45.72" x2="68.58" y2="45.72" width="0.1524" layer="91"/>
-<label x="68.58" y="45.72" size="1.778" layer="95"/>
-</segment>
-</net>
+</net>

Commit message: Revert "Merge branch 'oona'"
This reverts commit 7885927933e734fa401e9be7113e93554c34953f.
Changed lines of the file:
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@@
 <port name="D5" side="top" coord="-2.54" direction="io"/>
 <port name="GND" side="left" coord="-7.62" direction="pwr"/>
-<port name="RX" side="bottom" coord="-17.78" direction="in"/>
+<port name="RX" side="bottom" coord="-17.78" direction="out"/>
 <port name="TX" side="bottom" coord="-15.24" direction="out"/>
 <port name="SCL" side="top" coord="-15.24" direction="io"/>
@@
 <port name="CTS" side="right" coord="10.16" direction="in"/>
 <port name="DTR" side="right" coord="7.62" direction="in"/>
-<port name="RX" side="right" coord="5.08" direction="out"/>
+<port name="RX" side="right" coord="5.08" direction="in"/>
 <port name="TX" side="right" coord="2.54" direction="in"/>
 <port name="VID" side="right" coord="-5.08" direction="pwr"/>
@@
 </segment>
 </net>
-<net name="RX" class="0">
+<net name="TX" class="0">
 <segment>
 <pinref part="X1" gate="G$1" pin="4"/>
 <wire x1="99.06" y1="104.14" x2="101.6" y2="104.14" width="0.1524" layer="91"/>
 <label x="101.6" y="104.14" size="1.778" layer="95" xref="yes"/>
+</segment>
+</net>
+<net name="RX" class="0">
+<segment>
+<pinref part="X1" gate="G$1" pin="5"/>
+<wire x1="99.06" y1="106.68" x2="109.22" y2="106.68" width="0.1524" layer="91"/>
+<label x="109.22" y="106.68" size="1.778" layer="95" xref="yes"/>
 </segment>
 </net>
@@
 <wire x1="99.06" y1="71.12" x2="101.6" y2="71.12" width="0.1524" layer="91"/>
 <label x="101.6" y="71.12" size="1.778" layer="95" xref="yes"/>
-</segment>
-</net>
-<net name="TX" class="0">
-<segment>
-<pinref part="X1" gate="G$1" pin="5"/>
-<wire x1="99.06" y1="106.68" x2="109.22" y2="106.68" width="0.1524" layer="91"/>
-<label x="109.22" y="106.68" size="1.778" layer="95" xref="yes"/>
 </segment>
 </net>
@@
 <net name="TX" class="0">
 <segment>
+<portref moduleinst="ARDUINO1" port="RX"/>
+<wire x1="175.26" y1="93.98" x2="177.8" y2="93.98" width="0.1524" layer="91"/>
+<label x="177.8" y="93.98" size="1.778" layer="95" align="center-left"/>
+</segment>
+<segment>
 <portref moduleinst="ANSCHLUSS1" port="TX"/>
 <wire x1="66.04" y1="43.18" x2="68.58" y2="43.18" width="0.1524" layer="91"/>
 <label x="68.58" y="43.18" size="1.778" layer="95"/>
 </segment>
+</net>
+<net name="RX" class="0">
 <segment>
 <portref moduleinst="ARDUINO1" port="TX"/>
@@
 <label x="177.8" y="96.52" size="1.778" layer="95" align="center-left"/>
 </segment>
-</net>
-<net name="RX" class="0">
 <segment>
 <portref moduleinst="ANSCHLUSS1" port="RX"/>
@@
 <label x="68.58" y="45.72" size="1.778" layer="95"/>
 </segment>
-<segment>
-<portref moduleinst="ARDUINO1" port="RX"/>
-<wire x1="175.26" y1="93.98" x2="177.8" y2="93.98" width="0.1524" layer="91"/>
-<label x="177.8" y="93.98" size="1.778" layer="95" align="center-left"/>
-</segment>
-</net>
+</net>

Commit message: - bot.sch (corrections)
Other:
- note added: "Schaltregler"
- note added: "Übersichtsschaltplan"
- note removed: "5V-Schaltregler"

Commit message: - bot.sch (corrections)
Parts:
- added J1: TX, iceberg20:JUMPER-JP-3
- added J2: RX, iceberg20:JUMPER-JP-3
Connections:
- new net ARD-RX: J2.3
- new net ARD-TX: J1.3
- new net N$14: J1.2
- new net N$15: J2.2
- new net RX: J2.1
- new net TX: J1.1

Commit message: - bot.sch (layout perfections)
Parts:
- removed J1: TX, iceberg20:JUMPER-JP-3
- removed J2: RX, iceberg20:JUMPER-JP-3
Connections:
- removed net ARD-RX: J2.3
- removed net ARD-TX: J1.3
- removed net N$14: J1.2
- removed net N$15: J2.2
- removed net RX: J2.1
- removed net TX: J1.1
Changed lines of the file:
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@@
 <part name="R3" library="iceberg20" deviceset="R" device="" package3d_urn="urn:adsk.eagle:package:23553/2" value="100k"/>
 <part name="P+2" library="supply1" library_urn="urn:adsk.eagle:library:371" deviceset="+5V" device=""/>
-<part name="S1" library="iceberg20" deviceset="SMD-BUTTON" device=""/>
-<part name="GND5" library="supply1" library_urn="urn:adsk.eagle:library:371" deviceset="GND" device=""/>
 <part name="LED1" library="iceberg20" deviceset="LED-GREEN1" device="" package3d_urn="urn:adsk.eagle:package:12172548/5"/>
 <part name="R1" library="iceberg20" deviceset="R" device="" package3d_urn="urn:adsk.eagle:package:23553/2" value="110"/>
@@
 <attribute name="VALUE" x="78.74" y="139.7" size="1.778" layer="96" rot="R90"/>
 </instance>
-<instance part="S1" gate="G$1" x="71.12" y="139.7" smashed="yes">
-<attribute name="NAME" x="70.485" y="140.97" size="1.778" layer="95" rot="R180"/>
-<attribute name="VALUE" x="70.485" y="143.51" size="1.778" layer="96" rot="R180"/>
-</instance>
-<instance part="GND5" gate="1" x="73.66" y="152.4" smashed="yes" rot="R180">
-<attribute name="VALUE" x="76.2" y="154.94" size="1.778" layer="96" rot="R180"/>
-</instance>
 <instance part="LED1" gate="G$1" x="213.36" y="86.36" smashed="yes" rot="R90">
 <attribute name="NAME" x="217.932" y="89.916" size="1.778" layer="95" rot="R180"/>
@@
 <wire x1="99.06" y1="127" x2="91.44" y2="127" width="0.1524" layer="91"/>
 <wire x1="91.44" y1="127" x2="81.28" y2="127" width="0.1524" layer="91"/>
-<wire x1="81.28" y1="127" x2="73.66" y2="127" width="0.1524" layer="91"/>
-<wire x1="73.66" y1="127" x2="69.85" y2="127" width="0.1524" layer="91"/>
-<junction x="73.66" y="127"/>
+<wire x1="81.28" y1="127" x2="69.85" y2="127" width="0.1524" layer="91"/>
 <wire x1="81.28" y1="127" x2="81.28" y2="129.54" width="0.1524" layer="91"/>
 <junction x="81.28" y="127"/>
 <pinref part="R3" gate="G$1" pin="1"/>
-<pinref part="S1" gate="G$1" pin="P"/>
-<wire x1="73.66" y1="127" x2="73.66" y2="134.62" width="0.1524" layer="91"/>
 <wire x1="91.44" y1="127" x2="91.44" y2="142.24" width="0.1524" layer="91"/>
 <junction x="91.44" y="127"/>
@@
 <junction x="81.28" y="96.52"/>
 <pinref part="GND4" gate="1" pin="GND"/>
-</segment>
-<segment>
-<pinref part="S1" gate="G$1" pin="S"/>
-<wire x1="73.66" y1="144.78" x2="73.66" y2="149.86" width="0.1524" layer="91"/>
-<pinref part="GND5" gate="1" pin="GND"/>
 </segment>
 <segment>
@@
 <part name="P+5" library="supply1" library_urn="urn:adsk.eagle:library:371" deviceset="+5V" device=""/>
 <part name="P+8" library="supply1" library_urn="urn:adsk.eagle:library:371" deviceset="+5V" device=""/>
-<part name="J1" library="iceberg20" deviceset="JUMPER-JP-3" device="" value="TX"/>
-<part name="J2" library="iceberg20" deviceset="JUMPER-JP-3" device="" value="RX"/>
 </parts>
 <sheets>
@@
 <attribute name="VALUE" x="160.02" y="147.32" size="1.778" layer="96" rot="R90"/>
 </instance>
-<instance part="J1" gate="G$1" x="210.82" y="101.6" smashed="yes" rot="R270">
-<attribute name="NAME" x="210.82" y="105.41" size="1.778" layer="95"/>
-<attribute name="VALUE" x="210.82" y="95.885" size="1.778" layer="96"/>
-</instance>
-<instance part="J2" gate="G$1" x="210.82" y="88.9" smashed="yes" rot="R270">
-<attribute name="NAME" x="210.82" y="92.71" size="1.778" layer="95"/>
-<attribute name="VALUE" x="210.82" y="83.185" size="1.778" layer="96"/>
-</instance>
 </instances>
 <busses>
@@
 </segment>
 <segment>
-<pinref part="J1" gate="G$1" pin="1"/>
-<wire x1="208.28" y1="104.14" x2="205.74" y2="104.14" width="0.1524" layer="91"/>
-<label x="205.74" y="104.14" size="1.778" layer="95" rot="R180" align="center-left"/>
+<wire x1="60.96" y1="40.64" x2="58.42" y2="40.64" width="0.1524" layer="91"/>
+<label x="58.42" y="40.64" size="1.778" layer="95" rot="R180" align="center-left"/>
+</segment>
+<segment>
+<portref moduleinst="A" port="TX"/>
+<wire x1="180.34" y1="101.6" x2="182.88" y2="101.6" width="0.1524" layer="91"/>
+<label x="182.88" y="101.6" size="1.778" layer="95" align="center-left"/>
 </segment>
 </net>
@@
 </segment>
 <segment>
-<pinref part="J2" gate="G$1" pin="1"/>
-<wire x1="208.28" y1="91.44" x2="205.74" y2="91.44" width="0.1524" layer="91"/>
-<label x="205.74" y="91.44" size="1.778" layer="95" rot="R180" align="center-left"/>
+<wire x1="60.96" y1="43.18" x2="58.42" y2="43.18" width="0.1524" layer="91"/>
+<label x="58.42" y="43.18" size="1.778" layer="95" rot="R180" align="center-left"/>
+</segment>
+<segment>
+<portref moduleinst="A" port="RX"/>
+<wire x1="180.34" y1="99.06" x2="182.88" y2="99.06" width="0.1524" layer="91"/>
+<label x="182.88" y="99.06" size="1.778" layer="95" align="center-left"/>
 </segment>
 </net>
@@
 </segment>
 </net>
-<net name="ARD-RX" class="0">
-<segment>
-<wire x1="60.96" y1="43.18" x2="58.42" y2="43.18" width="0.1524" layer="91"/>
-<label x="58.42" y="43.18" size="1.778" layer="95" rot="R180" align="center-left"/>
-</segment>
-<segment>
-<pinref part="J2" gate="G$1" pin="3"/>
-<wire x1="208.28" y1="86.36" x2="205.74" y2="86.36" width="0.1524" layer="91"/>
-<label x="205.74" y="86.36" size="1.778" layer="95" rot="R180" align="center-left"/>
-</segment>
-</net>
-<net name="ARD-TX" class="0">
-<segment>
-<wire x1="60.96" y1="40.64" x2="58.42" y2="40.64" width="0.1524" layer="91"/>
-<label x="58.42" y="40.64" size="1.778" layer="95" rot="R180" align="center-left"/>
-</segment>
-<segment>
-<pinref part="J1" gate="G$1" pin="3"/>
-<wire x1="208.28" y1="99.06" x2="205.74" y2="99.06" width="0.1524" layer="91"/>
-<label x="205.74" y="99.06" size="1.778" layer="95" rot="R180" align="center-left"/>
-</segment>
-</net>
-<net name="N$14" class="0">
-<segment>
-<portref moduleinst="A" port="TX"/>
-<wire x1="180.34" y1="101.6" x2="208.28" y2="101.6" width="0.1524" layer="91"/>
-<pinref part="J1" gate="G$1" pin="2"/>
-</segment>
-</net>
-<net name="N$15" class="0">
-<segment>
-<portref moduleinst="A" port="RX"/>
-<wire x1="180.34" y1="99.06" x2="182.88" y2="99.06" width="0.1524" layer="91"/>
-<wire x1="182.88" y1="99.06" x2="182.88" y2="88.9" width="0.1524" layer="91"/>
-<wire x1="182.88" y1="88.9" x2="208.28" y2="88.9" width="0.1524" layer="91"/>
-<pinref part="J2" gate="G$1" pin="2"/>
-</segment>
-</net>
