File: bottom20.brd (EAGLE design)
At the start: 160 x 140 mm, 141 parts

Commit message: Revert "Merge branch 'oona'"
This reverts commit 7885927933e734fa401e9be7113e93554c34953f.
Parts:
- moved PHOTOTRANSISTOR2:T9 1513.2 mm to (-1361.4, -680.7)
- moved PHOTOTRANSISTOR2:T8 1493.8 mm to (-1355.1, -680.7), turned to 0 degrees
- moved PHOTOTRANSISTOR2:T7 1490.6 mm to (-1348.7, -680.7), turned to 0 degrees
- moved PHOTOTRANSISTOR2:T6 1487.5 mm to (-1342.4, -680.7), turned to 0 degrees
- moved PHOTOTRANSISTOR2:T5 1484.3 mm to (-1336.0, -680.7), turned to 0 degrees
- moved PHOTOTRANSISTOR2:T4 1481.3 mm to (-1329.7, -680.7), turned to 0 degrees
- moved PHOTOTRANSISTOR2:T3 1478.2 mm to (-1323.3, -680.7), turned to 0 degrees
- moved PHOTOTRANSISTOR2:T2 1475.2 mm to (-1317.0, -680.7), turned to 0 degrees
- moved PHOTOTRANSISTOR2:T1 1432.9 mm to (-1266.2, -680.7), turned to 0 degrees
- moved PHOTOTRANSISTOR2:T16 1430.9 mm to (-1310.6, -680.7)
- moved PHOTOTRANSISTOR2:T15 1430.6 mm to (-1304.3, -680.7)
- moved PHOTOTRANSISTOR2:T14 1430.3 mm to (-1297.9, -680.7)
- moved PHOTOTRANSISTOR2:T13 1430.0 mm to (-1291.6, -680.7)
- moved PHOTOTRANSISTOR2:T12 1429.7 mm to (-1285.2, -680.7)
- moved PHOTOTRANSISTOR2:T11 1429.4 mm to (-1278.9, -680.7)
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Connections:
- net RX: now also ANSCHLUSS1:X1.P$5, ARDUINO1:R2.2; no longer ANSCHLUSS1:X1.P$4, ARDUINO1:R1.2
- net TX: now also ANSCHLUSS1:X1.P$4, ARDUINO1:R1.2; no longer ANSCHLUSS1:X1.P$5, ARDUINO1:R2.2
Other:
- board size 160 x 140 mm -> 160 x 100 mm
