File: bottom20.brd (EAGLE design)
At the start: 160 x 140 mm, 142 parts, among them T1:IC1 MULTIPLEXER, T1:R1 20k, T1:R10 20k, T1:R11 20k, T1:R12 20k, T1:R13 20k, T1:R14 20k, T1:R15 20k, T1:R16 20k, T1:R17 10k, T1:R2 20k, T1:R3 20k, T1:R4 20k, T1:R5 20k, T1:R6 20k, T1:R7 20k, T1:R8 20k, T1:R9 20k, T1:T1 SFH320, T1:T10 SFH320, T1:T11 SFH320, T1:T12 SFH320, T1:T13 SFH320, T1:T14 SFH320, T1:T15 SFH320, T1:T16 SFH320, T1:T2 SFH320, T1:T3 SFH320, T1:T4 SFH320, T1:T5 SFH320, T1:T6 SFH320, T1:T7 SFH320, T1:T8 SFH320, T1:T9 SFH320, T2:IC1 MULTIPLEXER, T2:R1 20k, T2:R10 20k, T2:R11 20k, T2:R12 20k, T2:R13 20k, T2:R14 20k, T2:R15 20k, T2:R16 20k, T2:R17 10k, T2:R2 20k, T2:R3 20k, T2:R4 20k, T2:R5 20k, T2:R6 20k, T2:R7 20k, T2:R8 20k, T2:R9 20k, T2:T1 SFH320, T2:T10 SFH320, T2:T11 SFH320, T2:T12 SFH320, T2:T13 SFH320, T2:T14 SFH320, T2:T15 SFH320, T2:T16 SFH320, T2:T2 SFH320, T2:T3 SFH320, T2:T4 SFH320, T2:T5 SFH320, T2:T6 SFH320, T2:T7 SFH320, T2:T8 SFH320, T2:T9 SFH320

Commit message: - bot.brd (Routing - big progress)
Parts:
- moved A:LED2 40.1 mm to (57.3, -50.7), flipped to the bottom, turned to 270 degrees
- moved A:LED1 39.1 mm to (53.7, -53.9), flipped to the bottom, turned to 90 degrees
- moved A:S2 38.8 mm to (40.9, -61.4)
- moved P:X3 37.9 mm to (-16.2, -63.0), turned to 90 degrees
- moved A:R1 26.9 mm to (42.8, -52.2), turned to 270 degrees
- moved A:R2 20.3 mm to (53.6, -48.2), turned to 270 degrees
- moved A:C2 13.6 mm to (66.4, -37.0)
- moved A:C4 13.5 mm to (66.3, -39.9)
- moved A:C3 13.4 mm to (66.5, -43.9)
- moved L:C10 12.6 mm to (6.00, -17.3), turned to 0 degrees
- moved A:TP4 12.0 mm to (46.0, -54.0), flipped to the bottom
- moved X:D1 11.8 mm to (23.9, -61.2)
- moved L:LED25 10.8 mm to (-22.8, 7.50)
- moved L:LED9 10.8 mm to (22.8, -7.50)
- moved L:C14 9.58 mm to (-17.3, 9.00), turned to 270 degrees
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Connections:
- net A:N$5 renamed A:MOSI
- net A:N$6 renamed A:MISO
- net A:N$7 renamed A:SCK
- net ARD-INTERRUPT renamed A:ARD-INTERRUPT
- removed net X:+12V: X:X2.2, X:X2.5
- net +12V: now also X:X2.2, X:X2.5
Routing:
- net +5V: track 250.3 -> 824.3 mm, vias 17 -> 0
- net N$13: track 0.00 -> 104.8 mm, vias 0 -> 4
- net N$7: track 0.00 -> 97.7 mm, vias 0 -> 4
- net N$6: track 0.00 -> 97.1 mm, vias 0 -> 4
- net N$10: track 0.00 -> 94.3 mm, vias 0 -> 2
- net L:CON-3: track 0.00 -> 93.7 mm
- net N$5: track 0.00 -> 91.0 mm, vias 0 -> 2
- net X:ARD-INTERRUPT: track 0.00 -> 91.0 mm, vias 0 -> 2
- net N$11: track 0.00 -> 90.4 mm, vias 0 -> 4
- net N$12: track 12.1 -> 99.1 mm, vias 0 -> 2
- net L:CON-2: track 0.00 -> 86.9 mm, vias 0 -> 2
- net N$3: track 4.44 -> 89.6 mm, vias 0 -> 2
- net N$9: track 0.00 -> 84.0 mm, vias 0 -> 4
- net N$8: track 0.00 -> 83.4 mm, vias 0 -> 2
- net N$4: track 0.00 -> 79.1 mm, vias 0 -> 2
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