File: iceberg20.brd (EAGLE design)
At the start: 160 x 100 mm, 88 parts, among them M0:+ TPB1,27, M0:- TPB1,27, M0:C1 10nF, M0:C2 220nF, M0:C3 100nF, M0:C4 100uF, M0:C5 1nF, M0:C6 100nF, M0:D1 1N4148W, M0:D2 1N4148W, M0:EN TPB1,27, M0:I TPB1,27, M0:IC1 L6205N, M0:IC2 ACS712, M0:IN1 TPB1,27, M0:IN2 TPB1,27, M0:R1 100R, M0:R2 100k, M0:R3 10k, M0:VS TPB1,27, M1:+ TPB1,27, M1:- TPB1,27, M1:C1 10nF, M1:C2 220nF, M1:C3 100nF, M1:C4 100uF, M1:C5 1nF, M1:C6 100nF, M1:D1 1N4148W, M1:D2 1N4148W, M1:EN TPB1,27, M1:I TPB1,27, M1:IC1 L6205N, M1:IC2 ACS712, M1:IN1 TPB1,27, M1:IN2 TPB1,27, M1:R1 100R, M1:R2 100k, M1:R3 10k, M1:VS TPB1,27, M2:+ TPB1,27, M2:- TPB1,27, M2:C1 10nF, M2:C2 220nF, M2:C3 100nF, M2:C4 100uF, M2:C5 1nF, M2:C6 100nF, M2:D1 1N4148W, M2:D2 1N4148W, M2:EN TPB1,27, M2:I TPB1,27, M2:IC1 L6205N, M2:IC2 ACS712, M2:IN1 TPB1,27, M2:IN2 TPB1,27, M2:R1 100R, M2:R2 100k, M2:R3 10k, M2:VS TPB1,27, M3:+ TPB1,27, M3:- TPB1,27, M3:C1 10nF, M3:C2 220nF, M3:C3 100nF, M3:C4 100uF, M3:C5 1nF, M3:C6 100nF, M3:D1 1N4148W, M3:D2 1N4148W, M3:EN TPB1,27, M3:I TPB1,27, M3:IC1 L6205N, M3:IC2 ACS712, M3:IN1 TPB1,27, M3:IN2 TPB1,27, M3:R1 100R, M3:R2 100k, M3:R3 10k, M3:VS TPB1,27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

Commit message: ~ sch (Motor: alte Bauteile mit neuen ausgetauscht)
Parts:
- M0:C1, M0:C2, M0:C3, M0:C5, M0:C6, M1:C1, M1:C2, M1:C3, M1:C5, M1:C6, M2:C1, M2:C2, M2:C3, M2:C5, M2:C6, M3:C1, M3:C2, M3:C3, M3:C5, M3:C6: device eagle-ltspice:C1206 -> iceberg20:C0805
- M0:C4, M1:C4, M2:C4, M3:C4: value 100uF -> 100uF, 16V, ±20 %; device rcl:E2,5-6 -> iceberg20:CAPACITOR-THT-6.3
- M0:D1, M0:D2, M1:D1, M1:D2, M2:D1, M2:D2, M3:D1, M3:D2: value 1N4148W -> DIODE; device iceberg20:SOD123 -> iceberg20:DO-214BA
- M0:IC1, M1:IC1, M2:IC1, M3:IC1: device Lib:DIL20 -> iceberg20:DIL20
- M0:IC2, M1:IC2, M2:IC2, M3:IC2: value ACS712 -> ACS712ACS712-SOIC-8; device Lib:SOIC127P600X175-8 -> iceberg20:SOIC-8
- moved M3:IC2 368.7 mm to (-204.5, -228.6)
- moved M3:IC1 354.7 mm to (-146.1, -228.6)
- moved M2:IC2 341.4 mm to (-191.8, -228.6)
- moved M3:R1 326.0 mm to (-158.8, -185.4)
- moved M2:IC1 321.4 mm to (-146.1, -217.2)
- moved M1:IC2 314.2 mm to (-179.1, -228.6)
- moved M3:R2 300.7 mm to (-158.8, -160.0)
- moved M2:R1 298.2 mm to (-158.8, -179.1)
- moved M1:IC1 288.7 mm to (-146.1, -205.7)
- moved M0:IC2 286.9 mm to (-166.4, -228.6)
- moved M3:R3 275.5 mm to (-158.8, -134.6)
- moved M2:R2 273.2 mm to (-158.8, -153.7)
- moved M1:R1 271.0 mm to (-158.8, -172.7)
- moved M0:IC1 256.8 mm to (-146.1, -194.3)
- moved M2:R3 248.3 mm to (-158.8, -128.3)
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Connections:
- new net M0:N$1: M0:IC1.13
- new net M0:N$2: M0:IC1.7
- new net M1:N$1: M1:IC1.13
- new net M1:N$2: M1:IC1.7
- new net M2:N$1: M2:IC1.13
- new net M2:N$2: M2:IC1.7
- new net M3:N$1: M3:IC1.13
- new net M3:N$2: M3:IC1.7
- net M0:+5V: now also M0:C6.1; no longer M0:C6.2
- net M0:FILTER: now also M0:C5.1; no longer M0:C5.2
- net M0:GND: now also M0:C4.2, M0:C5.2, M0:C6.2; no longer M0:C4.-, M0:C5.1, M0:C6.1
- net M0:M+OUT: no longer M0:IC1.7
- net M0:M-: no longer M0:IC1.13
- net M0:N$4: now also M0:D1.2, M0:D2.1; no longer M0:D1.C, M0:D2.A
- net M0:N$6: now also M0:D1.1; no longer M0:D2.C
- net M1:+5V: now also M1:C6.1; no longer M1:C6.2
- net M1:FILTER: now also M1:C5.1; no longer M1:C5.2
- net M1:GND: now also M1:C4.2, M1:C5.2, M1:C6.2; no longer M1:C4.-, M1:C5.1, M1:C6.1
- net M1:M+OUT: no longer M1:IC1.7
- net M1:M-: no longer M1:IC1.13
- net M1:N$4: now also M1:D1.2, M1:D2.1; no longer M1:D1.C, M1:D2.A
- net M1:N$6: now also M1:D1.1; no longer M1:D2.C
- net M2:+5V: now also M2:C6.1; no longer M2:C6.2
- net M2:FILTER: now also M2:C5.1; no longer M2:C5.2
- net M2:GND: now also M2:C4.2, M2:C5.2, M2:C6.2; no longer M2:C4.-, M2:C5.1, M2:C6.1
- net M2:M+OUT: no longer M2:IC1.7
- net M2:M-: no longer M2:IC1.13
- net M2:N$4: now also M2:D1.2, M2:D2.1; no longer M2:D1.C, M2:D2.A
- net M2:N$6: now also M2:D1.1; no longer M2:D2.C
- net M3:+5V: now also M3:C6.1; no longer M3:C6.2
- net M3:FILTER: now also M3:C5.1; no longer M3:C5.2
- net M3:GND: now also M3:C4.2, M3:C5.2, M3:C6.2; no longer M3:C4.-, M3:C5.1, M3:C6.1
- net M3:M+OUT: no longer M3:IC1.7
- net M3:M-: no longer M3:IC1.13
- net M3:N$4: now also M3:D1.2, M3:D2.1; no longer M3:D1.C, M3:D2.A
- net M3:N$6: now also M3:D1.1; no longer M3:D2.C
- net MOTOR-SUPPLY: now also M0:C4.1, M0:D2.2, M1:C4.1, M1:D2.2, M2:C4.1, M2:D2.2, M3:C4.1, M3:D2.2; no longer M0:C4.+, M0:D1.A, M1:C4.+, M1:D1.A, M2:C4.+, M2:D1.A, M3:C4.+, M3:D1.A

Commit message: ~ sch (mehr alte Teile ausgetauscht)
Parts:
- F1:F1: value FUSESH22,5 -> (none); device fuse:SH22,5 -> iceberg20:SH22,5
- F1:LED1, F1:LED2: value (none) -> LED-GREEN1; device led:CHIPLED_1206 -> iceberg20:1206
- F1:R1: value 330R -> 270
- moved F1:F1 416.9 mm to (-210.8, -245.1)
- moved F1:R1 400.1 mm to (-222.2, -237.5)
- moved F1:LED2 395.9 mm to (-222.2, -229.9)
- moved F1:LED1 395.4 mm to (-215.9, -229.9)
Connections:
- net F1:N$166 renamed F1:N$1
- net F1:IN: now also F1:F1.1; no longer F1:F1.2
- net MOTOR-SUPPLY: now also F1:F1.2; no longer F1:F1.1
Changed lines of the file:
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@@
 </autorouter>
 <elements>
-<element name="F1:F1" library="fuse" library_urn="urn:adsk.eagle:library:233" package="SH22,5" package3d_urn="urn:adsk.eagle:package:14059/1" value="FUSESH22,5" x="-30.48" y="130.81" smashed="yes">
-<attribute name="MF" value="" x="-30.48" y="130.81" size="1.778" layer="27" display="off"/>
-<attribute name="MPN" value="" x="-30.48" y="130.81" size="1.778" layer="27" display="off"/>
-<attribute name="NAME" x="-30.48" y="130.81" size="1.778" layer="25" ratio="10"/>
-<attribute name="OC_FARNELL" value="unknown" x="-30.48" y="130.81" size="1.778" layer="27" display="off"/>
-<attribute name="OC_NEWARK" value="unknown" x="-30.48" y="130.81" size="1.778" layer="27" display="off"/>
-<attribute name="VALUE" x="-30.48" y="130.81" size="1.778" layer="27" ratio="10"/>
-</element>
-<element name="F1:LED1" library="led" library_urn="urn:adsk.eagle:library:259" package="CHIPLED_1206" package3d_urn="urn:adsk.eagle:package:15823/2" value="" x="-45.72" y="127" smashed="yes">
-<attribute name="NAME" x="-45.72" y="127" size="1.27" layer="25" rot="R90"/>
-<attribute name="VALUE" x="-45.72" y="127" size="1.27" layer="27" rot="R90"/>
-</element>
-<element name="F1:LED2" library="led" library_urn="urn:adsk.eagle:library:259" package="CHIPLED_1206" package3d_urn="urn:adsk.eagle:package:15823/2" value="" x="-50.8" y="127" smashed="yes">
-<attribute name="NAME" x="-50.8" y="127" size="1.27" layer="25" rot="R90"/>
-<attribute name="VALUE" x="-50.8" y="127" size="1.27" layer="27" rot="R90"/>
-</element>
-<element name="F1:R1" library="iceberg20" package="R0805" package3d_urn="urn:adsk.eagle:package:23553/2" value="330R" x="-57.15" y="127" smashed="yes">
-<attribute name="BESTAND" value="-" x="-57.15" y="127" size="1.778" layer="27" display="off"/>
-<attribute name="HERSTELLER" value="-" x="-57.15" y="127" size="1.778" layer="27" display="off"/>
-<attribute name="HERSTELLER-NR" value="-" x="-57.15" y="127" size="1.778" layer="27" display="off"/>
-<attribute name="NAME" x="-57.15" y="127" size="1" layer="25" font="vector" ratio="20"/>
-<attribute name="SUPPLIER" value="-" x="-57.15" y="127" size="1.778" layer="27" display="off"/>
-<attribute name="SUPPLIER-NR" value="-" x="-57.15" y="127" size="1.778" layer="27" display="off"/>
-<attribute name="TOLERANZ" value="5%" x="-57.15" y="127" size="1.778" layer="27" display="off"/>
-<attribute name="VALUE" x="-57.15" y="127" size="1" layer="27" font="vector" ratio="20"/>
-</element>
 <element name="M0:+" library="testpad" library_urn="urn:adsk.eagle:library:385" package="B1,27" package3d_urn="urn:adsk.eagle:package:27944/2" value="TPB1,27" x="-24.13" y="46.99" smashed="yes">
 <attribute name="NAME" x="-24.13" y="46.99" size="1.27" layer="25" ratio="10"/>
@@
 <attribute name="VALUE" x="-204.47" y="-231.7536" size="1" layer="27" font="vector" ratio="20" align="top-center"/>
 </element>
+<element name="F1:LED1" library="iceberg20" package="1206" package3d_urn="urn:adsk.eagle:package:12172548/5" value="LED-GREEN1" x="-215.9" y="-229.87" smashed="yes">
+<attribute name="BESTAND" value="" x="-215.9" y="-229.87" size="1.778" layer="27" display="off"/>
+<attribute name="HERSTELLER" value="EVERLIGHT" x="-215.9" y="-229.87" size="1.778" layer="27" display="off"/>
+<attribute name="HERSTELLER-NR" value="15-21SYGC/S530-E1/TR8 Everlight" x="-215.9" y="-229.87" size="1.778" layer="27" display="off"/>
+<attribute name="NAME" x="-218.44" y="-228.346" size="1" layer="25" font="vector" ratio="20"/>
+<attribute name="SUPPLIER" value="Bürklin" x="-215.9" y="-229.87" size="1.778" layer="27" display="off"/>
+<attribute name="SUPPLIER-NR" value="67S2004" x="-215.9" y="-229.87" size="1.778" layer="27" display="off"/>
+<attribute name="VALUE" x="-218.44" y="-232.41" size="1" layer="27" font="vector" ratio="20"/>
+</element>
+<element name="F1:LED2" library="iceberg20" package="1206" package3d_urn="urn:adsk.eagle:package:12172548/5" value="LED-GREEN1" x="-222.25" y="-229.87" smashed="yes">
+<attribute name="BESTAND" value="" x="-222.25" y="-229.87" size="1.778" layer="27" display="off"/>
+<attribute name="HERSTELLER" value="EVERLIGHT" x="-222.25" y="-229.87" size="1.778" layer="27" display="off"/>
+<attribute name="HERSTELLER-NR" value="15-21SYGC/S530-E1/TR8 Everlight" x="-222.25" y="-229.87" size="1.778" layer="27" display="off"/>
+<attribute name="NAME" x="-224.79" y="-228.346" size="1" layer="25" font="vector" ratio="20"/>
+<attribute name="SUPPLIER" value="Bürklin" x="-222.25" y="-229.87" size="1.778" layer="27" display="off"/>
+<attribute name="SUPPLIER-NR" value="67S2004" x="-222.25" y="-229.87" size="1.778" layer="27" display="off"/>
+<attribute name="VALUE" x="-224.79" y="-232.41" size="1" layer="27" font="vector" ratio="20"/>
+</element>
+<element name="F1:R1" library="iceberg20" package="R0805" package3d_urn="urn:adsk.eagle:package:23553/2" value="270" x="-222.25" y="-237.49" smashed="yes">
+<attribute name="BESTAND" value="-" x="-222.25" y="-237.49" size="1.778" layer="27" display="off"/>
+<attribute name="HERSTELLER" value="-" x="-222.25" y="-237.49" size="1.778" layer="27" display="off"/>
+<attribute name="HERSTELLER-NR" value="-" x="-222.25" y="-237.49" size="1.778" layer="27" display="off"/>
+<attribute name="NAME" x="-224.155" y="-236.22" size="1" layer="25" font="vector" ratio="20"/>
+<attribute name="SUPPLIER" value="-" x="-222.25" y="-237.49" size="1.778" layer="27" display="off"/>
+<attribute name="SUPPLIER-NR" value="-" x="-222.25" y="-237.49" size="1.778" layer="27" display="off"/>
+<attribute name="TOLERANZ" value="5%" x="-222.25" y="-237.49" size="1.778" layer="27" display="off"/>
+<attribute name="VALUE" x="-224.155" y="-240.03" size="1" layer="27" font="vector" ratio="20"/>
+</element>
+<element name="F1:F1" library="iceberg20" package="SH22,5" package3d_urn="urn:adsk.eagle:package:14059/1" value="" x="-210.82" y="-245.11" smashed="yes">
+<attribute name="BESTAND" value="?" x="-210.82" y="-245.11" size="1.778" layer="27" display="off"/>
+<attribute name="HERSTELLER" value="SCHURTER" x="-210.82" y="-245.11" size="1.778" layer="27" display="off"/>
+<attribute name="HERSTELLER-NR" value="0031.8201" x="-210.82" y="-245.11" size="1.778" layer="27" display="off"/>
+<attribute name="NAME" x="-223.52" y="-251.206" size="1.778" layer="25" ratio="10"/>
+<attribute name="SUPPLIER" value="Bürklin" x="-210.82" y="-245.11" size="1.778" layer="27" display="off"/>
+<attribute name="SUPPLIER-NR" value="46G6020" x="-210.82" y="-245.11" size="1.778" layer="27" display="off"/>
+<attribute name="VALUE" x="-209.677" y="-251.206" size="1.778" layer="27" ratio="10"/>
+</element>
 </elements>
 <signals>
@@
 <contactref element="M2:VS" pad="TP"/>
 <contactref element="M3:VS" pad="TP"/>
-<contactref element="F1:F1" pad="1"/>
-<contactref element="F1:R1" pad="2"/>
 <contactref element="M0:C3" pad="1"/>
 <contactref element="M1:C3" pad="1"/>
@@
 <contactref element="M2:IC1" pad="14"/>
 <contactref element="M3:IC1" pad="14"/>
+<contactref element="F1:R1" pad="2"/>
+<contactref element="F1:F1" pad="2"/>
 <wire x1="-155.1637" y1="-71.12" x2="-155.1637" y2="-78.74" width="0" layer="19" extent="1-1"/>
 <wire x1="-155.1637" y1="-63.5" x2="-155.1637" y2="-71.12" width="0" layer="19" extent="1-1"/>
@@
 <wire x1="-19.05" y1="95.25" x2="-19.05" y2="71.12" width="0" layer="19" extent="1-1"/>
 <wire x1="-19.05" y1="119.38" x2="-19.05" y2="95.25" width="0" layer="19" extent="1-1"/>
-<wire x1="-41.7322" y1="130.81" x2="-19.05" y2="119.38" width="0" layer="19" extent="1-1"/>
-<wire x1="-56.2" y1="127" x2="-41.7322" y2="130.81" width="0" layer="19" extent="1-1"/>
 <wire x1="-149.86" y1="-190.5" x2="-155.1637" y2="-78.74" width="0" layer="19" extent="1-1"/>
 <wire x1="-142.24" y1="-190.5" x2="-149.86" y2="-190.5" width="0" layer="19" extent="1-1"/>
@@
 <wire x1="-149.86" y1="-224.79" x2="-149.86" y2="-213.36" width="0" layer="19" extent="1-1"/>
 <wire x1="-142.24" y1="-224.79" x2="-149.86" y2="-224.79" width="0" layer="19" extent="1-1"/>
+<wire x1="-199.5678" y1="-245.11" x2="-149.86" y2="-224.79" width="0" layer="19" extent="1-1"/>
+<wire x1="-221.3" y1="-237.49" x2="-199.5678" y2="-245.11" width="0" layer="19" extent="1-1"/>
 </signal>
 <signal name="M0:+5V">
@@
 <wire x1="-24.13" y1="119.38" x2="-149.86" y2="-232.41" width="0" layer="19" extent="1-1"/>
 </signal>
-<signal name="F1:GND" class="3">
-<contactref element="F1:LED2" pad="C"/>
-</signal>
-<signal name="F1:N$165">
-<contactref element="F1:LED2" pad="A"/>
-<contactref element="F1:LED1" pad="C"/>
-<wire x1="-50.8" y1="125.25" x2="-45.72" y2="128.75" width="0" layer="19" extent="1-1"/>
-</signal>
-<signal name="F1:N$166">
-<contactref element="F1:LED1" pad="A"/>
-<contactref element="F1:R1" pad="1"/>
-<wire x1="-58.1" y1="127" x2="-45.72" y2="125.25" width="0" layer="19" extent="1-1"/>
-</signal>
-<signal name="F1:IN">
-<contactref element="F1:F1" pad="2"/>
-</signal>
 <signal name="P1:N$1">
 <contactref element="P1:U$1" pad="P2"/>
@@
 <contactref element="M3:IC1" pad="7"/>
 </signal>
+<signal name="F1:N$165">
+<contactref element="F1:LED1" pad="C"/>
+<contactref element="F1:LED2" pad="A"/>
+<wire x1="-214.4" y1="-229.87" x2="-223.75" y2="-229.87" width="0" layer="19" extent="1-1"/>
+</signal>
+<signal name="F1:GND" class="3">
+<contactref element="F1:LED2" pad="C"/>
+</signal>
+<signal name="F1:N$1">
+<contactref element="F1:R1" pad="1"/>
+<contactref element="F1:LED1" pad="A"/>
+<wire x1="-217.4" y1="-229.87" x2="-223.2" y2="-237.49" width="0" layer="19" extent="1-1"/>
+</signal>
+<signal name="F1:IN">
+<contactref element="F1:F1" pad="1"/>
+</signal>
 </signals>

Commit message: + sch (Module zur Übersicht hinzugefügt)
Parts:
- added 5V-LINEARWANDLER1:C1, ANSCHLUESSE1:C1, BLUETOOTH1:C1, SENSOREN1:C1, SENSOREN1:C2, SENSOREN1:C3, SENSOREN1:C4, SENSOREN1:C5, SENSOREN1:C6, SENSOREN1:C7, SENSOREN1:C8, X1:C1, Y1:C1: 100n, iceberg20:C0805
- added 5V-LINEARWANDLER1:C2: 330n, iceberg20:C0805
- added 5V-LINEARWANDLER1:IC1: L7805CV, iceberg20:DPAK
- added 5V-SCHALTREGLER1:C3: 100uF, 16V, ±20 %, iceberg20:CAPACITOR-THT-6.3
- added 5V-SCHALTREGLER1:C4: 1000uF, 25V, ±20 %, iceberg20:CAPACITOR-THT-10
- added 5V-SCHALTREGLER1:D1: 1N5822, iceberg20:DO-201AD
- added 5V-SCHALTREGLER1:IC2: LM2576, iceberg20:TO220-5PIN
- added 5V-SCHALTREGLER1:L1: L-100U, iceberg20:PISR
- added 5V-SCHALTREGLER1:R1, BLUETOOTH1:R2, K1:R2, X1:R1, X1:R2, X1:R4, X1:R6: 100k, iceberg20:R0805
- added ANSCHLUESSE-UNTEN1:X1: BUCHSENLEISTE-10, iceberg20:2X5
- added ANSCHLUESSE-UNTEN1:X2: WANNENSTECKER-30, iceberg20:2X15
- added ANSCHLUESSE1:C2, C1:C1: 1 uF, 50 V, ±20 %, iceberg20:CAPACITOR-THT-4
- added ANSCHLUESSE1:X1, ANSCHLUESSE1:X2, ANSCHLUESSE1:X3, ANSCHLUESSE1:X4, C1:X3, SENSOREN1:X1, SENSOREN1:X2: PS25/2GPS25/2GWS-1X02, iceberg20:CON-01X02
- added ANSCHLUESSE1:X5: PS25/4G, iceberg20:CON-01X04
- added BLUETOOTH1:IC1: HC-05, iceberg20:HC-05
- added C1:J1: JUMPER, iceberg20:JUMPER-SJ-3
- added C1:X1, C1:X2, PUI1:X4: WANNENSTECKER-6, iceberg20:2X3
- added EIN/AUSGABE1:LED1, EIN/AUSGABE1:LED2: GREEN, iceberg20:PLCC-2
- added EIN/AUSGABE1:LED3, EIN/AUSGABE1:LED4, EIN/AUSGABE1:LED6: LED-WHITE, iceberg20:PLCC-2
- added EIN/AUSGABE1:M1: SPEAKER, iceberg20:SPEAKER
- added EIN/AUSGABE1:R1, EIN/AUSGABE1:R2, X1:R3, X1:R5: 100, iceberg20:R0805
- added EIN/AUSGABE1:R3, EIN/AUSGABE1:R4, EIN/AUSGABE1:R5: 120R, iceberg20:R0805
- added EIN/AUSGABE1:S1: SWITCH, iceberg20:1801.2106
- added ENC1:IC1: TEENSY-3.2, iceberg20:TEENSY-3
- added K1:C1: 2,2 mF, 16 V, ±20 %, iceberg20:CAPACITOR-THT-13
- added K1:D1: DIODE, iceberg20:DO-214BA
- added K1:R1: 300R, iceberg20:R0805
- added K1:T1: IRF1405, iceberg20:TO220V
- added PUI1:X3: JST-XH-4, iceberg20:XH-4
- added SENSOREN1:IC1: LM-35, iceberg20:TO-92
- added SENSOREN1:IC2: CMPS12, iceberg20:CMPS12
- added SENSOREN1:IC3: RTC, iceberg20:RTC
- added SENSOREN1:IC4, SENSOREN1:IC5, SENSOREN1:IC6, SENSOREN1:IC7, SENSOREN1:IC8: SRF-08, iceberg20:SRF-08
- added SENSOREN1:J1: JUMPER-2, iceberg20:SJ
- added SENSOREN1:R1: 20k, iceberg20:R0805
- added SENSOREN1:R2: 470, iceberg20:R0805
- added SENSOREN1:T1: SFH320, iceberg20:PLCC-2
- added X1:IC1: DS1099, iceberg20:USOP-8
- added X1:LED1, X1:LED10, X1:LED11, X1:LED12, X1:LED13, X1:LED14, X1:LED2, X1:LED3, X1:LED4, X1:LED5, X1:LED6, X1:LED7, X1:LED8, X1:LED9: IR-LED, iceberg20:LED-3MM
- added X1:R7, X1:R8: 15, iceberg20:R0805
- added X1:T1, X1:T2: KMA3D6N20SA, iceberg20:SOT23
- added Y1:IC1, Y1:IC2, Y1:IC3, Y1:IC4, Y1:IC5, Y1:IC6: TSOP31433, iceberg20:TSOP312
- moved M2:C4 1.27 mm to (-139.7, -44.5)
Connections:
- removed net F1:GND: F1:LED2.C
- removed net F1:IN: F1:F1.1
- removed net M0:+5V: M0:C6.1, M0:IC2.8
- removed net M0:GND: M0:C3.2, M0:C4.2, M0:C5.2, M0:C6.2, M0:IC1.15, M0:IC1.16, M0:IC1.3, M0:IC1.5, M0:IC1.6, M0:IC1.8, M0:IC2.5, M0:R3.1
- removed net M1:+5V: M1:C6.1, M1:IC2.8
- removed net M1:GND: M1:C3.2, M1:C4.2, M1:C5.2, M1:C6.2, M1:IC1.15, M1:IC1.16, M1:IC1.3, M1:IC1.5, M1:IC1.6, M1:IC1.8, M1:IC2.5, M1:R3.1
- removed net M2:+5V: M2:C6.1, M2:IC2.8
- removed net M2:GND: M2:C3.2, M2:C4.2, M2:C5.2, M2:C6.2, M2:IC1.15, M2:IC1.16, M2:IC1.3, M2:IC1.5, M2:IC1.6, M2:IC1.8, M2:IC2.5, M2:R3.1
- removed net M3:+5V: M3:C6.1, M3:IC2.8
- removed net M3:GND: M3:C3.2, M3:C4.2, M3:C5.2, M3:C6.2, M3:IC1.15, M3:IC1.16, M3:IC1.3, M3:IC1.5, M3:IC1.6, M3:IC1.8, M3:IC2.5, M3:R3.1
- removed net P1:GND: P1:R1.1, P1:U$1.P1
- new net +12V: 5V-LINEARWANDLER1:C2.1, 5V-LINEARWANDLER1:IC1.1, 5V-SCHALTREGLER1:C3.1, 5V-SCHALTREGLER1:IC2.1, ANSCHLUESSE-UNTEN1:X2.19, ANSCHLUESSE-UNTEN1:X2.27, ANSCHLUESSE-UNTEN1:X2.28, ANSCHLUESSE1:C2.1, ANSCHLUESSE1:X2.1, C1:C1.1, C1:J1.3, C1:X3.2, F1:F1.1, PUI1:X4.6, X1:R7.2, X1:R8.2
- new net +5V: 5V-LINEARWANDLER1:C1.1, 5V-LINEARWANDLER1:IC1.2, 5V-SCHALTREGLER1:C4.1, 5V-SCHALTREGLER1:IC2.4, 5V-SCHALTREGLER1:L1.2, 5V-SCHALTREGLER1:R1.2, ANSCHLUESSE-UNTEN1:X2.1, ANSCHLUESSE-UNTEN1:X2.13, ANSCHLUESSE-UNTEN1:X2.5, ANSCHLUESSE-UNTEN1:X2.9, ANSCHLUESSE1:C1.1, ANSCHLUESSE1:X1.1, ANSCHLUESSE1:X5.4, BLUETOOTH1:C1.1, BLUETOOTH1:IC1.5, C1:J1.1, C1:X2.2, C1:X2.5, EIN/AUSGABE1:R1.2, ENC1:IC1.VIN, M0:C6.1, M0:IC2.8, M1:C6.1, M1:IC2.8, M2:C6.1, M2:IC2.8, M3:C6.1, M3:IC2.8, PUI1:X3.P$1, SENSOREN1:C1.1, SENSOREN1:C2.1, SENSOREN1:C3.1, SENSOREN1:C4.1, SENSOREN1:C5.1, SENSOREN1:C6.1, SENSOREN1:C7.1, SENSOREN1:C8.1, SENSOREN1:IC1.3, SENSOREN1:IC2.1, SENSOREN1:IC3.+, SENSOREN1:IC4.1, SENSOREN1:IC5.1, SENSOREN1:IC6.1, SENSOREN1:IC7.1, SENSOREN1:IC8.1, SENSOREN1:T1.A, X1:C1.1, X1:IC1.3, X1:R1.2, X1:R2.2, Y1:C1.1, Y1:IC1.2, Y1:IC2.2, Y1:IC3.2, Y1:IC4.2, Y1:IC5.2, Y1:IC6.2
- new net 5V-SCHALTREGLER1:N$1: 5V-SCHALTREGLER1:IC2.5, 5V-SCHALTREGLER1:R1.1
- new net 5V-SCHALTREGLER1:N$2: 5V-SCHALTREGLER1:D1.1, 5V-SCHALTREGLER1:IC2.2, 5V-SCHALTREGLER1:L1.1
- new net ANSCHLUESSE-UNTEN1:ENA0: ANSCHLUESSE-UNTEN1:X2.2
- new net ANSCHLUESSE-UNTEN1:ENA1: ANSCHLUESSE-UNTEN1:X2.7
- new net ANSCHLUESSE-UNTEN1:ENA2: ANSCHLUESSE-UNTEN1:X2.10
- new net ANSCHLUESSE-UNTEN1:ENA3: ANSCHLUESSE-UNTEN1:X2.14
- new net ANSCHLUESSE-UNTEN1:ENB0: ANSCHLUESSE-UNTEN1:X2.3
- new net ANSCHLUESSE-UNTEN1:ENB1: ANSCHLUESSE-UNTEN1:X2.6
- new net ANSCHLUESSE-UNTEN1:ENB2: ANSCHLUESSE-UNTEN1:X2.11
- new net ANSCHLUESSE-UNTEN1:ENB3: ANSCHLUESSE-UNTEN1:X2.15
- new net ANSCHLUESSE-UNTEN1:INTERRUPT-O: ANSCHLUESSE-UNTEN1:X2.18
- new net ANSCHLUESSE-UNTEN1:KICKA: ANSCHLUESSE-UNTEN1:X1.9
- new net ANSCHLUESSE-UNTEN1:KICKB: ANSCHLUESSE-UNTEN1:X1.10
- new net ANSCHLUESSE-UNTEN1:LED-I: ANSCHLUESSE-UNTEN1:X2.21
- new net ANSCHLUESSE-UNTEN1:MA0: ANSCHLUESSE-UNTEN1:X1.1
- new net ANSCHLUESSE-UNTEN1:MA1: ANSCHLUESSE-UNTEN1:X1.3
- new net ANSCHLUESSE-UNTEN1:MA2: ANSCHLUESSE-UNTEN1:X1.5
- new net ANSCHLUESSE-UNTEN1:MA3: ANSCHLUESSE-UNTEN1:X1.7, ANSCHLUESSE-UNTEN1:X1.8
- new net ANSCHLUESSE-UNTEN1:MB0: ANSCHLUESSE-UNTEN1:X1.2
- new net ANSCHLUESSE-UNTEN1:MB1: ANSCHLUESSE-UNTEN1:X1.4
- new net ANSCHLUESSE-UNTEN1:MB2: ANSCHLUESSE-UNTEN1:X1.6
- new net ANSCHLUESSE-UNTEN1:RST: ANSCHLUESSE-UNTEN1:X2.29
- new net ANSCHLUESSE-UNTEN1:SCL: ANSCHLUESSE-UNTEN1:X2.26
- new net ANSCHLUESSE-UNTEN1:SDA: ANSCHLUESSE-UNTEN1:X2.23
- new net ANSCHLUESSE1:A1: ANSCHLUESSE1:X3.1
- new net ANSCHLUESSE1:D1: ANSCHLUESSE1:X4.1
- new net ANSCHLUESSE1:SCL: ANSCHLUESSE1:X5.1
- new net ANSCHLUESSE1:SDA: ANSCHLUESSE1:X5.3
- new net BLUETOOTH1:IN: BLUETOOTH1:IC1.6, BLUETOOTH1:R2.1
- new net BLUETOOTH1:OUT: BLUETOOTH1:IC1.1
- new net BLUETOOTH1:RX: BLUETOOTH1:IC1.2
- new net BLUETOOTH1:TX: BLUETOOTH1:IC1.3
- new net C1:5V-CAMERA: C1:J1.2, C1:X1.2
- new net C1:CLK: C1:X1.3
- new net C1:CS: C1:X1.5
- new net C1:MISO: C1:X1.1
- new net C1:MOSI: C1:X1.4
- new net C1:RX-C: C1:X2.3
- new net C1:TX-C: C1:X2.4
- new net EIN/AUSGABE1:HB-I: EIN/AUSGABE1:LED1.C, EIN/AUSGABE1:R2.2
- new net EIN/AUSGABE1:LED1-I: EIN/AUSGABE1:R3.2
- new net EIN/AUSGABE1:LED2-I: EIN/AUSGABE1:R5.2
- new net EIN/AUSGABE1:LED3-I: EIN/AUSGABE1:R4.2
- new net EIN/AUSGABE1:N$1: EIN/AUSGABE1:LED1.A, EIN/AUSGABE1:R1.1
- new net EIN/AUSGABE1:N$2: EIN/AUSGABE1:LED2.A, EIN/AUSGABE1:R2.1
- new net EIN/AUSGABE1:N$3: EIN/AUSGABE1:LED3.A, EIN/AUSGABE1:R3.1
- new net EIN/AUSGABE1:N$4: EIN/AUSGABE1:LED6.A, EIN/AUSGABE1:R5.1
- new net EIN/AUSGABE1:N$5: EIN/AUSGABE1:LED4.A, EIN/AUSGABE1:R4.1
- new net EIN/AUSGABE1:SPEAKER-I: EIN/AUSGABE1:M1.1
- new net EIN/AUSGABE1:SWITCH-O: EIN/AUSGABE1:S1.2
- new net ENC1:3.3V: ENC1:IC1.3.3V
- new net ENC1:3V: ENC1:IC1.3V
- new net ENC1:ENA0: ENC1:IC1.2
- new net ENC1:ENA1: ENC1:IC1.4
- new net ENC1:ENA2: ENC1:IC1.14
- new net ENC1:ENA3: ENC1:IC1.16
- new net ENC1:ENB0: ENC1:IC1.3
- new net ENC1:ENB1: ENC1:IC1.5
- new net ENC1:ENB2: ENC1:IC1.15
- new net ENC1:ENB3: ENC1:IC1.17
- new net ENC1:SCL: ENC1:IC1.19
- new net ENC1:SDA: ENC1:IC1.18
- new net ENC1:VBAT: ENC1:IC1.VBAT
- new net ENC1:VUSB: ENC1:IC1.VUSB
- new net GND: 5V-LINEARWANDLER1:C1.2, 5V-LINEARWANDLER1:C2.2, 5V-LINEARWANDLER1:IC1.3, 5V-SCHALTREGLER1:C3.2, 5V-SCHALTREGLER1:C4.2, 5V-SCHALTREGLER1:D1.2, 5V-SCHALTREGLER1:IC2.3, ANSCHLUESSE-UNTEN1:X2.12, ANSCHLUESSE-UNTEN1:X2.16, ANSCHLUESSE-UNTEN1:X2.17, ANSCHLUESSE-UNTEN1:X2.20, ANSCHLUESSE-UNTEN1:X2.22, ANSCHLUESSE-UNTEN1:X2.24, ANSCHLUESSE-UNTEN1:X2.25, ANSCHLUESSE-UNTEN1:X2.30, ANSCHLUESSE-UNTEN1:X2.4, ANSCHLUESSE-UNTEN1:X2.8, ANSCHLUESSE1:C1.2, ANSCHLUESSE1:C2.2, ANSCHLUESSE1:X1.2, ANSCHLUESSE1:X2.2, ANSCHLUESSE1:X3.2, ANSCHLUESSE1:X4.2, ANSCHLUESSE1:X5.2, BLUETOOTH1:C1.2, BLUETOOTH1:IC1.4, BLUETOOTH1:R2.2, C1:C1.2, C1:X1.6, C1:X2.1, C1:X2.6, C1:X3.1, EIN/AUSGABE1:LED2.C, EIN/AUSGABE1:LED3.C, EIN/AUSGABE1:LED4.C, EIN/AUSGABE1:LED6.C, EIN/AUSGABE1:M1.2, EIN/AUSGABE1:S1.1, ENC1:IC1.AGND, ENC1:IC1.GND, ENC1:IC1.GND1, F1:LED2.C, K1:C1.2, K1:R2.1, K1:T1.3, M0:C3.2, M0:C4.2, M0:C5.2, M0:C6.2, M0:IC1.15, M0:IC1.16, M0:IC1.3, M0:IC1.5, M0:IC1.6, M0:IC1.8, M0:IC2.5, M0:R3.1, M1:C3.2, M1:C4.2, M1:C5.2, M1:C6.2, M1:IC1.15, M1:IC1.16, M1:IC1.3, M1:IC1.5, M1:IC1.6, M1:IC1.8, M1:IC2.5, M1:R3.1, M2:C3.2, M2:C4.2, M2:C5.2, M2:C6.2, M2:IC1.15, M2:IC1.16, M2:IC1.3, M2:IC1.5, M2:IC1.6, M2:IC1.8, M2:IC2.5, M2:R3.1, M3:C3.2, M3:C4.2, M3:C5.2, M3:C6.2, M3:IC1.15, M3:IC1.16, M3:IC1.3, M3:IC1.5, M3:IC1.6, M3:IC1.8, M3:IC2.5, M3:R3.1, P1:R1.1, P1:U$1.P1, PUI1:X3.P$4, PUI1:X4.1, PUI1:X4.3, SENSOREN1:C1.2, SENSOREN1:C2.2, SENSOREN1:C3.2, SENSOREN1:C4.2, SENSOREN1:C5.2, SENSOREN1:C6.2, SENSOREN1:C7.2, SENSOREN1:C8.2, SENSOREN1:IC1.1, SENSOREN1:IC2.6, SENSOREN1:IC3.-, SENSOREN1:IC4.5, SENSOREN1:IC5.5, SENSOREN1:IC6.5, SENSOREN1:IC7.5, SENSOREN1:IC8.5, SENSOREN1:J1.1, SENSOREN1:R1.1, SENSOREN1:X2.1, X1:C1.2, X1:IC1.4, X1:R4.1, X1:R6.1, X1:T1.1, X1:T2.1, Y1:C1.2, Y1:IC1.1, Y1:IC2.1, Y1:IC3.1, Y1:IC4.1, Y1:IC5.1, Y1:IC6.1
- new net K1:KICK-OUTA: K1:D1.2, K1:T1.2
- new net K1:KICK-OUTB: K1:C1.1, K1:D1.1
- new net K1:KICK_EN: K1:R1.1
- new net K1:N$1: K1:R1.2, K1:R2.2, K1:T1.1
- new net PUI1:RST: PUI1:X4.4
- new net PUI1:RX: PUI1:X3.P$3
- new net PUI1:SCL: PUI1:X4.5
- new net PUI1:SDA: PUI1:X4.2
- new net PUI1:TX: PUI1:X3.P$2
- new net SENSOREN1:BR-I: SENSOREN1:R2.2
- new net SENSOREN1:BR-O: SENSOREN1:X1.2
- new net SENSOREN1:N$1: SENSOREN1:IC2.4, SENSOREN1:J1.2
- new net SENSOREN1:N$2: SENSOREN1:R2.1, SENSOREN1:X2.2
- new net SENSOREN1:N$3: SENSOREN1:X1.1
- new net SENSOREN1:PHOTO-O: SENSOREN1:R1.2, SENSOREN1:T1.C
- new net SENSOREN1:SCL: SENSOREN1:IC2.3, SENSOREN1:IC3.C, SENSOREN1:IC4.3, SENSOREN1:IC5.3, SENSOREN1:IC6.3, SENSOREN1:IC7.3, SENSOREN1:IC8.3
- new net SENSOREN1:SDA: SENSOREN1:IC2.2, SENSOREN1:IC3.D, SENSOREN1:IC4.2, SENSOREN1:IC5.2, SENSOREN1:IC6.2, SENSOREN1:IC7.2, SENSOREN1:IC8.2
- new net SENSOREN1:TEMP-O: SENSOREN1:IC1.2
- new net X1:IN1: X1:IC1.5, X1:R1.1
- new net X1:IN2: X1:IC1.6, X1:R2.1
- new net X1:N$1: X1:R3.2, X1:R4.2, X1:T1.2
- new net X1:N$10: X1:R5.2, X1:R6.2, X1:T2.2
- new net X1:N$11: X1:IC1.2, X1:R3.1
- new net X1:N$12: X1:LED8.2, X1:T2.3
- new net X1:N$13: X1:LED8.1, X1:LED9.2
- new net X1:N$14: X1:LED10.2, X1:LED9.1
- new net X1:N$15: X1:LED10.1, X1:LED11.2
- new net X1:N$16: X1:LED11.1, X1:LED12.2
- new net X1:N$17: X1:LED12.1, X1:LED13.2
- new net X1:N$18: X1:LED13.1, X1:LED14.2
- new net X1:N$19: X1:LED14.1, X1:R8.1
- new net X1:N$2: X1:IC1.1, X1:R5.1
- new net X1:N$20: X1:LED7.1, X1:R7.1
- new net X1:N$3: X1:LED1.2, X1:T1.3
- new net X1:N$4: X1:LED1.1, X1:LED2.2
- new net X1:N$5: X1:LED2.1, X1:LED3.2
- new net X1:N$6: X1:LED3.1, X1:LED4.2
- new net X1:N$7: X1:LED4.1, X1:LED5.2
- new net X1:N$8: X1:LED5.1, X1:LED6.2
- new net X1:N$9: X1:LED6.1, X1:LED7.2
- new net Y1:OUT1: Y1:IC1.3
- new net Y1:OUT2: Y1:IC2.3
- new net Y1:OUT3: Y1:IC3.3
- new net Y1:OUT4: Y1:IC4.3
- new net Y1:OUT5: Y1:IC5.3
- new net Y1:OUT6: Y1:IC6.3
