File: iceberg20.brd (EAGLE design)
At the start: 160 x 100 mm, 189 parts, among them K1:C1 2,2 mF, 16 V, ±20 %, K1:D1 DIODE, K1:R1 300R, K1:R2 100k, K1:T1 IRF1405, M0:+ TPB1,27, M0:- TPB1,27, M0:C1 10nF, M0:C2 220nF, M0:C3 100nF, M0:C4 100uF, 16V, ±20 %, M0:C5 1nF, M0:C6 100nF, M0:D1 DIODE, M0:D2 DIODE, M0:EN TPB1,27, M0:I TPB1,27, M0:IC1 L6205N, M0:IC2 ACS712ACS712-SOIC-8, M0:IN1 TPB1,27, M0:IN2 TPB1,27, M0:R1 100R, M0:R2 100k, M0:R3 10k, M0:VS TPB1,27, M1:+ TPB1,27, M1:- TPB1,27, M1:C1 10nF, M1:C2 220nF, M1:C3 100nF, M1:C4 100uF, 16V, ±20 %, M1:C5 1nF, M1:C6 100nF, M1:D1 DIODE, M1:D2 DIODE, M1:EN TPB1,27, M1:I TPB1,27, M1:IC1 L6205N, M1:IC2 ACS712ACS712-SOIC-8, M1:IN1 TPB1,27, M1:IN2 TPB1,27, M1:R1 100R, M1:R2 100k, M1:R3 10k, M1:VS TPB1,27, M2:+ TPB1,27, M2:- TPB1,27, M2:C1 10nF, M2:C2 220nF, M2:C3 100nF, M2:C4 100uF, 16V, ±20 %, M2:C5 1nF, M2:C6 100nF, M2:D1 DIODE, M2:D2 DIODE, M2:EN TPB1,27, M2:I TPB1,27, M2:IC1 L6205N, M2:IC2 ACS712ACS712-SOIC-8, M2:IN1 TPB1,27, M2:IN2 TPB1,27, M2:R1 100R, M2:R2 100k, M2:R3 10k, M2:VS TPB1,27, M3:+ TPB1,27, M3:- TPB1,27, M3:C1 10nF, M3:C2 220nF, M3:C3 100nF, M3:C4 100uF, 16V, ±20 %, M3:C5 1nF, M3:C6 100nF, M3:D1 DIODE, M3:D2 DIODE, M3:EN TPB1,27, M3:I TPB1,27, M3:IC1 L6205N, M3:IC2 ACS712ACS712-SOIC-8, M3:IN1 TPB1,27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

Commit message: work in progress
Parts:
- renumbered C1:C1 to CAMERA1:C1, C1:J1 to CAMERA1:J1, C1:X1 to CAMERA1:X1, C1:X2 to CAMERA1:X2, C1:X3 to CAMERA1:X3, X1:C1 to IR_SENDER1:C1, X1:IC1 to IR_SENDER1:IC1, X1:LED1 to IR_SENDER1:LED1, X1:LED10 to IR_SENDER1:LED10, X1:LED11 to IR_SENDER1:LED11, X1:LED12 to IR_SENDER1:LED12, X1:LED13 to IR_SENDER1:LED13, X1:LED14 to IR_SENDER1:LED14, X1:LED2 to IR_SENDER1:LED2, X1:LED3 to IR_SENDER1:LED3, X1:LED4 to IR_SENDER1:LED4, X1:LED5 to IR_SENDER1:LED5, X1:LED6 to IR_SENDER1:LED6, X1:LED7 to IR_SENDER1:LED7, X1:LED8 to IR_SENDER1:LED8, X1:LED9 to IR_SENDER1:LED9, X1:R1 to IR_SENDER1:R1, X1:R2 to IR_SENDER1:R2, X1:R3 to IR_SENDER1:R3, X1:R4 to IR_SENDER1:R4, X1:R5 to IR_SENDER1:R5, X1:R6 to IR_SENDER1:R6, X1:R7 to IR_SENDER1:R7, X1:R8 to IR_SENDER1:R8, X1:T1 to IR_SENDER1:T1, X1:T2 to IR_SENDER1:T2, Y1:C1 to IR-EMPFAENGER1:C1, Y1:IC1 to IR-EMPFAENGER1:IC1, Y1:IC2 to IR-EMPFAENGER1:IC2, Y1:IC3 to IR-EMPFAENGER1:IC3, Y1:IC4 to IR-EMPFAENGER1:IC4, Y1:IC5 to IR-EMPFAENGER1:IC5, Y1:IC6 to IR-EMPFAENGER1:IC6
Connections:
- net ANSCHLUESSE-UNTEN1:INTERRUPT-O renamed INTERRUPT-O
- net ANSCHLUESSE-UNTEN1:LED-I renamed RGBLED-I
- net ANSCHLUESSE-UNTEN1:RST renamed RST2
- net ANSCHLUESSE1:A1 renamed A1
- net ANSCHLUESSE1:D1 renamed D1
- net BLUETOOTH1:IN renamed IN
- net BLUETOOTH1:OUT renamed OUT
- net BLUETOOTH1:RX renamed RX-B
- net BLUETOOTH1:TX renamed TX-B
- net C1:5V-CAMERA renamed CAMERA1:5V-CAMERA
- net C1:CLK renamed CLK
- net C1:CS renamed CS
- net C1:MISO renamed MISO
- net C1:MOSI renamed MOSI
- net C1:RX-C renamed RX-C
- net C1:TX-C renamed TX-C
- net EIN/AUSGABE1:HB-I renamed HB-I
- net EIN/AUSGABE1:LED1-I renamed LED1-I
- net EIN/AUSGABE1:LED2-I renamed LED2-I
- net EIN/AUSGABE1:LED3-I renamed LED3-I
- net EIN/AUSGABE1:SPEAKER-I renamed SPEAKER-I
- net EIN/AUSGABE1:SWITCH-O renamed SWITCH-O
- net K1:KICK_EN renamed KICK-EN
- net M3:M+OUT renamed MB3
- net PUI1:RST renamed RST1
- net PUI1:RX renamed RX-P
- net PUI1:TX renamed TX-P
- net SENSOREN1:BR-I renamed BR-I
- net SENSOREN1:BR-O renamed BR-O
- net SENSOREN1:PHOTO-O renamed PHOTO-O
- net SENSOREN1:TEMP-O renamed TEMP-O
- net X1:IN1 renamed IN1
- net X1:IN2 renamed IN2
- net X1:N$1 renamed IR_SENDER1:N$1
- net X1:N$10 renamed IR_SENDER1:N$10
- net X1:N$11 renamed IR_SENDER1:N$11
- net X1:N$12 renamed IR_SENDER1:N$12
- net X1:N$13 renamed IR_SENDER1:N$13
- net X1:N$14 renamed IR_SENDER1:N$14
- net X1:N$15 renamed IR_SENDER1:N$15
- net X1:N$16 renamed IR_SENDER1:N$16
- net X1:N$17 renamed IR_SENDER1:N$17
- net X1:N$18 renamed IR_SENDER1:N$18
- net X1:N$19 renamed IR_SENDER1:N$19
- net X1:N$2 renamed IR_SENDER1:N$2
- net X1:N$20 renamed IR_SENDER1:N$20
- net X1:N$3 renamed IR_SENDER1:N$3
- net X1:N$4 renamed IR_SENDER1:N$4
- net X1:N$5 renamed IR_SENDER1:N$5
- net X1:N$6 renamed IR_SENDER1:N$6
- net X1:N$7 renamed IR_SENDER1:N$7
- net X1:N$8 renamed IR_SENDER1:N$8
- net X1:N$9 renamed IR_SENDER1:N$9
- net Y1:OUT1 renamed OUT1
- net Y1:OUT2 renamed OUT2
- net Y1:OUT3 renamed OUT3
- net Y1:OUT4 renamed OUT4
- net Y1:OUT5 renamed OUT5
- net Y1:OUT6 renamed OUT6
- removed net ANSCHLUESSE-UNTEN1:ENA0: ANSCHLUESSE-UNTEN1:X2.2
- removed net ANSCHLUESSE-UNTEN1:ENA1: ANSCHLUESSE-UNTEN1:X2.7
- removed net ANSCHLUESSE-UNTEN1:ENA2: ANSCHLUESSE-UNTEN1:X2.10
- removed net ANSCHLUESSE-UNTEN1:ENA3: ANSCHLUESSE-UNTEN1:X2.14
- removed net ANSCHLUESSE-UNTEN1:ENB0: ANSCHLUESSE-UNTEN1:X2.3
- removed net ANSCHLUESSE-UNTEN1:ENB1: ANSCHLUESSE-UNTEN1:X2.6
- removed net ANSCHLUESSE-UNTEN1:ENB2: ANSCHLUESSE-UNTEN1:X2.11
- removed net ANSCHLUESSE-UNTEN1:ENB3: ANSCHLUESSE-UNTEN1:X2.15
- removed net ANSCHLUESSE-UNTEN1:KICKA: ANSCHLUESSE-UNTEN1:X1.9
- removed net ANSCHLUESSE-UNTEN1:KICKB: ANSCHLUESSE-UNTEN1:X1.10
- removed net ANSCHLUESSE-UNTEN1:MA0: ANSCHLUESSE-UNTEN1:X1.1
- removed net ANSCHLUESSE-UNTEN1:MA1: ANSCHLUESSE-UNTEN1:X1.3
- removed net ANSCHLUESSE-UNTEN1:MA2: ANSCHLUESSE-UNTEN1:X1.5
- removed net ANSCHLUESSE-UNTEN1:MA3: ANSCHLUESSE-UNTEN1:X1.7, ANSCHLUESSE-UNTEN1:X1.8
- removed net ANSCHLUESSE-UNTEN1:MB0: ANSCHLUESSE-UNTEN1:X1.2
- removed net ANSCHLUESSE-UNTEN1:MB1: ANSCHLUESSE-UNTEN1:X1.4
- removed net ANSCHLUESSE-UNTEN1:MB2: ANSCHLUESSE-UNTEN1:X1.6
- removed net ANSCHLUESSE-UNTEN1:SCL: ANSCHLUESSE-UNTEN1:X2.26
- removed net ANSCHLUESSE-UNTEN1:SDA: ANSCHLUESSE-UNTEN1:X2.23
- removed net ANSCHLUESSE1:SCL: ANSCHLUESSE1:X5.1
- removed net ANSCHLUESSE1:SDA: ANSCHLUESSE1:X5.3
- removed net ENC1:ENA0: ENC1:IC1.2
- removed net ENC1:ENA1: ENC1:IC1.4
- removed net ENC1:ENA2: ENC1:IC1.14
- removed net ENC1:ENA3: ENC1:IC1.16
- removed net ENC1:ENB0: ENC1:IC1.3
- removed net ENC1:ENB1: ENC1:IC1.5
- removed net ENC1:ENB2: ENC1:IC1.15
- removed net ENC1:ENB3: ENC1:IC1.17
- removed net ENC1:SCL: ENC1:IC1.19
- removed net ENC1:SDA: ENC1:IC1.18
- removed net K1:KICK-OUTA: K1:D1.2, K1:T1.2
- removed net K1:KICK-OUTB: K1:C1.1, K1:D1.1
- removed net M0:M+OUT: M0:+.TP, M0:IC1.4
- removed net M0:M-OUT: M0:-.TP, M0:IC2.1, M0:IC2.2
- removed net M1:M+OUT: M1:+.TP, M1:IC1.4
- removed net M1:M-OUT: M1:-.TP, M1:IC2.1, M1:IC2.2
- removed net M2:M+OUT: M2:+.TP, M2:IC1.4
- removed net M2:M-OUT: M2:-.TP, M2:IC2.1, M2:IC2.2
- removed net M3:M-OUT: M3:-.TP, M3:IC2.1, M3:IC2.2
- removed net PUI1:SCL: PUI1:X4.5
- removed net PUI1:SDA: PUI1:X4.2
- removed net SENSOREN1:SCL: SENSOREN1:IC2.3, SENSOREN1:IC3.C, SENSOREN1:IC4.3, SENSOREN1:IC5.3, SENSOREN1:IC6.3, SENSOREN1:IC7.3, SENSOREN1:IC8.3
- removed net SENSOREN1:SDA: SENSOREN1:IC2.2, SENSOREN1:IC3.D, SENSOREN1:IC4.2, SENSOREN1:IC5.2, SENSOREN1:IC6.2, SENSOREN1:IC7.2, SENSOREN1:IC8.2
- new net ENA0: ANSCHLUESSE-UNTEN1:X2.2, ENC1:IC1.2
- new net ENA1: ANSCHLUESSE-UNTEN1:X2.7, ENC1:IC1.4
- new net ENA2: ANSCHLUESSE-UNTEN1:X2.10, ENC1:IC1.14
- new net ENA3: ANSCHLUESSE-UNTEN1:X2.14, ENC1:IC1.16
- new net ENB0: ANSCHLUESSE-UNTEN1:X2.3, ENC1:IC1.3
- new net ENB1: ANSCHLUESSE-UNTEN1:X2.6, ENC1:IC1.5
- new net ENB2: ANSCHLUESSE-UNTEN1:X2.11, ENC1:IC1.15
- new net ENB3: ANSCHLUESSE-UNTEN1:X2.15, ENC1:IC1.17
- new net KICKA: ANSCHLUESSE-UNTEN1:X1.9, K1:D1.2, K1:T1.2
- new net KICKB: ANSCHLUESSE-UNTEN1:X1.10, K1:C1.1, K1:D1.1
- new net MA0: ANSCHLUESSE-UNTEN1:X1.1, M0:-.TP, M0:IC2.1, M0:IC2.2
- new net MA1: ANSCHLUESSE-UNTEN1:X1.3, M1:-.TP, M1:IC2.1, M1:IC2.2
- new net MA2: ANSCHLUESSE-UNTEN1:X1.5, M2:-.TP, M2:IC2.1, M2:IC2.2
- new net MA3: ANSCHLUESSE-UNTEN1:X1.7, ANSCHLUESSE-UNTEN1:X1.8, M3:-.TP, M3:IC2.1, M3:IC2.2
- new net MB0: ANSCHLUESSE-UNTEN1:X1.2, M0:+.TP, M0:IC1.4
- new net MB1: ANSCHLUESSE-UNTEN1:X1.4, M1:+.TP, M1:IC1.4
- new net MB2: ANSCHLUESSE-UNTEN1:X1.6, M2:+.TP, M2:IC1.4
- new net SCL: ANSCHLUESSE-UNTEN1:X2.26, ANSCHLUESSE1:X5.1, ENC1:IC1.19, PUI1:X4.5, SENSOREN1:IC2.3, SENSOREN1:IC3.C, SENSOREN1:IC4.3, SENSOREN1:IC5.3, SENSOREN1:IC6.3, SENSOREN1:IC7.3, SENSOREN1:IC8.3
- new net SDA: ANSCHLUESSE-UNTEN1:X2.23, ANSCHLUESSE1:X5.3, ENC1:IC1.18, PUI1:X4.2, SENSOREN1:IC2.2, SENSOREN1:IC3.D, SENSOREN1:IC4.2, SENSOREN1:IC5.2, SENSOREN1:IC6.2, SENSOREN1:IC7.2, SENSOREN1:IC8.2

Commit message: + sch(Übersicht fürs erste beendet)
Parts:
- added 5V-LINEARWANDLER2:C1, 5V-LINEARWANDLER4:C1: 100n, iceberg20:C0805
- added 5V-LINEARWANDLER2:C2, 5V-LINEARWANDLER4:C2: 330n, iceberg20:C0805
- added 5V-LINEARWANDLER2:IC1, 5V-LINEARWANDLER4:IC1: L7805CV, iceberg20:DPAK
- added ARDUINO1:IC1: ARUINO-MEGA, iceberg20:ARDUINO_MEGA
- added F2:F1, F3:F1, F4:F1, F5:F1, F6:F1: (no value), iceberg20:SH22,5
- added F2:LED1, F2:LED2, F3:LED1, F3:LED2, F4:LED1, F4:LED2, F5:LED1, F5:LED2, F6:LED1, F6:LED2: LED-GREEN1, iceberg20:1206
- added F2:R1, F3:R1, F4:R1, F5:R1, F6:R1: 270, iceberg20:R0805
Connections:
- net KICKA renamed N$3
- net KICKB renamed N$5
- removed net A1: ANSCHLUESSE1:X3.1
- removed net BR-I: SENSOREN1:R2.2
- removed net BR-O: SENSOREN1:X1.2
- removed net CLK: CAMERA1:X1.3
- removed net CS: CAMERA1:X1.5
- removed net D1: ANSCHLUESSE1:X4.1
- removed net HB-I: EIN/AUSGABE1:LED1.C, EIN/AUSGABE1:R2.2
- removed net IN: BLUETOOTH1:IC1.6, BLUETOOTH1:R2.1
- removed net IN1: IR_SENDER1:IC1.5, IR_SENDER1:R1.1
- removed net IN2: IR_SENDER1:IC1.6, IR_SENDER1:R2.1
- removed net LED1-I: EIN/AUSGABE1:R3.2
- removed net LED2-I: EIN/AUSGABE1:R5.2
- removed net LED3-I: EIN/AUSGABE1:R4.2
- removed net MISO: CAMERA1:X1.1
- removed net MOSI: CAMERA1:X1.4
- removed net OUT: BLUETOOTH1:IC1.1
- removed net OUT1: IR-EMPFAENGER1:IC1.3
- removed net OUT2: IR-EMPFAENGER1:IC2.3
- removed net OUT3: IR-EMPFAENGER1:IC3.3
- removed net OUT4: IR-EMPFAENGER1:IC4.3
- removed net OUT5: IR-EMPFAENGER1:IC5.3
- removed net OUT6: IR-EMPFAENGER1:IC6.3
- removed net PHOTO-O: SENSOREN1:R1.2, SENSOREN1:T1.C
- removed net RST1: PUI1:X4.4
- removed net RST2: ANSCHLUESSE-UNTEN1:X2.29
- removed net RX-B: BLUETOOTH1:IC1.2
- removed net RX-C: CAMERA1:X2.3
- removed net RX-P: PUI1:X3.P$3
- removed net SPEAKER-I: EIN/AUSGABE1:M1.1
- removed net SWITCH-O: EIN/AUSGABE1:S1.2
- removed net TEMP-O: SENSOREN1:IC1.2
- removed net TX-B: BLUETOOTH1:IC1.3
- removed net TX-C: CAMERA1:X2.4
- removed net TX-P: PUI1:X3.P$2
- new net 3V3: ANSCHLUESSE-UNTEN1:X2.1, ANSCHLUESSE-UNTEN1:X2.13, ANSCHLUESSE-UNTEN1:X2.5, ANSCHLUESSE-UNTEN1:X2.9, ARDUINO1:IC1.3.3V
- new net ANSCHLUSS: ANSCHLUESSE-UNTEN1:X2.19, ANSCHLUESSE-UNTEN1:X2.27, ANSCHLUESSE-UNTEN1:X2.28, ANSCHLUESSE-UNTEN1:X2.29, F4:F1.2, F4:R1.2
- new net ETC-12V: ANSCHLUESSE1:C2.1, ANSCHLUESSE1:X2.1, CAMERA1:C1.1, CAMERA1:J1.3, CAMERA1:X3.2, F6:F1.2, F6:R1.2, IR_SENDER1:R7.2, IR_SENDER1:R8.2
- new net ETC-5V: 5V-LINEARWANDLER1:C1.1, 5V-LINEARWANDLER1:IC1.2, ANSCHLUESSE1:C1.1, ANSCHLUESSE1:X1.1, ANSCHLUESSE1:X5.4, BLUETOOTH1:C1.1, BLUETOOTH1:IC1.5, EIN/AUSGABE1:R1.2, ENC1:IC1.VIN, IR-EMPFAENGER1:C1.1, IR-EMPFAENGER1:IC1.2, IR-EMPFAENGER1:IC2.2, IR-EMPFAENGER1:IC3.2, IR-EMPFAENGER1:IC4.2, IR-EMPFAENGER1:IC5.2, IR-EMPFAENGER1:IC6.2, IR_SENDER1:C1.1, IR_SENDER1:IC1.3, IR_SENDER1:R1.2, IR_SENDER1:R2.2, SENSOREN1:C1.1, SENSOREN1:C2.1, SENSOREN1:C3.1, SENSOREN1:C4.1, SENSOREN1:C5.1, SENSOREN1:C6.1, SENSOREN1:C7.1, SENSOREN1:C8.1, SENSOREN1:IC1.3, SENSOREN1:IC2.1, SENSOREN1:IC3.+, SENSOREN1:IC4.1, SENSOREN1:IC5.1, SENSOREN1:IC6.1, SENSOREN1:IC7.1, SENSOREN1:IC8.1, SENSOREN1:T1.A
- new net F2:N$1: F2:LED1.A, F2:R1.1
- new net F2:N$165: F2:LED1.C, F2:LED2.A
- new net F3:N$1: F3:LED1.A, F3:R1.1
- new net F3:N$165: F3:LED1.C, F3:LED2.A
- new net F4:N$1: F4:LED1.A, F4:R1.1
- new net F4:N$165: F4:LED1.C, F4:LED2.A
- new net F5:N$1: F5:LED1.A, F5:R1.1
- new net F5:N$165: F5:LED1.C, F5:LED2.A
- new net F6:N$1: F6:LED1.A, F6:R1.1
- new net F6:N$165: F6:LED1.C, F6:LED2.A
- new net INTERUPT-O: ARDUINO1:IC1.13
- new net KICK: F5:F1.2, F5:R1.2
- new net N$1: ARDUINO1:IC1.2, IR_SENDER1:IC1.5, IR_SENDER1:R1.1
- new net N$10: ANSCHLUESSE1:X4.1, ARDUINO1:IC1.10
- new net N$11: ARDUINO1:IC1.3, IR_SENDER1:IC1.6, IR_SENDER1:R2.1
- new net N$12: ARDUINO1:IC1.A7, SENSOREN1:R1.2, SENSOREN1:T1.C
- new net N$13: ARDUINO1:IC1.A8, SENSOREN1:IC1.2
- new net N$14: ARDUINO1:IC1.A6, SENSOREN1:R2.2
- new net N$15: ARDUINO1:IC1.4, SENSOREN1:X1.2
- new net N$16: ARDUINO1:IC1.22, BLUETOOTH1:IC1.2
- new net N$17: ARDUINO1:IC1.23, BLUETOOTH1:IC1.3
- new net N$18: ARDUINO1:IC1.17, BLUETOOTH1:IC1.6, BLUETOOTH1:R2.1
- new net N$19: ARDUINO1:IC1.16, BLUETOOTH1:IC1.1
- new net N$2: 5V-LINEARWANDLER2:C1.1, 5V-LINEARWANDLER2:IC1.2, CAMERA1:J1.1, CAMERA1:X2.2, CAMERA1:X2.5
- new net N$20: ARDUINO1:IC1.14, CAMERA1:X2.4
- new net N$21: ARDUINO1:IC1.15, CAMERA1:X2.3
- new net N$22: ARDUINO1:IC1.53, CAMERA1:X1.5
- new net N$23: ARDUINO1:IC1.52, CAMERA1:X1.3
- new net N$24: ARDUINO1:IC1.51, CAMERA1:X1.4
- new net N$25: ARDUINO1:IC1.50, CAMERA1:X1.1
- new net N$26: ARDUINO1:IC1.A0, IR-EMPFAENGER1:IC1.3
- new net N$27: ARDUINO1:IC1.A1, IR-EMPFAENGER1:IC2.3
- new net N$28: ARDUINO1:IC1.A2, IR-EMPFAENGER1:IC3.3
- new net N$29: ARDUINO1:IC1.A3, IR-EMPFAENGER1:IC4.3
- new net N$30: ARDUINO1:IC1.A4, IR-EMPFAENGER1:IC5.3
- new net N$31: ARDUINO1:IC1.A5, IR-EMPFAENGER1:IC6.3
- new net N$32: ARDUINO1:IC1.5, EIN/AUSGABE1:S1.2
- new net N$33: ARDUINO1:IC1.A9, EIN/AUSGABE1:M1.1
- new net N$34: ARDUINO1:IC1.9, EIN/AUSGABE1:R4.2
- new net N$35: ARDUINO1:IC1.8, EIN/AUSGABE1:R5.2
- new net N$36: ARDUINO1:IC1.7, EIN/AUSGABE1:R3.2
- new net N$37: ARDUINO1:IC1.6, EIN/AUSGABE1:LED1.C, EIN/AUSGABE1:R2.2
- new net N$38: ARDUINO1:IC1.VIN, F2:F1.2, F2:R1.2
- new net N$4: 5V-LINEARWANDLER4:C1.1, 5V-LINEARWANDLER4:IC1.2, PUI1:X3.P$1
- new net N$6: ARDUINO1:IC1.RESET, PUI1:X4.4
- new net N$7: ARDUINO1:IC1.19, PUI1:X3.P$3
- new net N$8: ARDUINO1:IC1.18, PUI1:X3.P$2
- new net N$9: ANSCHLUESSE1:X3.1, ARDUINO1:IC1.A10
- new net PUI: F3:F1.2, F3:R1.2, PUI1:X4.6
- net +12V: now also 5V-LINEARWANDLER2:C2.1, 5V-LINEARWANDLER2:IC1.1, 5V-LINEARWANDLER4:C2.1, 5V-LINEARWANDLER4:IC1.1, F2:F1.1, F3:F1.1, F4:F1.1, F5:F1.1, F6:F1.1; no longer ANSCHLUESSE-UNTEN1:X2.19, ANSCHLUESSE-UNTEN1:X2.27, ANSCHLUESSE-UNTEN1:X2.28, ANSCHLUESSE1:C2.1, ANSCHLUESSE1:X2.1, CAMERA1:C1.1, CAMERA1:J1.3, CAMERA1:X3.2, IR_SENDER1:R7.2, IR_SENDER1:R8.2, PUI1:X4.6
- net +5V: no longer 5V-LINEARWANDLER1:C1.1, 5V-LINEARWANDLER1:IC1.2, ANSCHLUESSE-UNTEN1:X2.1, ANSCHLUESSE-UNTEN1:X2.13, ANSCHLUESSE-UNTEN1:X2.5, ANSCHLUESSE-UNTEN1:X2.9, ANSCHLUESSE1:C1.1, ANSCHLUESSE1:X1.1, ANSCHLUESSE1:X5.4, BLUETOOTH1:C1.1, BLUETOOTH1:IC1.5, CAMERA1:J1.1, CAMERA1:X2.2, CAMERA1:X2.5, EIN/AUSGABE1:R1.2, ENC1:IC1.VIN, IR-EMPFAENGER1:C1.1, IR-EMPFAENGER1:IC1.2, IR-EMPFAENGER1:IC2.2, IR-EMPFAENGER1:IC3.2, IR-EMPFAENGER1:IC4.2, IR-EMPFAENGER1:IC5.2, IR-EMPFAENGER1:IC6.2, IR_SENDER1:C1.1, IR_SENDER1:IC1.3, IR_SENDER1:R1.2, IR_SENDER1:R2.2, PUI1:X3.P$1, SENSOREN1:C1.1, SENSOREN1:C2.1, SENSOREN1:C3.1, SENSOREN1:C4.1, SENSOREN1:C5.1, SENSOREN1:C6.1, SENSOREN1:C7.1, SENSOREN1:C8.1, SENSOREN1:IC1.3, SENSOREN1:IC2.1, SENSOREN1:IC3.+, SENSOREN1:IC4.1, SENSOREN1:IC5.1, SENSOREN1:IC6.1, SENSOREN1:IC7.1, SENSOREN1:IC8.1, SENSOREN1:T1.A
- net EN0: now also ARDUINO1:IC1.24
- net EN1: now also ARDUINO1:IC1.25
- net EN2: now also ARDUINO1:IC1.26
- net EN3: now also ARDUINO1:IC1.27
- net GND: now also 5V-LINEARWANDLER2:C1.2, 5V-LINEARWANDLER2:C2.2, 5V-LINEARWANDLER2:IC1.3, 5V-LINEARWANDLER4:C1.2, 5V-LINEARWANDLER4:C2.2, 5V-LINEARWANDLER4:IC1.3, ARDUINO1:IC1.GND@0, ARDUINO1:IC1.GND@1, ARDUINO1:IC1.GND@2, ARDUINO1:IC1.GND@3, ARDUINO1:IC1.GND@4, F2:LED2.C, F3:LED2.C, F4:LED2.C, F5:LED2.C, F6:LED2.C
- net I-MOTOR0: now also ARDUINO1:IC1.36
- net I-MOTOR1: now also ARDUINO1:IC1.37
- net I-MOTOR2: now also ARDUINO1:IC1.38
- net I-MOTOR3: now also ARDUINO1:IC1.39
- net INA0: now also ARDUINO1:IC1.28
- net INA1: now also ARDUINO1:IC1.30
- net INA2: now also ARDUINO1:IC1.32
- net INA3: now also ARDUINO1:IC1.34
- net INB0: now also ARDUINO1:IC1.29
- net INB1: now also ARDUINO1:IC1.31
- net INB2: now also ARDUINO1:IC1.33
- net INB3: now also ARDUINO1:IC1.35
- net KICK-EN: now also ARDUINO1:IC1.11
- net RGBLED-I: now also ARDUINO1:IC1.12
- net SCL: now also ARDUINO1:IC1.21
- net SDA: now also ARDUINO1:IC1.20

Commit message: + sch (layout beginning)
Parts:
- removed 5V-SCHALTREGLER1:C3: 100uF, 16V, ±20 %, iceberg20:CAPACITOR-THT-6.3
- removed 5V-SCHALTREGLER1:C4: 1000uF, 25V, ±20 %, iceberg20:CAPACITOR-THT-10
- removed 5V-SCHALTREGLER1:D1: 1N5822, iceberg20:DO-201AD
- removed 5V-SCHALTREGLER1:IC2: LM2576, iceberg20:TO220-5PIN
- removed 5V-SCHALTREGLER1:L1: L-100U, iceberg20:PISR
- removed 5V-SCHALTREGLER1:R1: 100k, iceberg20:R0805
- moved ARDUINO1:IC1 1327.3 mm to (209.6, -8.89), turned to 90 degrees
- moved EIN/AUSGABE1:S1 1243.2 mm to (262.9, -16.5)
- moved ANSCHLUESSE-UNTEN1:X2 1122.0 mm to (242.6, 14.0)
- moved SENSOREN1:IC7 1109.7 mm to (264.2, 69.8)
- moved SENSOREN1:IC6 1097.7 mm to (292.1, 21.6), turned to 270 degrees
- moved SENSOREN1:IC2 1049.4 mm to (284.5, -16.5)
- moved ANSCHLUESSE-UNTEN1:X1 1033.7 mm to (124.5, 39.4), turned to 270 degrees
- moved SENSOREN1:IC8 1027.7 mm to (149.9, 68.6)
- moved SENSOREN1:IC4 967.8 mm to (212.1, -64.8), turned to 180 degrees
- moved SENSOREN1:IC5 935.5 mm to (123.2, 10.2), turned to 90 degrees
- moved PUI1:X4 928.7 mm to (243.8, -22.9)
- moved PUI1:X3 913.4 mm to (245.1, -36.8)
- moved IR-EMPFAENGER1:IC1 907.5 mm to (285.8, -33.0)
- moved IR-EMPFAENGER1:IC2 885.2 mm to (266.7, -54.6)
- moved ENC1:IC1 883.2 mm to (259.1, 19.1)
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Connections:
- removed net 5V-SCHALTREGLER1:N$1: 5V-SCHALTREGLER1:IC2.5, 5V-SCHALTREGLER1:R1.1
- removed net 5V-SCHALTREGLER1:N$2: 5V-SCHALTREGLER1:D1.1, 5V-SCHALTREGLER1:IC2.2, 5V-SCHALTREGLER1:L1.1
- net +12V: no longer 5V-SCHALTREGLER1:C3.1, 5V-SCHALTREGLER1:IC2.1
- net +5V: no longer 5V-SCHALTREGLER1:C4.1, 5V-SCHALTREGLER1:IC2.4, 5V-SCHALTREGLER1:L1.2, 5V-SCHALTREGLER1:R1.2
- net GND: no longer 5V-SCHALTREGLER1:C3.2, 5V-SCHALTREGLER1:C4.2, 5V-SCHALTREGLER1:D1.2, 5V-SCHALTREGLER1:IC2.3
Routing:
- added copper zone on layer 16, net GND
Other:
- board size 160 x 100 mm -> 210 x 172.5 mm

Commit message: + sch (Bus Buffer)
Parts:
- added ANSCHLUESSE-UNTEN1:IC1: P82B96, iceberg20:SO8
- added ANSCHLUESSE-UNTEN1:R1, ANSCHLUESSE-UNTEN1:R2, ANSCHLUESSE-UNTEN1:R3, ANSCHLUESSE-UNTEN1:R4: 10k, iceberg20:R0805
Connections:
- new net ANSCHLUESSE-UNTEN1:RX(SDA): ANSCHLUESSE-UNTEN1:IC1.2, ANSCHLUESSE-UNTEN1:R3.1, ANSCHLUESSE-UNTEN1:X2.23
- new net ANSCHLUESSE-UNTEN1:RY(SCL): ANSCHLUESSE-UNTEN1:IC1.6, ANSCHLUESSE-UNTEN1:R4.1, ANSCHLUESSE-UNTEN1:X2.26
- new net ANSCHLUESSE-UNTEN1:TX(SDA): ANSCHLUESSE-UNTEN1:IC1.3, ANSCHLUESSE-UNTEN1:R2.1, ANSCHLUESSE-UNTEN1:X2.22
- new net ANSCHLUESSE-UNTEN1:TY(SCL): ANSCHLUESSE-UNTEN1:IC1.5, ANSCHLUESSE-UNTEN1:R1.1, ANSCHLUESSE-UNTEN1:X2.25
- net ANSCHLUSS: now also ANSCHLUESSE-UNTEN1:IC1.8, ANSCHLUESSE-UNTEN1:R1.2, ANSCHLUESSE-UNTEN1:R2.2, ANSCHLUESSE-UNTEN1:R3.2, ANSCHLUESSE-UNTEN1:R4.2
- net GND: now also ANSCHLUESSE-UNTEN1:IC1.4; no longer ANSCHLUESSE-UNTEN1:X2.22, ANSCHLUESSE-UNTEN1:X2.25
- net SCL: now also ANSCHLUESSE-UNTEN1:IC1.7; no longer ANSCHLUESSE-UNTEN1:X2.26
- net SDA: now also ANSCHLUESSE-UNTEN1:IC1.1; no longer ANSCHLUESSE-UNTEN1:X2.23
