File: iceberg20.brd (EAGLE design)
At the start: 210 x 172.5 mm, 215 parts, among them K1:C1 2,2 mF, 16 V, ±20 %, K1:D1 DIODE, K1:R1 300R, K1:R2 100k, K1:T1 IRF1405, M0:+ TPB1,27, M0:- TPB1,27, M0:C1 10nF, M0:C2 220nF, M0:C3 100nF, M0:C4 100uF, 16V, ±20 %, M0:C5 1nF, M0:C6 100nF, M0:D1 DIODE, M0:D2 DIODE, M0:EN TPB1,27, M0:I TPB1,27, M0:IC1 L6205N, M0:IC2 ACS712ACS712-SOIC-8, M0:IN1 TPB1,27, M0:IN2 TPB1,27, M0:R1 100R, M0:R2 100k, M0:R3 10k, M0:VS TPB1,27, M1:+ TPB1,27, M1:- TPB1,27, M1:C1 10nF, M1:C2 220nF, M1:C3 100nF, M1:C4 100uF, 16V, ±20 %, M1:C5 1nF, M1:C6 100nF, M1:D1 DIODE, M1:D2 DIODE, M1:EN TPB1,27, M1:I TPB1,27, M1:IC1 L6205N, M1:IC2 ACS712ACS712-SOIC-8, M1:IN1 TPB1,27, M1:IN2 TPB1,27, M1:R1 100R, M1:R2 100k, M1:R3 10k, M1:VS TPB1,27, M2:+ TPB1,27, M2:- TPB1,27, M2:C1 10nF, M2:C2 220nF, M2:C3 100nF, M2:C4 100uF, 16V, ±20 %, M2:C5 1nF, M2:C6 100nF, M2:D1 DIODE, M2:D2 DIODE, M2:EN TPB1,27, M2:I TPB1,27, M2:IC1 L6205N, M2:IC2 ACS712ACS712-SOIC-8, M2:IN1 TPB1,27, M2:IN2 TPB1,27, M2:R1 100R, M2:R2 100k, M2:R3 10k, M2:VS TPB1,27, M3:+ TPB1,27, M3:- TPB1,27, M3:C1 10nF, M3:C2 220nF, M3:C3 100nF, M3:C4 100uF, 16V, ±20 %, M3:C5 1nF, M3:C6 100nF, M3:D1 DIODE, M3:D2 DIODE, M3:EN TPB1,27, M3:I TPB1,27, M3:IC1 L6205N, M3:IC2 ACS712ACS712-SOIC-8, M3:IN1 TPB1,27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

Commit message: ~ sch (fix)
Parts:
- removed ANSCHLUESSE-UNTEN1:R3, ANSCHLUESSE-UNTEN1:R4: 10k, iceberg20:R0805
Connections:
- removed net ANSCHLUESSE-UNTEN1:RX(SDA): ANSCHLUESSE-UNTEN1:IC1.2, ANSCHLUESSE-UNTEN1:R3.1, ANSCHLUESSE-UNTEN1:X2.23
- removed net ANSCHLUESSE-UNTEN1:RY(SCL): ANSCHLUESSE-UNTEN1:IC1.6, ANSCHLUESSE-UNTEN1:R4.1, ANSCHLUESSE-UNTEN1:X2.26
- removed net ANSCHLUESSE-UNTEN1:TX(SDA): ANSCHLUESSE-UNTEN1:IC1.3, ANSCHLUESSE-UNTEN1:R2.1, ANSCHLUESSE-UNTEN1:X2.22
- removed net ANSCHLUESSE-UNTEN1:TY(SCL): ANSCHLUESSE-UNTEN1:IC1.5, ANSCHLUESSE-UNTEN1:R1.1, ANSCHLUESSE-UNTEN1:X2.25
- new net ANSCHLUESSE-UNTEN1:SCL-12V: ANSCHLUESSE-UNTEN1:IC1.5, ANSCHLUESSE-UNTEN1:IC1.6, ANSCHLUESSE-UNTEN1:R2.1, ANSCHLUESSE-UNTEN1:X2.26
- new net ANSCHLUESSE-UNTEN1:SDA-12V: ANSCHLUESSE-UNTEN1:IC1.2, ANSCHLUESSE-UNTEN1:IC1.3, ANSCHLUESSE-UNTEN1:R1.1, ANSCHLUESSE-UNTEN1:X2.23
- net ANSCHLUSS: no longer ANSCHLUESSE-UNTEN1:R3.2, ANSCHLUESSE-UNTEN1:R4.2
- net GND: now also ANSCHLUESSE-UNTEN1:X2.22, ANSCHLUESSE-UNTEN1:X2.25
Changed lines of the file:
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@@
 <attribute name="VALUE" x="-897.255" y="-812.8" size="1" layer="27" font="vector" ratio="20"/>
-</element>
-<element name="ANSCHLUESSE-UNTEN1:R3" library="iceberg20" package="R0805" package3d_urn="urn:adsk.eagle:package:23553/2" value="10k" x="-895.35" y="-816.61" smashed="yes">
-<attribute name="BESTAND" value="-" x="-895.35" y="-816.61" size="1.778" layer="27" display="off"/>
-<attribute name="HERSTELLER" value="-" x="-895.35" y="-816.61" size="1.778" layer="27" display="off"/>
-<attribute name="HERSTELLER-NR" value="-" x="-895.35" y="-816.61" size="1.778" layer="27" display="off"/>
-<attribute name="NAME" x="-897.255" y="-815.34" size="1" layer="25" font="vector" ratio="20"/>
-<attribute name="SUPPLIER" value="-" x="-895.35" y="-816.61" size="1.778" layer="27" display="off"/>
-<attribute name="SUPPLIER-NR" value="-" x="-895.35" y="-816.61" size="1.778" layer="27" display="off"/>
-<attribute name="TOLERANZ" value="5%" x="-895.35" y="-816.61" size="1.778" layer="27" display="off"/>
-<attribute name="VALUE" x="-897.255" y="-819.15" size="1" layer="27" font="vector" ratio="20"/>
-</element>
-<element name="ANSCHLUESSE-UNTEN1:R4" library="iceberg20" package="R0805" package3d_urn="urn:adsk.eagle:package:23553/2" value="10k" x="-895.35" y="-822.96" smashed="yes">
-<attribute name="BESTAND" value="-" x="-895.35" y="-822.96" size="1.778" layer="27" display="off"/>
-<attribute name="HERSTELLER" value="-" x="-895.35" y="-822.96" size="1.778" layer="27" display="off"/>
-<attribute name="HERSTELLER-NR" value="-" x="-895.35" y="-822.96" size="1.778" layer="27" display="off"/>
-<attribute name="NAME" x="-897.255" y="-821.69" size="1" layer="25" font="vector" ratio="20"/>
-<attribute name="SUPPLIER" value="-" x="-895.35" y="-822.96" size="1.778" layer="27" display="off"/>
-<attribute name="SUPPLIER-NR" value="-" x="-895.35" y="-822.96" size="1.778" layer="27" display="off"/>
-<attribute name="TOLERANZ" value="5%" x="-895.35" y="-822.96" size="1.778" layer="27" display="off"/>
-<attribute name="VALUE" x="-897.255" y="-825.5" size="1" layer="27" font="vector" ratio="20"/>
 </element>
 </elements>
@@
 <contactref element="BLUETOOTH1:IC1" pad="4"/>
 <contactref element="ANSCHLUESSE-UNTEN1:IC1" pad="4"/>
+<contactref element="ANSCHLUESSE-UNTEN1:X2" pad="22"/>
+<contactref element="ANSCHLUESSE-UNTEN1:X2" pad="25"/>
+<wire x1="243.84" y1="6.35" x2="243.84" y2="8.89" width="0" layer="19" extent="1-1"/>
+<wire x1="243.84" y1="3.81" x2="243.84" y2="6.35" width="0" layer="19" extent="1-1"/>
 <wire x1="241.3" y1="11.43" x2="243.84" y2="8.89" width="0" layer="19" extent="1-1"/>
+<wire x1="241.3" y1="1.27" x2="243.84" y2="3.81" width="0" layer="19" extent="1-1"/>
 <wire x1="243.84" y1="13.97" x2="241.3" y2="11.43" width="0" layer="19" extent="1-1"/>
-<wire x1="243.84" y1="3.81" x2="243.84" y2="8.89" width="0" layer="19" extent="1-1"/>
 <wire x1="243.84" y1="19.05" x2="243.84" y2="13.97" width="0" layer="19" extent="1-1"/>
 <wire x1="243.84" y1="24.13" x2="243.84" y2="19.05" width="0" layer="19" extent="1-1"/>
 <wire x1="243.84" y1="29.21" x2="243.84" y2="24.13" width="0" layer="19" extent="1-1"/>
-<wire x1="243.84" y1="-3.81" x2="243.84" y2="3.81" width="0" layer="19" extent="1-1"/>
-<wire x1="251.46" y1="5.08" x2="243.84" y2="3.81" width="0" layer="19" extent="1-1"/>
+<wire x1="243.84" y1="-3.81" x2="241.3" y2="1.27" width="0" layer="19" extent="1-1"/>
+<wire x1="251.46" y1="5.08" x2="243.84" y2="6.35" width="0" layer="19" extent="1-1"/>
 <wire x1="266.7" y1="2.54" x2="251.46" y2="5.08" width="0" layer="19" extent="1-1"/>
 <wire x1="259.08" y1="35.56" x2="243.84" y2="29.21" width="0" layer="19" extent="1-1"/>
@@
 <contactref element="ANSCHLUESSE-UNTEN1:R1" pad="2"/>
 <contactref element="ANSCHLUESSE-UNTEN1:R2" pad="2"/>
-<contactref element="ANSCHLUESSE-UNTEN1:R3" pad="2"/>
-<contactref element="ANSCHLUESSE-UNTEN1:R4" pad="2"/>
 <wire x1="241.3" y1="-1.27" x2="241.3" y2="8.89" width="0" layer="19" extent="1-1"/>
 <wire x1="243.84" y1="-1.27" x2="241.3" y2="-1.27" width="0" layer="19" extent="1-1"/>
@@
 <wire x1="-894.4" y1="-803.91" x2="-895.985" y2="-791.15" width="0" layer="19" extent="1-1"/>
 <wire x1="-894.4" y1="-810.26" x2="-894.4" y2="-803.91" width="0" layer="19" extent="1-1"/>
-<wire x1="-894.4" y1="-816.61" x2="-894.4" y2="-810.26" width="0" layer="19" extent="1-1"/>
-<wire x1="-894.4" y1="-822.96" x2="-894.4" y2="-816.61" width="0" layer="19" extent="1-1"/>
 </signal>
 <signal name="KICK">
@@
 <wire x1="232.41" y1="-15.24" x2="-835.98" y2="-654.05" width="0" layer="19" extent="1-1"/>
 </signal>
-<signal name="ANSCHLUESSE-UNTEN1:TY(SCL)">
-<contactref element="ANSCHLUESSE-UNTEN1:X2" pad="25"/>
-<contactref element="ANSCHLUESSE-UNTEN1:IC1" pad="5"/>
-<contactref element="ANSCHLUESSE-UNTEN1:R1" pad="1"/>
-<wire x1="-896.3" y1="-803.91" x2="241.3" y2="1.27" width="0" layer="19" extent="1-1"/>
-<wire x1="-892.175" y1="-791.15" x2="-896.3" y2="-803.91" width="0" layer="19" extent="1-1"/>
-</signal>
-<signal name="ANSCHLUESSE-UNTEN1:TX(SDA)">
-<contactref element="ANSCHLUESSE-UNTEN1:X2" pad="22"/>
-<contactref element="ANSCHLUESSE-UNTEN1:IC1" pad="3"/>
-<contactref element="ANSCHLUESSE-UNTEN1:R2" pad="1"/>
-<wire x1="-896.3" y1="-810.26" x2="243.84" y2="6.35" width="0" layer="19" extent="1-1"/>
-<wire x1="-893.445" y1="-796.35" x2="-896.3" y2="-810.26" width="0" layer="19" extent="1-1"/>
-</signal>
-<signal name="ANSCHLUESSE-UNTEN1:RY(SCL)">
-<contactref element="ANSCHLUESSE-UNTEN1:X2" pad="26"/>
-<contactref element="ANSCHLUESSE-UNTEN1:IC1" pad="6"/>
-<contactref element="ANSCHLUESSE-UNTEN1:R4" pad="1"/>
-<wire x1="-896.3" y1="-822.96" x2="243.84" y2="1.27" width="0" layer="19" extent="1-1"/>
-<wire x1="-893.445" y1="-791.15" x2="-896.3" y2="-822.96" width="0" layer="19" extent="1-1"/>
-</signal>
-<signal name="ANSCHLUESSE-UNTEN1:RX(SDA)">
+<signal name="ANSCHLUESSE-UNTEN1:SDA-12V">
 <contactref element="ANSCHLUESSE-UNTEN1:X2" pad="23"/>
 <contactref element="ANSCHLUESSE-UNTEN1:IC1" pad="2"/>
-<contactref element="ANSCHLUESSE-UNTEN1:R3" pad="1"/>
-<wire x1="-896.3" y1="-816.61" x2="241.3" y2="3.81" width="0" layer="19" extent="1-1"/>
-<wire x1="-894.715" y1="-796.35" x2="-896.3" y2="-816.61" width="0" layer="19" extent="1-1"/>
+<contactref element="ANSCHLUESSE-UNTEN1:R1" pad="1"/>
+<contactref element="ANSCHLUESSE-UNTEN1:IC1" pad="3"/>
+<wire x1="-896.3" y1="-803.91" x2="241.3" y2="3.81" width="0" layer="19" extent="1-1"/>
+<wire x1="-894.715" y1="-796.35" x2="-896.3" y2="-803.91" width="0" layer="19" extent="1-1"/>
+<wire x1="-893.445" y1="-796.35" x2="-894.715" y2="-796.35" width="0" layer="19" extent="1-1"/>
+</signal>
+<signal name="ANSCHLUESSE-UNTEN1:SCL-12V">
+<contactref element="ANSCHLUESSE-UNTEN1:X2" pad="26"/>
+<contactref element="ANSCHLUESSE-UNTEN1:IC1" pad="5"/>
+<contactref element="ANSCHLUESSE-UNTEN1:IC1" pad="6"/>
+<contactref element="ANSCHLUESSE-UNTEN1:R2" pad="1"/>
+<wire x1="-896.3" y1="-810.26" x2="243.84" y2="1.27" width="0" layer="19" extent="1-1"/>
+<wire x1="-893.445" y1="-791.15" x2="-896.3" y2="-810.26" width="0" layer="19" extent="1-1"/>
+<wire x1="-892.175" y1="-791.15" x2="-893.445" y2="-791.15" width="0" layer="19" extent="1-1"/>
 </signal>
 </signals>
