File: iceberg20.brd (EAGLE design)
At the start: 210 x 172.5 mm, 213 parts, among them K1:C1 2,2 mF, 16 V, ±20 %, K1:D1 DIODE, K1:R1 300R, K1:R2 100k, K1:T1 IRF1405, M0:+ TPB1,27, M0:- TPB1,27, M0:C1 10nF, M0:C2 220nF, M0:C3 100nF, M0:C4 100uF, 16V, ±20 %, M0:C5 1nF, M0:C6 100nF, M0:D1 DIODE, M0:D2 DIODE, M0:EN TPB1,27, M0:I TPB1,27, M0:IC1 L6205N, M0:IC2 ACS712ACS712-SOIC-8, M0:IN1 TPB1,27, M0:IN2 TPB1,27, M0:R1 100R, M0:R2 100k, M0:R3 10k, M0:VS TPB1,27, M1:+ TPB1,27, M1:- TPB1,27, M1:C1 10nF, M1:C2 220nF, M1:C3 100nF, M1:C4 100uF, 16V, ±20 %, M1:C5 1nF, M1:C6 100nF, M1:D1 DIODE, M1:D2 DIODE, M1:EN TPB1,27, M1:I TPB1,27, M1:IC1 L6205N, M1:IC2 ACS712ACS712-SOIC-8, M1:IN1 TPB1,27, M1:IN2 TPB1,27, M1:R1 100R, M1:R2 100k, M1:R3 10k, M1:VS TPB1,27, M2:+ TPB1,27, M2:- TPB1,27, M2:C1 10nF, M2:C2 220nF, M2:C3 100nF, M2:C4 100uF, 16V, ±20 %, M2:C5 1nF, M2:C6 100nF, M2:D1 DIODE, M2:D2 DIODE, M2:EN TPB1,27, M2:I TPB1,27, M2:IC1 L6205N, M2:IC2 ACS712ACS712-SOIC-8, M2:IN1 TPB1,27, M2:IN2 TPB1,27, M2:R1 100R, M2:R2 100k, M2:R3 10k, M2:VS TPB1,27, M3:+ TPB1,27, M3:- TPB1,27, M3:C1 10nF, M3:C2 220nF, M3:C3 100nF, M3:C4 100uF, 16V, ±20 %, M3:C5 1nF, M3:C6 100nF, M3:D1 DIODE, M3:D2 DIODE, M3:EN TPB1,27, M3:I TPB1,27, M3:IC1 L6205N, M3:IC2 ACS712ACS712-SOIC-8, M3:IN1 TPB1,27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

Commit message: ~ sch (alles überarbeitet)
A3 Rahmen hat auch nicht gepasst, bibliotheken updaten?
Connections:
- net 3V3 renamed +3V3
- net EN0 renamed M-EN0
- net EN1 renamed M-EN1
- net EN2 renamed M-EN2
- net EN3 renamed M-EN3
- net I-MOTOR0 renamed I-M0
- net I-MOTOR1 renamed I-M1
- net INA0 renamed M-DIR-A0
- net INA1 renamed M-DIR-A1
- net INA2 renamed M-DIR-A2
- net INA3 renamed M-DIR-A3
- net INB0 renamed M-DIR-B0
- net INB1 renamed M-DIR-B1
- net INB2 renamed M-DIR-B2
- net INB3 renamed M-DIR-B3
- net MOTOR-SUPPLY renamed MOTOR-12V
- net N$1 renamed IR-EN1
- net N$10 renamed D1
- net N$11 renamed IR-EN2
- net N$12 renamed PHOTO
- net N$13 renamed TEMP
- net N$2 renamed 5V-CAMERA
- net N$20 renamed TX-C
- net N$21 renamed RX-C
- net N$22 renamed CS
- net N$23 renamed CLK
- net N$24 renamed MOSI
- net N$25 renamed MISO
- net N$32 renamed SWITCH
- net N$33 renamed SPEAKER
- net N$34 renamed LED3
- net N$35 renamed LED2
- net N$36 renamed LED1
- net N$37 renamed HEARTBEAT
- net N$4 renamed 5V-PUI
- net N$6 renamed RESET
- net N$7 renamed RX-P
- net N$8 renamed TX-P
- net N$9 renamed A1
- net RGBLED-I renamed RGBLED
- removed net ANSCHLUSS: ANSCHLUESSE-UNTEN1:IC1.8, ANSCHLUESSE-UNTEN1:R1.2, ANSCHLUESSE-UNTEN1:R2.2, ANSCHLUESSE-UNTEN1:X2.19, ANSCHLUESSE-UNTEN1:X2.27, ANSCHLUESSE-UNTEN1:X2.28, ANSCHLUESSE-UNTEN1:X2.29, F4:F1.2, F4:R1.2
- removed net ETC-5V: 5V-LINEARWANDLER1:C1.1, 5V-LINEARWANDLER1:IC1.2, ANSCHLUESSE1:C1.1, ANSCHLUESSE1:X1.1, ANSCHLUESSE1:X5.4, BLUETOOTH1:C1.1, BLUETOOTH1:IC1.5, EIN/AUSGABE1:R1.2, ENC1:IC1.VIN, IR-EMPFAENGER1:C1.1, IR-EMPFAENGER1:IC1.2, IR-EMPFAENGER1:IC2.2, IR-EMPFAENGER1:IC3.2, IR-EMPFAENGER1:IC4.2, IR-EMPFAENGER1:IC5.2, IR-EMPFAENGER1:IC6.2, IR_SENDER1:C1.1, IR_SENDER1:IC1.3, IR_SENDER1:R1.2, IR_SENDER1:R2.2, SENSOREN1:C1.1, SENSOREN1:C2.1, SENSOREN1:C3.1, SENSOREN1:C4.1, SENSOREN1:C5.1, SENSOREN1:C6.1, SENSOREN1:C7.1, SENSOREN1:C8.1, SENSOREN1:IC1.3, SENSOREN1:IC2.1, SENSOREN1:IC3.+, SENSOREN1:IC4.1, SENSOREN1:IC5.1, SENSOREN1:IC6.1, SENSOREN1:IC7.1, SENSOREN1:IC8.1, SENSOREN1:T1.A
- removed net I-MOTOR2: ARDUINO1:IC1.38, M2:I.TP, M2:IC2.7
- removed net I-MOTOR3: ARDUINO1:IC1.39, M3:I.TP, M3:IC2.7
- removed net INTERRUPT-O: ANSCHLUESSE-UNTEN1:X2.18
- removed net INTERUPT-O: ARDUINO1:IC1.13
- removed net N$14: ARDUINO1:IC1.A6, SENSOREN1:R2.2
- removed net N$15: ARDUINO1:IC1.4, SENSOREN1:X1.2
- removed net N$16: ARDUINO1:IC1.22, BLUETOOTH1:IC1.2
- removed net N$17: ARDUINO1:IC1.23, BLUETOOTH1:IC1.3
- removed net N$18: ARDUINO1:IC1.17, BLUETOOTH1:IC1.6, BLUETOOTH1:R2.1
- removed net N$19: ARDUINO1:IC1.16, BLUETOOTH1:IC1.1
- removed net N$26: ARDUINO1:IC1.A0, IR-EMPFAENGER1:IC1.3
- removed net N$27: ARDUINO1:IC1.A1, IR-EMPFAENGER1:IC2.3
- removed net N$28: ARDUINO1:IC1.A2, IR-EMPFAENGER1:IC3.3
- removed net N$29: ARDUINO1:IC1.A3, IR-EMPFAENGER1:IC4.3
- removed net N$3: ANSCHLUESSE-UNTEN1:X1.9, K1:D1.2, K1:T1.2
- removed net N$30: ARDUINO1:IC1.A4, IR-EMPFAENGER1:IC5.3
- removed net N$31: ARDUINO1:IC1.A5, IR-EMPFAENGER1:IC6.3
- removed net N$5: ANSCHLUESSE-UNTEN1:X1.10, K1:C1.1, K1:D1.1
- removed net PUI: F3:F1.2, F3:R1.2, PUI1:X4.6
- new net 12V-PUI: 5V-LINEARWANDLER4:C2.1, 5V-LINEARWANDLER4:IC1.1, F3:F1.2, F3:R1.2, PUI1:X4.6
- new net ANSCHLUSS-12V: ANSCHLUESSE-UNTEN1:IC1.8, ANSCHLUESSE-UNTEN1:R1.2, ANSCHLUESSE-UNTEN1:R2.2, ANSCHLUESSE-UNTEN1:X2.19, ANSCHLUESSE-UNTEN1:X2.27, ANSCHLUESSE-UNTEN1:X2.28, F4:F1.2, F4:R1.2
- new net ARDUINO1:IR-SIG1: ARDUINO1:IC1.A0
- new net ARDUINO1:IR-SIG2: ARDUINO1:IC1.A1
- new net ARDUINO1:IR-SIG3: ARDUINO1:IC1.A2
- new net ARDUINO1:IR-SIG4: ARDUINO1:IC1.A3
- new net ARDUINO1:IR-SIG5: ARDUINO1:IC1.A4
- new net ARDUINO1:IR-SIG6: ARDUINO1:IC1.A5
- new net BR-I: ARDUINO1:IC1.A6, SENSOREN1:X1.2
- new net BR-LED: ARDUINO1:IC1.4, SENSOREN1:R2.2
- new net EN-B: ARDUINO1:IC1.22, BLUETOOTH1:IC1.6, BLUETOOTH1:R2.1
- new net I-M2: M2:I.TP, M2:IC2.7
- new net I-M3: ARDUINO1:IC1.38, ARDUINO1:IC1.39, M3:I.TP, M3:IC2.7
- new net INTERRUPT: ANSCHLUESSE-UNTEN1:X2.18, ARDUINO1:IC1.13
- new net IR-EMPFAENGER1:IR-SIG1: IR-EMPFAENGER1:IC1.3
- new net IR-EMPFAENGER1:IR-SIG2: IR-EMPFAENGER1:IC2.3
- new net IR-EMPFAENGER1:IR-SIG3: IR-EMPFAENGER1:IC3.3
- new net IR-EMPFAENGER1:IR-SIG4: IR-EMPFAENGER1:IC4.3
- new net IR-EMPFAENGER1:IR-SIG5: IR-EMPFAENGER1:IC5.3
- new net IR-EMPFAENGER1:IR-SIG6: IR-EMPFAENGER1:IC6.3
- new net KICK+: ANSCHLUESSE-UNTEN1:X1.9, K1:C1.1, K1:D1.1
- new net KICK-: ANSCHLUESSE-UNTEN1:X1.10, K1:D1.2, K1:T1.2
- new net MOTORSTROM:I-M0: ARDUINO1:IC1.36
- new net MOTORSTROM:I-M1: ARDUINO1:IC1.37
- new net MOTORSTROM:I-M3: ARDUINO1:IC1.38, ARDUINO1:IC1.39
- new net RST-NANO: ANSCHLUESSE-UNTEN1:X2.29, ARDUINO1:IC1.40
- new net RX-B: ARDUINO1:IC1.17, BLUETOOTH1:IC1.3
- new net STATE-B: ARDUINO1:IC1.23, BLUETOOTH1:IC1.1
- new net TX-B: ARDUINO1:IC1.16, BLUETOOTH1:IC1.2
- net +12V: no longer 5V-LINEARWANDLER1:C2.1, 5V-LINEARWANDLER1:IC1.1, 5V-LINEARWANDLER2:C2.1, 5V-LINEARWANDLER2:IC1.1, 5V-LINEARWANDLER4:C2.1, 5V-LINEARWANDLER4:IC1.1
- net +5V: now also 5V-LINEARWANDLER1:C1.1, 5V-LINEARWANDLER1:IC1.2, ANSCHLUESSE1:C1.1, ANSCHLUESSE1:X1.1, ANSCHLUESSE1:X5.4, BLUETOOTH1:C1.1, BLUETOOTH1:IC1.5, EIN/AUSGABE1:R1.2, ENC1:IC1.VIN, IR-EMPFAENGER1:C1.1, IR-EMPFAENGER1:IC1.2, IR-EMPFAENGER1:IC2.2, IR-EMPFAENGER1:IC3.2, IR-EMPFAENGER1:IC4.2, IR-EMPFAENGER1:IC5.2, IR-EMPFAENGER1:IC6.2, IR_SENDER1:C1.1, IR_SENDER1:IC1.3, IR_SENDER1:R1.2, IR_SENDER1:R2.2, SENSOREN1:C1.1, SENSOREN1:C2.1, SENSOREN1:C3.1, SENSOREN1:C4.1, SENSOREN1:C5.1, SENSOREN1:C6.1, SENSOREN1:C7.1, SENSOREN1:C8.1, SENSOREN1:IC1.3, SENSOREN1:IC2.1, SENSOREN1:IC3.+, SENSOREN1:IC4.1, SENSOREN1:IC5.1, SENSOREN1:IC6.1, SENSOREN1:IC7.1, SENSOREN1:IC8.1, SENSOREN1:T1.A
- net ETC-12V: now also 5V-LINEARWANDLER1:C2.1, 5V-LINEARWANDLER1:IC1.1, 5V-LINEARWANDLER2:C2.1, 5V-LINEARWANDLER2:IC1.1

Commit message: ~ brd (reset)
Parts:
- removed BLUETOOTH1:R2: 100k, iceberg20:R0805
- removed EIN/AUSGABE1:LED6: LED-WHITE, iceberg20:PLCC-2
- removed P1:U$1: TERMINAL-2, iceberg20:LIB_WECO121
- added ARDUINO1:R1, ARDUINO1:R2: 1k, iceberg20:R0805
- added ARDUINO1:R3, ARDUINO1:R4: 100k, iceberg20:R0805
- added ARDUINO1:TP1, ARDUINO1:TP2: TESTPAD, iceberg20:TESTPAD_B2,54
- added EIN/AUSGABE1:LED5, ENC1:LED1, ENC1:LED2, ENC1:LED3, ENC1:LED4: LED-WHITE, iceberg20:PLCC-2
- added ENC1:R1, ENC1:R2, ENC1:R3, ENC1:R4: 120R, iceberg20:R0805
- added IR-EMPFAENGER1:C2, IR-EMPFAENGER1:C3, IR-EMPFAENGER1:C4, IR-EMPFAENGER1:C5, IR-EMPFAENGER1:C6: 100n, iceberg20:C0805
- added P1:X1: TERMINAL-2, iceberg20:LIB_WECO121
- EIN/AUSGABE1:R1, EIN/AUSGABE1:R2, IR_SENDER1:R3, IR_SENDER1:R5: value 100 -> 100R
- F1:R1, F2:R1, F3:R1, F4:R1, F5:R1, F6:R1: value 270 -> 270R
- IR_SENDER1:R7, IR_SENDER1:R8: value 15 -> 15R
- M0:+, M0:-, M0:EN, M0:I, M0:IN1, M0:IN2, M0:VS, M1:+, M1:-, M1:EN, M1:I, M1:IN1, M1:IN2, M1:VS, M2:+, M2:-, M2:EN, M2:I, M2:IN1, M2:IN2, M2:VS, M3:+, M3:-, M3:EN, M3:I, M3:IN1, M3:IN2, M3:VS: value TPB1,27 -> TESTPAD; device testpad:B1,27 -> iceberg20:TESTPAD_B2,54
- moved 5V-LINEARWANDLER4:IC1 1331.3 mm to (-163.8, 339.1)
- moved 5V-LINEARWANDLER4:C1 1326.6 mm to (-182.9, 336.6)
- moved F4:F1 1325.1 mm to (-25.4, 367.0)
- moved 5V-LINEARWANDLER2:IC1 1322.8 mm to (-108.0, 339.1)
- moved 5V-LINEARWANDLER4:C2 1322.7 mm to (-200.7, 336.6)
- moved F4:LED1 1322.5 mm to (-45.7, 363.2)
- moved F4:R1 1322.4 mm to (-62.2, 363.2)
- moved F4:LED2 1320.2 mm to (-55.9, 363.2)
- moved 5V-LINEARWANDLER2:C1 1317.0 mm to (-127.0, 336.6)
- moved F5:F1 1315.6 mm to (-77.5, 367.0)
- moved F5:R1 1313.4 mm to (-114.3, 363.2)
- moved F5:LED1 1313.1 mm to (-97.8, 363.2)
- moved 5V-LINEARWANDLER2:C2 1312.1 mm to (-144.8, 336.6)
- moved F5:LED2 1310.9 mm to (-108.0, 363.2)
- moved F6:F1 1307.5 mm to (-129.5, 367.0)
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Connections:
- removed net +3V3: ANSCHLUESSE-UNTEN1:X2.1, ANSCHLUESSE-UNTEN1:X2.13, ANSCHLUESSE-UNTEN1:X2.5, ANSCHLUESSE-UNTEN1:X2.9, ARDUINO1:IC1.3.3V
- removed net ARDUINO1:IR-SIG1: ARDUINO1:IC1.A0
- removed net ARDUINO1:IR-SIG2: ARDUINO1:IC1.A1
- removed net ARDUINO1:IR-SIG3: ARDUINO1:IC1.A2
- removed net ARDUINO1:IR-SIG4: ARDUINO1:IC1.A3
- removed net ARDUINO1:IR-SIG5: ARDUINO1:IC1.A4
- removed net ARDUINO1:IR-SIG6: ARDUINO1:IC1.A5
- removed net IR-EMPFAENGER1:IR-SIG1: IR-EMPFAENGER1:IC1.3
- removed net IR-EMPFAENGER1:IR-SIG2: IR-EMPFAENGER1:IC2.3
- removed net IR-EMPFAENGER1:IR-SIG3: IR-EMPFAENGER1:IC3.3
- removed net IR-EMPFAENGER1:IR-SIG4: IR-EMPFAENGER1:IC4.3
- removed net IR-EMPFAENGER1:IR-SIG5: IR-EMPFAENGER1:IC5.3
- removed net IR-EMPFAENGER1:IR-SIG6: IR-EMPFAENGER1:IC6.3
- removed net M0:N$1: M0:IC1.13
- removed net M0:N$2: M0:IC1.7
- removed net M1:N$1: M1:IC1.13
- removed net M1:N$2: M1:IC1.7
- removed net M2:N$1: M2:IC1.13
- removed net M2:N$2: M2:IC1.7
- removed net M3:N$1: M3:IC1.13
- removed net M3:N$2: M3:IC1.7
- removed net MOTORSTROM:I-M0: ARDUINO1:IC1.36
- removed net MOTORSTROM:I-M1: ARDUINO1:IC1.37
- removed net MOTORSTROM:I-M3: ARDUINO1:IC1.38, ARDUINO1:IC1.39
- new net ARDUINO1:+5V: ARDUINO1:IC1.5V@0, ARDUINO1:IC1.5V@1, ARDUINO1:IC1.5V@2, ARDUINO1:R1.2, ARDUINO1:R2.2, ARDUINO1:R3.2, ARDUINO1:R4.2
- new net ARDUINO1:N$1: ARDUINO1:IC1.A11, ARDUINO1:TP2.TP
- new net ARDUINO1:N$2: ARDUINO1:IC1.24, ARDUINO1:TP1.TP
- new net ENC1:LED1: ENC1:IC1.20, ENC1:R1.2
- new net ENC1:LED2: ENC1:IC1.21, ENC1:R2.2
- new net ENC1:LED3: ENC1:IC1.22, ENC1:R3.2
- new net ENC1:LED4: ENC1:IC1.23, ENC1:R4.2
- new net ENC1:N$3: ENC1:LED1.A, ENC1:R1.1
- new net ENC1:N$4: ENC1:LED2.A, ENC1:R2.1
- new net ENC1:N$5: ENC1:LED3.A, ENC1:R3.1
- new net ENC1:N$8: ENC1:LED4.A, ENC1:R4.1
- new net IR-SIG1: ARDUINO1:IC1.A0, IR-EMPFAENGER1:IC1.3
- new net IR-SIG2: ARDUINO1:IC1.A1, IR-EMPFAENGER1:IC2.3
- new net IR-SIG3: ARDUINO1:IC1.A2, IR-EMPFAENGER1:IC3.3
- new net IR-SIG4: ARDUINO1:IC1.A3, IR-EMPFAENGER1:IC4.3
- new net IR-SIG5: ARDUINO1:IC1.A4, IR-EMPFAENGER1:IC5.3
- new net IR-SIG6: ARDUINO1:IC1.A5, IR-EMPFAENGER1:IC6.3
- net +5V: now also ANSCHLUESSE-UNTEN1:X2.1, ANSCHLUESSE-UNTEN1:X2.13, ANSCHLUESSE-UNTEN1:X2.5, ANSCHLUESSE-UNTEN1:X2.9, IR-EMPFAENGER1:C2.1, IR-EMPFAENGER1:C3.1, IR-EMPFAENGER1:C4.1, IR-EMPFAENGER1:C5.1, IR-EMPFAENGER1:C6.1, SENSOREN1:R1.2; no longer SENSOREN1:T1.A
- net BR-LED: now also ARDUINO1:IC1.A9; no longer ARDUINO1:IC1.4
- net D1: now also ARDUINO1:IC1.43; no longer ARDUINO1:IC1.10
- net EIN/AUSGABE1:N$4: now also EIN/AUSGABE1:LED4.A; no longer EIN/AUSGABE1:LED6.A
- net EIN/AUSGABE1:N$5: now also EIN/AUSGABE1:LED5.A; no longer EIN/AUSGABE1:LED4.A
- net EN-B: no longer BLUETOOTH1:R2.1
- net ENA1: now also ANSCHLUESSE-UNTEN1:X2.6; no longer ANSCHLUESSE-UNTEN1:X2.7
- net ENB1: now also ANSCHLUESSE-UNTEN1:X2.7; no longer ANSCHLUESSE-UNTEN1:X2.6
- net GND: now also EIN/AUSGABE1:LED5.C, ENC1:LED1.C, ENC1:LED2.C, ENC1:LED3.C, ENC1:LED4.C, IR-EMPFAENGER1:C2.2, IR-EMPFAENGER1:C3.2, IR-EMPFAENGER1:C4.2, IR-EMPFAENGER1:C5.2, IR-EMPFAENGER1:C6.2, P1:X1.P1, SENSOREN1:T1.C; no longer BLUETOOTH1:R2.2, EIN/AUSGABE1:LED6.C, P1:U$1.P1, SENSOREN1:R1.1
- net HEARTBEAT: now also ARDUINO1:IC1.3; no longer ARDUINO1:IC1.6
- net INTERRUPT: now also ARDUINO1:IC1.2, ARDUINO1:R4.1; no longer ARDUINO1:IC1.13
- net IR-EN1: now also ARDUINO1:IC1.41; no longer ARDUINO1:IC1.2
- net IR-EN2: now also ARDUINO1:IC1.42; no longer ARDUINO1:IC1.3
- net KICK-EN: now also ARDUINO1:IC1.8; no longer ARDUINO1:IC1.11
- net LED1: now also ARDUINO1:IC1.5; no longer ARDUINO1:IC1.7
- net LED2: now also ARDUINO1:IC1.6; no longer ARDUINO1:IC1.8
- net LED3: now also ARDUINO1:IC1.7; no longer ARDUINO1:IC1.9
- net M-EN0: now also ARDUINO1:IC1.10; no longer ARDUINO1:IC1.24
- net M-EN1: now also ARDUINO1:IC1.11; no longer ARDUINO1:IC1.25
- net M-EN2: now also ARDUINO1:IC1.12; no longer ARDUINO1:IC1.26
- net M-EN3: now also ARDUINO1:IC1.13; no longer ARDUINO1:IC1.27
- net M0:M-: now also M0:IC1.13
- net M1:M-: now also M1:IC1.13
- net M2:M-: now also M2:IC1.13
- net M3:M-: now also M3:IC1.13
- net MB0: now also M0:IC1.7
- net MB1: now also M1:IC1.7
- net MB2: now also M2:IC1.7
- net MB3: now also M3:IC1.7
- net P1:N$1: now also P1:X1.P2; no longer P1:U$1.P2
- net PHOTO: now also SENSOREN1:R1.1, SENSOREN1:T1.A; no longer SENSOREN1:R1.2, SENSOREN1:T1.C
- net RESET: now also ARDUINO1:R3.1
- net RGBLED: now also ARDUINO1:IC1.9; no longer ARDUINO1:IC1.12
- net SCL: now also ARDUINO1:R2.1
- net SDA: now also ARDUINO1:R1.1
- net SPEAKER: now also ARDUINO1:IC1.4; no longer ARDUINO1:IC1.A9
- net SWITCH: now also ARDUINO1:IC1.49; no longer ARDUINO1:IC1.5
Routing:
- removed copper zone on layer 16, net GND
Other:
- board size 210 x 172.5 mm -> 160 x 100 mm
