File: nano19.sch (EAGLE design)
At the start: 5 parts, among them J3 JUMPER-JP-2, J4 JUMPER-JP-2

Commit message: - nano.brd (Routing + Layout + Text)
Connections:
- removed net LED: X1.14
Other:
- note added: "NANO"
Changed lines of the file:
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@@
 <sheet>
 <plain>
+<text x="217.17" y="20.32" size="2.54" layer="94">NANO</text>
 </plain>
 <instances>
@@
 </segment>
 </net>
-<net name="LED" class="0">
-<segment>
-<pinref part="X1" gate="G$1" pin="14"/>
-<wire x1="109.22" y1="134.62" x2="111.76" y2="134.62" width="0.1524" layer="91"/>
-<label x="111.76" y="134.62" size="1.778" layer="95"/>
-</segment>
-</net>
