File: pui20.brd (EAGLE design)
At the start: 95 x 30 mm, 32 parts

Commit message: + pui.brd (Display)
Parts:
- removed EXPANDER1:C1: 200nF, iceberg20:C0805
- removed EXPANDER1:R1: 1k, iceberg20:R0805
- added DISPLAY1:GND, DISPLAY1:RX, DISPLAY1:TX, DISPLAY1:VIN: TESTPAD-LONG, iceberg20:TESTPAD-LONG
- added EXP:C1: 200nF, iceberg20:C0805
- added EXP:R1: 1k, iceberg20:R0805
- added IC1: L7805, iceberg20:TO220V
- renumbered ANSCHLUSS1:X1 to X:X1, AUSGABE1:LED1 to OUT:LED1, AUSGABE1:LED10 to OUT:LED10, AUSGABE1:LED11 to OUT:LED11, AUSGABE1:LED12 to OUT:LED12, AUSGABE1:LED2 to OUT:LED2, AUSGABE1:LED3 to OUT:LED3, AUSGABE1:LED4 to OUT:LED4, AUSGABE1:LED5 to OUT:LED5, AUSGABE1:LED6 to OUT:LED6, AUSGABE1:LED7 to OUT:LED7, AUSGABE1:LED8 to OUT:LED8, AUSGABE1:LED9 to OUT:LED9, AUSGABE1:R1 to OUT:R1, AUSGABE1:R2 to OUT:R2, AUSGABE1:R3 to OUT:R3, AUSGABE1:R4 to OUT:R4, AUSGABE1:R5 to OUT:R5, AUSGABE1:R6 to OUT:R6, EINGABE1:S1 to IN:S1, EINGABE1:S2 to IN:S2, EINGABE1:S3 to IN:S3, EINGABE1:S4 to IN:S4, EINGABE1:S5 to IN:S5, EINGABE1:S6 to IN:S6, EINGABE1:S7 to IN:S7, EINGABE1:S8 to IN:S8, EINGABE1:S9 to IN:S9, EINGABE1:U$1 to IN:U$1, EXPANDER1:IC1 to EXP:IC1
Connections:
- net ANSCHLUSS1:INTERRUPT renamed X:INTERRUPT
- net AUSGABE1:N$1 renamed OUT:N$1
- net AUSGABE1:N$11 renamed OUT:N$11
- net AUSGABE1:N$12 renamed OUT:N$12
- net AUSGABE1:N$2 renamed OUT:N$2
- net AUSGABE1:N$3 renamed OUT:N$3
- net AUSGABE1:N$4 renamed OUT:N$4
- net AUSGABE1:N$5 renamed OUT:N$5
- net AUSGABE1:N$6 renamed OUT:N$6
- net AUSGABE1:N$7 renamed OUT:N$7
- net AUSGABE1:N$8 renamed OUT:N$8
- net AUSGABE1:N$9 renamed OUT:N$9
- net EXPANDER1:A0 renamed EXP:A0
- net EXPANDER1:A1 renamed EXP:A1
- net EXPANDER1:A2 renamed EXP:A2
- net EXPANDER1:GPA7 renamed EXP:GPA7
- net EXPANDER1:INTA renamed EXP:INTA
- net EXPANDER1:INTB renamed EXP:INTB
- net EXPANDER1:NC renamed EXP:NC
- removed net EXPANDER1:GPA5: EXP:IC1.26
- removed net EXPANDER1:GPA6: EXP:IC1.27
- removed net EXPANDER1:RESET: EXP:IC1.18, EXPANDER1:R1.1
- new net EXP:RESET: EXP:IC1.18, EXP:R1.1
- new net N$18: DISPLAY1:VIN.P$1, IC1.3
- new net RX: DISPLAY1:RX.P$1, EXP:IC1.26
- new net TX: DISPLAY1:TX.P$1, EXP:IC1.27
- net +12V: now also IC1.1
- net +5V: now also EXP:C1.1, EXP:R1.2; no longer EXPANDER1:C1.1, EXPANDER1:R1.2
- net GND: now also DISPLAY1:GND.P$1, EXP:C1.2, IC1.2; no longer EXPANDER1:C1.2
Routing:
- net +12V: track 0.00 -> 73.4 mm, vias 0 -> 1
- net +5V: track 16.0 -> 81.1 mm, vias 0 -> 7
- net SDA: track 0.00 -> 54.3 mm, vias 0 -> 2
- net SCL: track 0.00 -> 49.0 mm, vias 0 -> 2
- net N$17: track 32.0 -> 0.00 mm
- net N$10: track 32.0 -> 0.00 mm
- net N$8: track 31.0 -> 0.00 mm
- net RX: track 0.00 -> 12.9 mm
- net TX: track 0.00 -> 12.7 mm
- net N$18: track 0.00 -> 5.35 mm
- net EXP:RESET: track 0.00 -> 4.02 mm
- net GND: track 32.4 -> 36.3 mm, vias 14 -> 16
- net EXPANDER1:RESET: track 3.67 -> 0.00 mm
- net HEADSTART-LED: track 43.2 -> 44.7 mm
- net N$5: track 80.9 -> 79.8 mm
Other:
- board text added: "+"
- board text added: "-"
- board text added: "CALIBRATION"
- board text added: "DEFENDER"
- board text added: "H"
- board text added: "K"
- board text added: "KICK"
- board text added: "M"
- board text added: "RESET"
- board text added: "RX"
- board text added: "SHIFT"
- board text added: "START"
- board text added: "STOP"
- board text added: "STRIKER"
- board text added: "TX"

Commit message: - brd (Labeling)
Parts:
- moved IN:U$1 0.79 mm to (49.8, 8.75)
Routing:
- net N$14: track 32.3 -> 31.4 mm
- net N$15: track 25.3 -> 24.7 mm
Other:
- board text added: "-->"
- board text added: "2002"
- board text added: "BALL"
- board text added: "Design by Oona"
- board text added: "Iceberg Robots"
- board text added: "PUI"
- board text added: "STATE"
- board text added: "www.iceberg-robots.de"

Commit message: - pui (Corrections)
Parts:
- moved DISPLAY1:GND 73.7 mm to (10.4, 14.7)
- moved DISPLAY1:RX 73.7 mm to (4.39, 14.7)
- moved DISPLAY1:TX 73.7 mm to (7.39, 14.7)
- moved DISPLAY1:VIN 73.7 mm to (13.1, 14.7)
- moved EXP:C1 2.50 mm to (68.7, 6.86)
- moved EXP:R1 1.46 mm to (61.5, 14.5)
Connections:
- net N$4 renamed RESET-B
- net N$5 renamed LED-IN
- removed net EXP:A0: EXP:IC1.15
- removed net EXP:A1: EXP:IC1.16
- removed net EXP:A2: EXP:IC1.17
- removed net EXP:GPA7: EXP:IC1.28
- removed net EXP:NC: EXP:IC1.11
- removed net N$1: X:X1.3, X:X1.5, X:X1.7
- removed net N$11: EXP:IC1.3, IN:S3.A1, IN:S3.A2
- removed net N$12: EXP:IC1.4, IN:U$1.A
- removed net N$13: EXP:IC1.5, IN:U$1.CENTER
- removed net N$14: EXP:IC1.6, IN:U$1.C
- removed net N$15: EXP:IC1.7, IN:U$1.D
- removed net N$16: EXP:IC1.8, IN:U$1.B
- removed net N$18: DISPLAY1:VIN.P$1, IC1.3
- removed net N$2: IN:S4.1, X:X1.8
- removed net N$3: IN:S5.1, X:X1.9
- removed net N$6: EXP:IC1.24, OUT:R6.1
- removed net N$7: EXP:IC1.25, OUT:R5.1
- removed net N$9: EXP:IC1.2, IN:S2.A1, IN:S2.A2
- new net CALIBRATION-B: EXP:IC1.2, IN:S3.A1, IN:S3.A2
- new net CENTER-J: EXP:IC1.25, IN:U$1.CENTER
- new net DEFENCE-LED: EXP:IC1.5, OUT:R6.1
- new net DOWN-J: EXP:IC1.26, IN:U$1.C
- new net KICK-B: EXP:IC1.1, IN:S2.A1, IN:S2.A2
- new net LEFT-J: EXP:IC1.24, IN:U$1.A
- new net RIGHT-J: EXP:IC1.27, IN:U$1.D
- new net START-B: IN:S4.1, X:X1.13
- new net STOP-B: IN:S5.1, X:X1.11
- new net STRIKER-LED: EXP:IC1.4, OUT:R5.1
- new net UP-J: EXP:IC1.28, IN:U$1.B
- net +5V: now also DISPLAY1:VIN.P$1, IC1.3, IN:S7.C, IN:S8.C, IN:S9.C
- net GND: now also EXP:IC1.15, EXP:IC1.16, EXP:IC1.17, EXP:IC1.6, EXP:IC1.7, EXP:IC1.8, X:X1.10, X:X1.12, X:X1.3, X:X1.5, X:X1.7; no longer IN:S7.C, IN:S8.C, IN:S9.C
- net RX: now also X:X1.9; no longer EXP:IC1.26
- net SHIFT-LED: now also EXP:IC1.3; no longer EXP:IC1.1
- net TX: now also X:X1.8; no longer EXP:IC1.27
Routing:
- net KICK-B: track 0.00 -> 86.6 mm
- net N$9: track 82.3 -> 0.00 mm, vias 2 -> 0
- net CALIBRATION-B: track 0.00 -> 77.7 mm
- net N$11: track 68.1 -> 0.00 mm
- net DEFENCE-LED: track 0.00 -> 47.3 mm
- net +5V: track 81.1 -> 124.9 mm, vias 7 -> 6
- net N$12: track 43.7 -> 0.00 mm
- net UP-J: track 0.00 -> 42.7 mm
- net DOWN-J: track 0.00 -> 42.5 mm, vias 0 -> 1
- net CENTER-J: track 0.00 -> 41.4 mm, vias 0 -> 2
- net N$13: track 38.8 -> 0.00 mm
- net LEFT-J: track 0.00 -> 36.0 mm, vias 0 -> 2
- net RIGHT-J: track 0.00 -> 35.9 mm
- net STRIKER-LED: track 0.00 -> 34.8 mm
- net N$14: track 31.4 -> 0.00 mm
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