File: pui20.brd (EAGLE design)
At the start: 95 x 30 mm, 37 parts, among them IC1 L7805

Commit message: - pui/lbr (Corrections 2.0)
Parts:
- added C1, C2: 200nF, iceberg20:C0805
- added EXP:R2, EXP:R3, EXP:R4: 330R, iceberg20:R0805
- OUT:R1, OUT:R2, OUT:R3, OUT:R4: value 330 -> 50R
- OUT:R5, OUT:R6: value R -> 220R
- moved EXP:C1 2.00 mm to (66.7, 6.86)
Connections:
- removed net EXP:INTA: EXP:IC1.20
- removed net EXP:INTB: EXP:IC1.19
- removed net X:INTERRUPT: X:X1.16
- new net EXP:N$1: EXP:IC1.21, EXP:R2.2
- new net EXP:N$2: EXP:IC1.22, EXP:R3.2
- new net EXP:N$3: EXP:IC1.23, EXP:R4.2
- new net INT-B: EXP:IC1.19, X:X1.16
- net +12V: now also C1.1
- net +5V: now also C2.1; no longer X:X1.2
- net GND: now also C1.2, C2.2; no longer EXP:IC1.6, EXP:IC1.7, EXP:IC1.8, X:X1.10, X:X1.12
- net HEADSTART-LED: now also EXP:R4.1; no longer EXP:IC1.23
- net KICKER-LED: now also EXP:R2.1; no longer EXP:IC1.21
- net MOTOR-LED: now also EXP:R3.1; no longer EXP:IC1.22
Routing:
- net INT-B: track 0.00 -> 70.1 mm, vias 0 -> 4
- net EXP:N$3: track 0.00 -> 38.4 mm, vias 0 -> 1
- net HEADSTART-LED: track 44.7 -> 6.59 mm, vias 0 -> 1
- net EXP:N$2: track 0.00 -> 34.5 mm, vias 0 -> 1
- net MOTOR-LED: track 38.9 -> 6.57 mm, vias 0 -> 1
- net EXP:N$1: track 0.00 -> 30.6 mm, vias 0 -> 1
- net KICKER-LED: track 34.9 -> 6.05 mm, vias 0 -> 1
- net +12V: track 72.5 -> 76.2 mm
- net CALIBRATION-B: track 77.7 -> 75.0 mm
- net +5V: track 124.9 -> 126.8 mm, vias 6 -> 10
- net GND: track 33.4 -> 31.7 mm
- net START-B: track 23.0 -> 21.9 mm
- net SDA: track 47.2 -> 48.3 mm
- net STOP-B: track 24.9 -> 23.9 mm
- net SCL: track 50.0 -> 49.2 mm
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