File: pui20.sch (EAGLE design)
At the start: 0 parts

Commit message: - pui.brd (Layout + Routing)
Changed lines of the file:
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@@
 <port name="STOP-B" side="left" coord="7.62" direction="out"/>
 <port name="RESET-B" side="left" coord="5.08" direction="out"/>
-<port name="KICKER-S" side="right" coord="-15.24" direction="out"/>
-<port name="HEADSTART-S" side="right" coord="-10.16" direction="out"/>
+<port name="KICKER-S" side="right" coord="-10.16" direction="out"/>
+<port name="HEADSTART-S" side="right" coord="-15.24" direction="out"/>
 <port name="MOTOR-S" side="right" coord="-12.7" direction="out"/>
 <port name="KICK-B" side="right" coord="7.62" direction="out"/>
 <port name="SHIFT-B" side="right" coord="10.16" direction="out"/>
 <port name="CALIBRATION-B" side="right" coord="5.08" direction="out"/>
-<port name="CENTER-J" side="right" coord="2.54" direction="out"/>
-<port name="DOWN-J" side="right" coord="0" direction="out"/>
-<port name="LEFT-J" side="right" coord="-2.54" direction="out"/>
+<port name="CENTER-J" side="right" coord="0" direction="out"/>
+<port name="DOWN-J" side="right" coord="-2.54" direction="out"/>
+<port name="LEFT-J" side="right" coord="2.54" direction="out"/>
 <port name="RIGHT-J" side="right" coord="-5.08" direction="out"/>
 <port name="UP-J" side="right" coord="-7.62" direction="out"/>
@@
 </segment>
 </net>
-<net name="N$12" class="0">
-<segment>
-<portref moduleinst="EINGABE1" port="CENTER-J"/>
-<portref moduleinst="EXPANDER1" port="GPB3"/>
-<wire x1="139.7" y1="137.16" x2="160.02" y2="137.16" width="0.1524" layer="91"/>
-</segment>
-</net>
-<net name="N$13" class="0">
-<segment>
-<portref moduleinst="EINGABE1" port="DOWN-J"/>
-<portref moduleinst="EXPANDER1" port="GPB4"/>
-<wire x1="139.7" y1="134.62" x2="160.02" y2="134.62" width="0.1524" layer="91"/>
-</segment>
-</net>
-<net name="N$14" class="0">
-<segment>
-<portref moduleinst="EINGABE1" port="LEFT-J"/>
-<portref moduleinst="EXPANDER1" port="GPB5"/>
-<wire x1="139.7" y1="132.08" x2="160.02" y2="132.08" width="0.1524" layer="91"/>
-</segment>
-</net>
 <net name="N$15" class="0">
 <segment>
@@
 <segment>
 <portref moduleinst="EINGABE1" port="KICKER-S"/>
-<portref moduleinst="EXPANDER1" port="GPA2"/>
-<wire x1="139.7" y1="119.38" x2="160.02" y2="119.38" width="0.1524" layer="91"/>
-<label x="139.7" y="119.38" size="1.778" layer="95"/>
+<portref moduleinst="EXPANDER1" port="GPA0"/>
+<wire x1="139.7" y1="124.46" x2="160.02" y2="124.46" width="0.1524" layer="91"/>
+<label x="139.7" y="124.46" size="1.778" layer="95"/>
 </segment>
 </net>
@@
 </segment>
 <segment>
+<portref moduleinst="EXPANDER1" port="GPA2"/>
 <portref moduleinst="EINGABE1" port="HEADSTART-S"/>
-<portref moduleinst="EXPANDER1" port="GPA0"/>
-<wire x1="139.7" y1="124.46" x2="160.02" y2="124.46" width="0.1524" layer="91"/>
-<label x="139.7" y="124.46" size="1.778" layer="95"/>
+<wire x1="160.02" y1="119.38" x2="139.7" y2="119.38" width="0.1524" layer="91"/>
+<label x="139.7" y="119.38" size="1.778" layer="95"/>
 </segment>
 </net>
@@
 </segment>
 </net>
+<net name="N$12" class="0">
+<segment>
+<portref moduleinst="EINGABE1" port="LEFT-J"/>
+<portref moduleinst="EXPANDER1" port="GPB3"/>
+<wire x1="139.7" y1="137.16" x2="160.02" y2="137.16" width="0.1524" layer="91"/>
+</segment>
+</net>
+<net name="N$13" class="0">
+<segment>
+<portref moduleinst="EINGABE1" port="CENTER-J"/>
+<portref moduleinst="EXPANDER1" port="GPB4"/>
+<wire x1="139.7" y1="134.62" x2="160.02" y2="134.62" width="0.1524" layer="91"/>
+</segment>
+</net>
+<net name="N$14" class="0">
+<segment>
+<portref moduleinst="EINGABE1" port="DOWN-J"/>
+<portref moduleinst="EXPANDER1" port="GPB5"/>
+<wire x1="139.7" y1="132.08" x2="160.02" y2="132.08" width="0.1524" layer="91"/>
+</segment>
+</net>

Commit message: + pui.sch (Display)
Parts:
- added IC1: L7805, iceberg20:L7805
Connections:
- new net +12V: IC1.VI
- new net +5V: IC1.VDD
- new net A0: IC1.A0
- new net A1: IC1.A1
- new net A2: IC1.A2
- new net GND: IC1.GND, IC1.VSS
- new net GPA0: IC1.GPA0
- new net GPA1: IC1.GPA1
- new net GPA2: IC1.GPA2
- new net GPA3: IC1.GPA3
- new net GPA4: IC1.GPA4
- new net GPA5: IC1.GPA5
- new net GPA6: IC1.GPA6
- new net GPA7: IC1.GPA7
- new net GPB0: IC1.GPB0
- new net GPB1: IC1.GPB1
- new net GPB2: IC1.GPB2
- new net GPB3: IC1.GPB3
- new net GPB4: IC1.GPB4
- new net GPB5: IC1.GPB5
- new net GPB6: IC1.GPB6
- new net GPB7: IC1.GPB7
- new net INTA: IC1.INTA
- new net INTB: IC1.INTB
- new net N$18: IC1.VO
- new net NC: IC1.NC
- new net RESET: IC1.RESET
- new net SCL: IC1.SCL
- new net SDA: IC1.SDA

Commit message: - pui (Corrections)
Connections:
- net GPA0 renamed KICKER-S
- net GPA1 renamed MOTOR-S
- net GPA2 renamed HEADSTART-S
- net GPA3 renamed LEFT-J
- net GPA4 renamed CENTER-J
- net GPA5 renamed DOWN-J
- net GPA6 renamed RIGHT-J
- net GPA7 renamed UP-J
- net GPB0 renamed KICK-B
- net GPB1 renamed CALIBRATION-B
- net GPB2 renamed SHIFT-B
- net GPB3 renamed STRIKER-LED
- net GPB4 renamed DEFENCE-LED
- removed net A0: IC1.A0
- removed net A1: IC1.A1
- removed net A2: IC1.A2
- removed net GPB5: IC1.GPB5
- removed net GPB6: IC1.GPB6
- removed net GPB7: IC1.GPB7
- removed net N$18: IC1.VO
- removed net NC: IC1.NC
- net +5V: now also IC1.VO
- net GND: now also IC1.A0, IC1.A1, IC1.A2, IC1.GPB5, IC1.GPB6, IC1.GPB7
Other:
- note added: "Ausgabe"
- note added: "Display"
- note added: "Eingabe"
- note added: "Expander"
- note added: "Übersicht"
- moved on the sheet: IC1

Commit message: - pui/lbr (Corrections 2.0)
Parts:
- added C1, C2: 200nF, iceberg20:C0805
Connections:
- net HEADSTART-S renamed N$3
- net KICKER-S renamed N$1
- net MOTOR-S renamed N$2
- removed net INTA: IC1.INTA
- net +12V: now also C1.1
- net +5V: now also C1.1, C2.1
- net GND: now also C1.2, C2.2; no longer IC1.GPB5, IC1.GPB6, IC1.GPB7
Other:
- moved on the sheet: IC1
